File: hardware/PPOW Power distribution module/ppow/ppow.kicad_sch (KiCad schematic)
At the start: 48 parts, among them J1 Conn_01x02_Male, J10 Screw_Terminal_01x02, J11 Screw_Terminal_01x02, J12 Screw_Terminal_01x02, J13 Screw_Terminal_01x02, J14 Screw_Terminal_01x02, J15 Screw_Terminal_01x02, J16 Screw_Terminal_01x02, J17 Screw_Terminal_01x02, J18 Screw_Terminal_01x02, J19 Screw_Terminal_01x02, J2 ATX-20, J20 Screw_Terminal_01x02, J21 Screw_Terminal_01x02, J22 Screw_Terminal_01x02, J23 Screw_Terminal_01x02, J24 Screw_Terminal_01x02, J25 Screw_Terminal_01x02, J26 Screw_Terminal_01x05, J27 Screw_Terminal_01x05, J28 Conn_01x03_Male, J29 Conn_01x03_Male, J3 Conn_01x04_Male, J4 Screw_Terminal_01x02, J5 Screw_Terminal_01x02, J6 Screw_Terminal_01x02, J7 Screw_Terminal_01x02, J8 Screw_Terminal_01x02, J9 Screw_Terminal_01x02, U1 ROM-0524S, U2 ROM-0524S

Commit message: 251205
Parts:
- F1, F2, F3, F4, F5, F6, F7, F8: value Fuse -> 1A F
- F10, F11, F9: value Fuse -> 0.5A F
- R1, R2: value 470 -> 2.2k
