File: hardware/PCOX COVOX module/pcox/pcox.kicad_pcb (KiCad board)
At the start: 2 copper layers, 57 parts, among them J1 Screw_Terminal_01x02, J2 Conn_02x40_Top_Bottom, J3 Screw_Terminal_01x02, J4 Screw_Terminal_01x02, J5 Screw_Terminal_01x02, SW1 SW_DIP_x08, U1 74LS32, U2 7809, U3 74HCT688, U4 MC3340P, U5 LM386, U6 74LS273

Commit message: 251228
Parts:
- removed C3: 1n, Capacitor_THT:C_Disc_D5.0mm_W2.5mm_P5.00mm
- C1: value 220u -> 100n; footprint Capacitor_THT:CP_Radial_D8.0mm_P3.80mm -> Capacitor_THT:C_Disc_D5.0mm_W2.5mm_P5.00mm
- C10: value 100n -> 220u; footprint Capacitor_THT:C_Disc_D5.0mm_W2.5mm_P5.00mm -> Capacitor_THT:CP_Radial_D8.0mm_P3.80mm
- C11: value 100u -> 1n
- C13: value 220u -> 50n; footprint Capacitor_THT:CP_Radial_D8.0mm_P3.80mm -> Capacitor_THT:C_Disc_D5.0mm_W2.5mm_P5.00mm
- C14: value 220u -> 1n; footprint Capacitor_THT:CP_Radial_D8.0mm_P3.80mm -> Capacitor_THT:C_Disc_D5.0mm_W2.5mm_P5.00mm
- C15: value 10u -> 220u; footprint Capacitor_THT:CP_Radial_D8.0mm_P2.50mm -> Capacitor_THT:CP_Radial_D8.0mm_P3.80mm
- C16, C7: value 100n -> 1u Ta; footprint Capacitor_THT:C_Disc_D5.0mm_W2.5mm_P5.00mm -> Capacitor_THT:CP_Radial_Tantal_D5.0mm_P2.50mm
- C17: value 50n -> 100n
- C18: value ** -> 100u; footprint Capacitor_THT:C_Disc_D5.0mm_W2.5mm_P5.00mm -> Capacitor_THT:CP_Radial_D8.0mm_P3.80mm
- C19: value 50n -> **
- C2: value 1n -> 47u; footprint Capacitor_THT:C_Disc_D5.0mm_W2.5mm_P5.00mm -> Capacitor_THT:CP_Radial_D8.0mm_P3.80mm
- C20: value 1u Ta -> 50n; footprint Capacitor_THT:CP_Radial_Tantal_D5.0mm_P2.50mm -> Capacitor_THT:C_Disc_D5.0mm_W2.5mm_P5.00mm
- C21: value 10n -> 220u; footprint Capacitor_THT:C_Disc_D5.0mm_W2.5mm_P5.00mm -> Capacitor_THT:CP_Radial_D8.0mm_P3.80mm
- C4: value 1u Ta -> 100n; footprint Capacitor_THT:CP_Radial_Tantal_D5.0mm_P2.50mm -> Capacitor_THT:C_Disc_D5.0mm_W2.5mm_P5.00mm
- C5: value 47u -> 100n; footprint Capacitor_THT:CP_Radial_D8.0mm_P3.80mm -> Capacitor_THT:C_Disc_D5.0mm_W2.5mm_P5.00mm
- C6: value 100n -> 10n
- C8: value 10u -> 100n; footprint Capacitor_THT:CP_Radial_D8.0mm_P2.50mm -> Capacitor_THT:C_Disc_D5.0mm_W2.5mm_P5.00mm
- C9: value 100n -> 10u; footprint Capacitor_THT:C_Disc_D5.0mm_W2.5mm_P5.00mm -> Capacitor_THT:CP_Radial_D5.0mm_P2.50mm
- D1: value D_Schottky -> 1N5395; footprint Diode_THT:D_DO-41_SOD81_P3.81mm_Vertical_AnodeUp -> Diode_THT:D_DO-15_P5.08mm_Vertical_KathodeUp
- D2: footprint Capacitor_THT:CP_Radial_D8.0mm_P3.80mm -> LED_THT:LED_Rectangular_W5.0mm_H2.0mm_Horizontal_O1.27mm_Z1.0mm
- J1: value Screw_Terminal_01x02 -> Conn_02x40_Top_Bottom; footprint TerminalBlock:TerminalBlock_bornier-2_P5.08mm -> pinhead:PinHeader_2x40_P2.54mm_Vertical_Top_Bottom
- J2: value Conn_02x40_Top_Bottom -> Screw_Terminal_01x02; footprint Connector_PinHeader_2.54mm:PinHeader_2x40_P2.54mm_Horizontal -> TerminalBlock:TerminalBlock_bornier-2_P5.08mm
- R1: value 3,3k -> 20k; footprint Resistor_THT:R_Axial_DIN0207_L6.3mm_D2.5mm_P5.08mm_Vertical -> Resistor_THT:R_Axial_DIN0207_L6.3mm_D2.5mm_P2.54mm_Vertical
- R10: value 47k-100k -> 10k; footprint Resistor_THT:R_Axial_DIN0207_L6.3mm_D2.5mm_P5.08mm_Vertical -> Resistor_THT:R_Axial_DIN0207_L6.3mm_D2.5mm_P2.54mm_Vertical
- R11, R13, R15, R17: value 20k -> 10k; footprint Resistor_THT:R_Axial_DIN0207_L6.3mm_D2.5mm_P5.08mm_Vertical -> Resistor_THT:R_Axial_DIN0207_L6.3mm_D2.5mm_P2.54mm_Vertical
- R12, R14, R16, R2, R4, R8, R9: footprint Resistor_THT:R_Axial_DIN0207_L6.3mm_D2.5mm_P5.08mm_Vertical -> Resistor_THT:R_Axial_DIN0207_L6.3mm_D2.5mm_P2.54mm_Vertical
- R18: value 10k -> 47k-100k; footprint Resistor_THT:R_Axial_DIN0207_L6.3mm_D2.5mm_P5.08mm_Vertical -> Resistor_THT:R_Axial_DIN0207_L6.3mm_D2.5mm_P2.54mm_Vertical
- R19: value 20k -> 470; footprint Resistor_THT:R_Axial_DIN0207_L6.3mm_D2.5mm_P5.08mm_Vertical -> Resistor_THT:R_Axial_DIN0207_L6.3mm_D2.5mm_P2.54mm_Vertical
- R20: value 10k -> *; footprint Resistor_THT:R_Axial_DIN0207_L6.3mm_D2.5mm_P5.08mm_Vertical -> Resistor_THT:R_Axial_DIN0207_L6.3mm_D2.5mm_P2.54mm_Vertical
- R21: value 10k -> 10; footprint Resistor_THT:R_Axial_DIN0207_L6.3mm_D2.5mm_P5.08mm_Vertical -> Resistor_THT:R_Axial_DIN0207_L6.3mm_D2.5mm_P2.54mm_Vertical
- R3, R5: value 10k -> 20k; footprint Resistor_THT:R_Axial_DIN0207_L6.3mm_D2.5mm_P5.08mm_Vertical -> Resistor_THT:R_Axial_DIN0207_L6.3mm_D2.5mm_P2.54mm_Vertical
- R6: value * -> 20k; footprint Resistor_THT:R_Axial_DIN0207_L6.3mm_D2.5mm_P5.08mm_Vertical -> Resistor_THT:R_Axial_DIN0207_L6.3mm_D2.5mm_P2.54mm_Vertical
- R7: value 10 -> 20k; footprint Resistor_THT:R_Axial_DIN0207_L6.3mm_D2.5mm_P5.08mm_Vertical -> Resistor_THT:R_Axial_DIN0207_L6.3mm_D2.5mm_P2.54mm_Vertical
- U2: value 7809 -> 74LS273; footprint Package_TO_SOT_THT:TO-220-3_Vertical -> Package_DIP:DIP-20_W7.62mm_Socket_LongPads
- U5: value LM386 -> 7809; footprint Package_DIP:DIP-8_W7.62mm_Socket_LongPads -> Package_TO_SOT_THT:TO-220-3_Horizontal_TabDown
- U6: value 74LS273 -> LM386; footprint Package_DIP:DIP-20_W7.62mm_Socket_LongPads -> Package_DIP:DIP-8_W7.62mm_Socket_LongPads
- moved J3 363.2 mm to (193.0, 60.3), turned to -90 degrees
- moved R8 349.1 mm to (188.0, 93.8), turned to -90 degrees
- moved R7 346.9 mm to (184.2, 93.8), turned to -90 degrees
- moved R17 344.1 mm to (191.8, 96.4)
- moved R16 342.0 mm to (188.0, 90.0), turned to 90 degrees
- moved R6 341.1 mm to (180.3, 93.8), turned to -90 degrees
- moved R2 336.6 mm to (165.1, 93.8), turned to -90 degrees
- moved C8 331.8 mm to (186.7, 65.4), turned to 90 degrees
- moved R15 327.4 mm to (184.2, 90.0), turned to 90 degrees
- moved R13 326.3 mm to (176.5, 90.0), turned to 90 degrees
- moved R18 324.1 mm to (172.7, 78.2)
- moved R1 321.5 mm to (161.3, 93.8), turned to -90 degrees
- moved R3 320.5 mm to (168.9, 93.8), turned to -90 degrees
- moved U2 319.4 mm to (158.8, 114.6), turned to 90 degrees
- moved R11 319.2 mm to (168.9, 90.0), turned to 90 degrees
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Connections:
- C1 pad 1: Net-(C1-Pad1) -> +5VD
- C10 pad 1: GNDA -> /+12VA
- C10 pad 2: +9VA -> GNDA
- C11 pad 1: +9VA -> /+12VA
- C12 pad 1: +5VD -> +9VA
- C13 pad 2: Net-(C13-Pad2) -> GNDA
- C14 pad 1: Net-(C14-Pad1) -> +9VA
- C14 pad 2: Net-(C14-Pad2) -> GNDA
- C15 pad 1: +5VD -> Net-(C15-Pad1)
- C15 pad 2: GNDA -> Net-(C15-Pad2)
- C16 pad 1: GNDA -> +9VA
- C16 pad 2: +5VD -> GNDA
- C17 pad 1: Net-(C17-Pad1) -> GNDA
- C17 pad 2: GNDA -> +9VA
- C18 pad 1: Net-(C18-Pad1) -> +9VA
- C18 pad 2: Net-(C18-Pad2) -> GNDA
- C19 pad 2: GNDA -> Net-(C19-Pad2)
- C2 pad 1: Net-(C1-Pad1) -> +5VD
- C20 pad 2: Net-(C20-Pad2) -> GNDA
- C21 pad 1: GNDA -> Net-(C21-Pad1)
- C21 pad 2: Net-(C20-Pad1) -> Net-(C21-Pad2)
- C4 pad 1: +9VA -> GNDA
- C4 pad 2: GNDA -> +5VD
- C6 pad 1: +5VD -> GNDA
- C6 pad 2: GNDA -> Net-(C6-Pad2)
- C7 pad 1: GNDA -> Net-(C6-Pad2)
- C8 pad 1: Net-(C7-Pad2) -> GNDA
- C8 pad 2: GNDA -> Net-(C8-Pad2)
- C9 pad 1: +9VA -> Net-(C8-Pad2)
- D1 pad 1: Net-(C1-Pad1) -> /+12VA
- D1 pad 2: Net-(D1-Pad2) -> GNDA
- J1 pad 1: Net-(D1-Pad2) -> unconnected-(J1-Pad1)
- J1 pad 2: GNDA -> unconnected-(J1-Pad2)
- J2 pad 1: unconnected-(J2-Pad1) -> Net-(C7-Pad2)
- J2 pad 2: unconnected-(J2-Pad2) -> GNDA
- J3 pad 1: Net-(C20-Pad2) -> Net-(C8-Pad2)
- J4 pad 1: Net-(C7-Pad2) -> /+12VA
- J5 pad 1: Net-(C14-Pad2) -> Net-(C21-Pad2)
- R1 pad 1: GNDA -> Net-(R1-Pad1)
- R1 pad 2: Net-(D2-Pad1) -> Net-(R1-Pad2)
- R10 pad 1: GNDA -> Net-(R10-Pad1)
- R10 pad 2: Net-(C20-Pad2) -> Net-(R1-Pad1)
- R11 pad 2: Net-(R11-Pad2) -> Net-(R10-Pad1)
- R12 pad 1: Net-(R11-Pad2) -> Net-(R12-Pad1)
- R12 pad 2: Net-(R12-Pad2) -> Net-(R11-Pad1)
- R13 pad 2: Net-(R13-Pad2) -> Net-(R12-Pad1)
- R14 pad 1: Net-(R13-Pad2) -> Net-(R6-Pad1)
- R14 pad 2: Net-(R11-Pad2) -> Net-(R13-Pad1)
- R15 pad 2: Net-(R15-Pad2) -> Net-(R6-Pad1)
- R16 pad 1: Net-(R15-Pad2) -> Net-(R16-Pad1)
- R16 pad 2: Net-(R13-Pad2) -> Net-(R15-Pad1)
- R17 pad 1: Net-(R17-Pad1) -> Net-(R16-Pad1)
- R17 pad 2: Net-(R17-Pad2) -> Net-(C6-Pad2)
- R18 pad 1: Net-(R17-Pad2) -> GNDA
- R18 pad 2: Net-(R15-Pad2) -> Net-(C7-Pad2)
- R19 pad 1: Net-(R19-Pad1) -> GNDA
- R19 pad 2: Net-(R19-Pad2) -> Net-(D2-Pad1)
- R2 pad 1: Net-(R2-Pad1) -> Net-(R10-Pad1)
- R20 pad 1: Net-(R19-Pad2) -> Net-(C19-Pad1)
- R20 pad 2: Net-(R17-Pad2) -> Net-(R20-Pad2)
- R21 pad 1: Net-(R19-Pad2) -> Net-(C20-Pad1)
- R21 pad 2: Net-(C20-Pad1) -> Net-(C21-Pad1)
- R3 pad 1: Net-(R2-Pad2) -> Net-(R11-Pad1)
- R3 pad 2: GNDA -> Net-(R3-Pad2)
- R4 pad 1: Net-(R4-Pad1) -> Net-(R12-Pad1)
- R5 pad 1: Net-(R4-Pad2) -> Net-(R13-Pad1)
- R5 pad 2: Net-(R2-Pad2) -> Net-(R5-Pad2)
- R6 pad 1: Net-(C18-Pad1) -> Net-(R6-Pad1)
- R7 pad 1: Net-(C19-Pad1) -> Net-(R15-Pad1)
- R7 pad 2: Net-(C14-Pad1) -> Net-(R7-Pad2)
- R8 pad 1: Net-(R8-Pad1) -> Net-(R16-Pad1)
- R8 pad 2: Net-(R12-Pad2) -> Net-(R8-Pad2)
- R9 pad 1: Net-(R12-Pad2) -> Net-(R1-Pad1)
- R9 pad 2: Net-(R4-Pad2) -> GNDA
- RN1 pad 2: Net-(RN1-Pad2) -> Net-(SW1-Pad16)
- SW1 pad 10: Net-(RN1-Pad3) -> Net-(RN1-Pad8)
- SW1 pad 11: Net-(RN1-Pad4) -> Net-(RN1-Pad7)
- SW1 pad 12: Net-(RN1-Pad5) -> Net-(RN1-Pad6)
- SW1 pad 13: Net-(RN1-Pad6) -> Net-(RN1-Pad5)
- SW1 pad 14: Net-(RN1-Pad7) -> Net-(RN1-Pad4)
- SW1 pad 15: Net-(RN1-Pad8) -> Net-(RN1-Pad3)
- SW1 pad 16: Net-(RN1-Pad9) -> Net-(SW1-Pad16)
- SW1 pad 9: Net-(RN1-Pad2) -> Net-(RN1-Pad9)
- U1 pad 3: Net-(U6-Pad11) -> Net-(U1-Pad3)
- U2 pad 1: Net-(C1-Pad1) -> /RESET
- U2 pad 2: GNDA -> Net-(R1-Pad2)
- U2 pad 3: +9VA -> /D0
- U3 pad 17: Net-(RN1-Pad2) -> Net-(SW1-Pad16)
- U4 pad 1: Net-(C20-Pad2) -> Net-(C7-Pad2)
- U4 pad 2: Net-(C7-Pad2) -> Net-(C8-Pad2)
- U4 pad 6: Net-(C17-Pad1) -> Net-(C13-Pad1)
- U4 pad 7: Net-(C13-Pad1) -> Net-(C15-Pad1)
- U5 pad 1: Net-(R6-Pad2) -> /+12VA
- U5 pad 3: Net-(C13-Pad2) -> +9VA
- U6 pad 1: /RESET -> Net-(R20-Pad2)
- U6 pad 2: Net-(R2-Pad1) -> GNDA
- U6 pad 3: /D0 -> Net-(C15-Pad2)
- U6 pad 4: /D1 -> GNDA
- U6 pad 5: Net-(R4-Pad1) -> Net-(C21-Pad1)
- U6 pad 6: Net-(R8-Pad1) -> +9VA
- U6 pad 7: /D2 -> unconnected-(U6-Pad7)
- U6 pad 8: /D3 -> Net-(C19-Pad2)
Routing:
- net GNDA: track 0.00 -> 563.5 mm
- net +5VD: track 0.00 -> 170.4 mm
- net /-IORQ: track 0.00 -> 69.3 mm, vias 0 -> 1
- net Net-(RN1-Pad9): track 0.00 -> 49.8 mm
- net Net-(U1-Pad3): track 0.00 -> 46.3 mm, vias 0 -> 2
- net Net-(RN1-Pad8): track 0.00 -> 42.1 mm
- net /A7: track 0.00 -> 41.6 mm
- net /A0: track 0.00 -> 38.9 mm
- net Net-(R8-Pad2): track 0.00 -> 37.3 mm, vias 0 -> 2
- net /-WR: track 0.00 -> 36.5 mm
- net /A6: track 0.00 -> 35.7 mm
- net Net-(RN1-Pad7): track 0.00 -> 35.6 mm
- net /D7: track 0.00 -> 35.0 mm, vias 0 -> 2
- net /A1: track 0.00 -> 32.4 mm
- net /D6: track 0.00 -> 31.8 mm, vias 0 -> 2
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Other:
- board outline added: 101.6 x 53.3 mm
- board text added: "analog GND"
- board text added: "digital GND"

Commit message: 251230
Parts:
- C10: renamed from C11; footprint Capacitor_THT:C_Disc_D5.0mm_W2.5mm_P5.00mm -> Capacitor_THT:C_Disc_D5.0mm_W2.5mm_P2.50mm
- C13: renamed from C14; footprint Capacitor_THT:C_Disc_D5.0mm_W2.5mm_P5.00mm -> Capacitor_THT:C_Disc_D5.0mm_W2.5mm_P2.50mm
- J2, J3, J4, J5: footprint TerminalBlock:TerminalBlock_bornier-2_P5.08mm -> TerminalBlock:TerminalBlock_MaiXu_MX126-5.0-02P_1x02_P5.00mm
- moved C12 130.3 mm to (173.7, 63.5), turned to 90 degrees
- moved C18 123.3 mm to (154.3, 78.1), turned to 180 degrees
- moved R21 118.4 mm to (146.1, 69.2), turned to 90 degrees
- moved R20 116.9 mm to (157.5, 78.1)
- moved C19 108.3 mm to (146.1, 73.7), turned to -90 degrees
- moved C13 94.1 mm to (125.8, 78.7)
- moved D2 90.4 mm to (132.7, 67.9), turned to 180 degrees
- moved C15 75.6 mm to (133.3, 76.2), turned to -90 degrees
- moved C9 51.4 mm to (101.1, 75.6)
- moved C10 47.5 mm to (111.8, 78.7), turned to 180 degrees
- moved R19 46.1 mm to (130.4, 72.4), turned to 0 degrees
- moved C17 42.0 mm to (168.2, 61.6), turned to 180 degrees
- moved D1 41.6 mm to (101.0, 67.3)
- moved C8 18.4 mm to (179.7, 59.7), turned to -90 degrees
- moved J5 17.8 mm to (144.8, 60.3)
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- renumbered C12 to C11, C13 to C12, C15 to C14, C16 to C15, C17 to C16, C18 to C17, C19 to C18, C20 to C19, C21 to C20, C4 to C3, C5 to C4, C6 to C5, C7 to C6, C8 to C7, C9 to C8, C10 to C9
Routing:
- net +9VA: track 4.39 -> 123.5 mm
- net +5VD: track 170.4 -> 83.2 mm
- net /+12VA: track 0.00 -> 44.7 mm
- net GNDA: track 563.5 -> 605.3 mm
- net Net-(J2-Pin_1): track 6.46 -> 31.4 mm
- net Net-(J3-Pin_1): track 13.8 -> 31.9 mm
- net Net-(C20-Pad1): track 0.00 -> 17.0 mm
- net Net-(J5-Pin_1): track 0.00 -> 13.6 mm
- net Net-(U4-Output): track 17.7 -> 5.51 mm
- net Net-(U4-Roll-off): track 0.00 -> 9.35 mm
- net Net-(U6-+): track 0.00 -> 6.69 mm
- net Net-(D2-K): track 0.00 -> 4.59 mm
- net Net-(C18-Pad2): track 0.00 -> 4.57 mm
- net Net-(C19-Pad1): track 0.00 -> 4.44 mm
- net Net-(R20-Pad2): track 0.00 -> 4.35 mm
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Other:
- board size 101.6 x 53.3 mm -> 102.6 x 72.4 mm
- board text added: "PCOX"
- board text added: "Pozsár Zsolt 2025"

Commit message: 260105
Connections:
- RN1 pad 1: GNDA -> +5VD
Routing:
- net +5VD: track 83.2 -> 112.3 mm
- net GNDA: track 605.3 -> 595.5 mm
Changed lines of the file:
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@@
 		(tenting front back)
 		(pcbplotparams
-			(layerselection 0x00000000_00000000_55555555_55555571)
-			(plot_on_all_layers_selection 0x00000000_00000000_00000000_02000000)
+			(layerselection 0x00000000_00000000_55555555_5755557f)
+			(plot_on_all_layers_selection 0x00000000_00000000_00000000_00000000)
 			(disableapertmacros no)
 			(usegerberextensions no)
@@
 			(dashed_line_gap_ratio 3.000000)
 			(svgprecision 6)
-			(plotframeref yes)
+			(plotframeref no)
 			(mode 1)
 			(useauxorigin no)
@@
 			(crossoutdnponfab yes)
 			(subtractmaskfromsilk no)
-			(outputformat 4)
+			(outputformat 1)
 			(mirror no)
-			(drillshape 2)
+			(drillshape 0)
 			(scaleselection 1)
 			(outputdirectory "")
@@
 			(layers "*.Cu" "*.Mask")
 			(remove_unused_layers no)
-			(net 9 "GNDA")
+			(net 10 "+5VD")
 			(pinfunction "common")
 			(pintype "passive")
@@
 	)
 	(segment
-		(start 113.605 92.695)
-		(end 114.315 92.695)
-		(width 0.25)
-		(layer "F.Cu")
-		(net 9)
-	)
-	(segment
 		(start 121.285 115.57)
 		(end 121.255 115.54)
@@
 	)
 	(segment
-		(start 113.605 84.395)
-		(end 113.03 83.82)
-		(width 1.27)
-		(layer "B.Cu")
-		(net 9)
-	)
-	(segment
 		(start 178.5 78)
 		(end 178.5 81.215)
@@
 	)
 	(segment
-		(start 113.605 92.695)
-		(end 113.605 84.395)
-		(width 1.27)
-		(layer "B.Cu")
-		(net 9)
-	)
-	(segment
 		(start 156.21 97.79)
 		(end 156.21 96.12)
@@
 	)
 	(segment
+		(start 126.92 83.82)
+		(end 129.54 83.82)
+		(width 1.27)
+		(layer "F.Cu")
+		(net 10)
+	)
+	(segment
 		(start 135.128 99.314)
 		(end 134.112 98.298)
@@
 	)
 	(segment
-		(start 129.86 85.96)
-		(end 140.43 85.96)
+		(start 129.46 83.9)
+		(end 129.54 83.82)
 		(width 1.27)
 		(layer "F.Cu")
@@
 	)
 	(segment
+		(start 129.46 86.36)
+		(end 129.46 83.9)
+		(width 1.27)
+		(layer "F.Cu")
+		(net 10)
+	)
+	(segment
 		(start 134.112 98.298)
 		(end 134.112 95.808)
@@
 	)
 	(segment
+		(start 126.92 83.82)
+		(end 114.935 83.82)
+		(width 1.27)
+		(layer "F.Cu")
+		(net 10)
+	)
+	(segment
+		(start 114.935 83.82)
+		(end 113.605 85.15)
+		(width 1.27)
+		(layer "F.Cu")
+		(net 10)
+	)
+	(segment
+		(start 113.605 85.15)
+		(end 113.605 92.695)
+		(width 1.27)
+		(layer "F.Cu")
+		(net 10)
+	)
+	(segment
+		(start 113.605 92.695)
+		(end 114.315 92.695)
+		(width 0.25)
+		(layer "F.Cu")
+		(net 10)
+	)
+	(segment
 		(start 140.97 90.17)
 		(end 140.97 86.5)
@@
 	)
 	(segment
-		(start 129.46 86.36)
-		(end 129.86 85.96)
+		(start 140.97 84.455)
+		(end 140.97 86.5)
+		(width 1.27)
+		(layer "F.Cu")
+		(net 10)
+	)
+	(segment
+		(start 129.54 83.82)
+		(end 140.335 83.82)
 		(width 1.27)
 		(layer "F.Cu")
@@
 	)
 	(segment
-		(start 140.43 85.96)
-		(end 140.97 86.5)
+		(start 140.335 83.82)
+		(end 140.97 84.455)
 		(width 1.27)
 		(layer "F.Cu")
