File: hardware/PCOX COVOX module/pcox/pcox.kicad_sch (KiCad schematic)
At the start: 57 parts, among them J1 Screw_Terminal_01x02, J2 Conn_02x40_Top_Bottom, J3 Screw_Terminal_01x02, J4 Screw_Terminal_01x02, J5 Screw_Terminal_01x02, SW1 SW_DIP_x08, U1 74LS32, U2 7809, U3 74HCT688, U4 MC3340P, U5 LM386, U6 74LS273

Commit message: 251228
Parts:
- removed C15: 10u, Capacitor_THT:CP_Radial_D8.0mm_P2.50mm, symbol Device:C_Polarized
- removed D1: D_Schottky, Diode_THT:D_DO-41_SOD81_P3.81mm_Vertical_AnodeUp, symbol Device:D_Schottky
- added D1: 1N5395, Diode_THT:D_DO-15_P5.08mm_Vertical_KathodeUp, symbol Device:D
- C18: renamed from C11; footprint Capacitor_THT:C_Disc_D5.0mm_W2.5mm_P5.00mm -> Capacitor_THT:CP_Radial_D8.0mm_P3.80mm
- C9: renamed from C8; footprint Capacitor_THT:CP_Radial_D8.0mm_P2.50mm -> Capacitor_THT:CP_Radial_D5.0mm_P2.50mm
- D2: footprint Capacitor_THT:CP_Radial_D8.0mm_P3.80mm -> LED_THT:LED_Rectangular_W5.0mm_H2.0mm_Horizontal_O1.27mm_Z1.0mm
- J1: renamed from J2; footprint Connector_PinHeader_2.54mm:PinHeader_2x40_P2.54mm_Horizontal -> pinhead:PinHeader_2x40_P2.54mm_Vertical_Top_Bottom
- R1: renamed from R2; footprint Resistor_THT:R_Axial_DIN0207_L6.3mm_D2.5mm_P5.08mm_Vertical -> Resistor_THT:R_Axial_DIN0207_L6.3mm_D2.5mm_P2.54mm_Vertical
- R10: renamed from R5; footprint Resistor_THT:R_Axial_DIN0207_L6.3mm_D2.5mm_P5.08mm_Vertical -> Resistor_THT:R_Axial_DIN0207_L6.3mm_D2.5mm_P2.54mm_Vertical
- R11: renamed from R9; footprint Resistor_THT:R_Axial_DIN0207_L6.3mm_D2.5mm_P5.08mm_Vertical -> Resistor_THT:R_Axial_DIN0207_L6.3mm_D2.5mm_P2.54mm_Vertical
- R12: footprint Resistor_THT:R_Axial_DIN0207_L6.3mm_D2.5mm_P5.08mm_Vertical -> Resistor_THT:R_Axial_DIN0207_L6.3mm_D2.5mm_P2.54mm_Vertical
- R13: renamed from R14; footprint Resistor_THT:R_Axial_DIN0207_L6.3mm_D2.5mm_P5.08mm_Vertical -> Resistor_THT:R_Axial_DIN0207_L6.3mm_D2.5mm_P2.54mm_Vertical
- R14: renamed from R16; footprint Resistor_THT:R_Axial_DIN0207_L6.3mm_D2.5mm_P5.08mm_Vertical -> Resistor_THT:R_Axial_DIN0207_L6.3mm_D2.5mm_P2.54mm_Vertical
- R15: renamed from R18; footprint Resistor_THT:R_Axial_DIN0207_L6.3mm_D2.5mm_P5.08mm_Vertical -> Resistor_THT:R_Axial_DIN0207_L6.3mm_D2.5mm_P2.54mm_Vertical
- R16: renamed from R20; footprint Resistor_THT:R_Axial_DIN0207_L6.3mm_D2.5mm_P5.08mm_Vertical -> Resistor_THT:R_Axial_DIN0207_L6.3mm_D2.5mm_P2.54mm_Vertical
- R17: renamed from R21; footprint Resistor_THT:R_Axial_DIN0207_L6.3mm_D2.5mm_P5.08mm_Vertical -> Resistor_THT:R_Axial_DIN0207_L6.3mm_D2.5mm_P2.54mm_Vertical
- R18: renamed from R10; footprint Resistor_THT:R_Axial_DIN0207_L6.3mm_D2.5mm_P5.08mm_Vertical -> Resistor_THT:R_Axial_DIN0207_L6.3mm_D2.5mm_P2.54mm_Vertical
- R19: renamed from R1; value 3,3k -> 470; footprint Resistor_THT:R_Axial_DIN0207_L6.3mm_D2.5mm_P5.08mm_Vertical -> Resistor_THT:R_Axial_DIN0207_L6.3mm_D2.5mm_P2.54mm_Vertical
- R2: renamed from R4; footprint Resistor_THT:R_Axial_DIN0207_L6.3mm_D2.5mm_P5.08mm_Vertical -> Resistor_THT:R_Axial_DIN0207_L6.3mm_D2.5mm_P2.54mm_Vertical
- R20: renamed from R6; footprint Resistor_THT:R_Axial_DIN0207_L6.3mm_D2.5mm_P5.08mm_Vertical -> Resistor_THT:R_Axial_DIN0207_L6.3mm_D2.5mm_P2.54mm_Vertical
- R21: renamed from R7; footprint Resistor_THT:R_Axial_DIN0207_L6.3mm_D2.5mm_P5.08mm_Vertical -> Resistor_THT:R_Axial_DIN0207_L6.3mm_D2.5mm_P2.54mm_Vertical
- R3: renamed from R8; footprint Resistor_THT:R_Axial_DIN0207_L6.3mm_D2.5mm_P5.08mm_Vertical -> Resistor_THT:R_Axial_DIN0207_L6.3mm_D2.5mm_P2.54mm_Vertical
- R4: renamed from R11; footprint Resistor_THT:R_Axial_DIN0207_L6.3mm_D2.5mm_P5.08mm_Vertical -> Resistor_THT:R_Axial_DIN0207_L6.3mm_D2.5mm_P2.54mm_Vertical
- R5: renamed from R13; footprint Resistor_THT:R_Axial_DIN0207_L6.3mm_D2.5mm_P5.08mm_Vertical -> Resistor_THT:R_Axial_DIN0207_L6.3mm_D2.5mm_P2.54mm_Vertical
- R6: renamed from R15; footprint Resistor_THT:R_Axial_DIN0207_L6.3mm_D2.5mm_P5.08mm_Vertical -> Resistor_THT:R_Axial_DIN0207_L6.3mm_D2.5mm_P2.54mm_Vertical
- R7: renamed from R17; footprint Resistor_THT:R_Axial_DIN0207_L6.3mm_D2.5mm_P5.08mm_Vertical -> Resistor_THT:R_Axial_DIN0207_L6.3mm_D2.5mm_P2.54mm_Vertical
- R8: renamed from R19; footprint Resistor_THT:R_Axial_DIN0207_L6.3mm_D2.5mm_P5.08mm_Vertical -> Resistor_THT:R_Axial_DIN0207_L6.3mm_D2.5mm_P2.54mm_Vertical
- R9: renamed from R3; footprint Resistor_THT:R_Axial_DIN0207_L6.3mm_D2.5mm_P5.08mm_Vertical -> Resistor_THT:R_Axial_DIN0207_L6.3mm_D2.5mm_P2.54mm_Vertical
- U5: renamed from U2; footprint Package_TO_SOT_THT:TO-220-3_Vertical -> Package_TO_SOT_THT:TO-220-3_Horizontal_TabDown
- renumbered C6 to C1, C1 to C10, C2 to C11, C9 to C12, C17 to C13, C3 to C14, C13 to C15, C4 to C16, C10 to C17, C18 to C19, C5 to C2, C19 to C20, C14 to C21, C16 to C4, C12 to C5, C21 to C6, C20 to C7, C7 to C8, J3 to J2, J4 to J3, J1 to J4, U6 to U2, U5 to U6
Connections:
- net +5VD: now also J1.58 (Pin_58)
- net GNDA: now also J1.57 (Pin_57), D1.2 (A)
- net at R11.1, R12.2: now also R3.1; no longer R3.2
- net at R10.1, R11.2: now also R2.1; no longer R2.2
- net at U2.6 (Q2): now also R3.2; no longer R3.1
- net +12VA: now reaches C10.1, C11.1, U5.1 (IN)
- net +12VA: now also J4.1 (Pin_1), D1.1 (K)
- net at R13.1, R14.2: now also R5.1; no longer R5.2
- net at R12.1, R13.2: now also R4.1; no longer R4.2
- net at R8.1: now also R16.1, R17.1; no longer U2.19 (Q7)
- net at R10.2, R9.1: now also R1.1; no longer R1.2
- net at R6.1: now also R14.1, R15.2; no longer U2.15 (Q5)
- net at RN1.3 (R2), U3.15 (P6): now also SW1.15; no longer SW1.10
- net at RN1.4 (R3), U3.13 (P5): now also SW1.14; no longer SW1.11
- net at RN1.5 (R4), U3.11 (P4): now also SW1.13; no longer SW1.12
- net at RN1.6 (R5), U3.8 (P3): now also SW1.12; no longer SW1.13
- net at RN1.7 (R6), U3.6 (P2): now also SW1.11; no longer SW1.14
- net at RN1.8 (R7), U3.4 (P1): now also SW1.10; no longer SW1.15
- net at RN1.9 (R8), U3.2 (P0): now also SW1.9; no longer SW1.16
- net at RN1.2 (R1), U3.17 (P7): now also SW1.16; no longer SW1.9
- net at U2.5 (Q1): now also R2.2; no longer R2.1
- net at R7.1: now also R15.1, R16.2; no longer U2.16 (Q6)
- net at U2.12 (Q4): now also R5.2; no longer R5.1
- net at U2.2 (Q0): now also R1.2; no longer R1.1
- net at U2.9 (Q3): now also R4.2; no longer R4.1
- new net: R8.2, U2.19 (Q7)
- new net: R6.2, U2.15 (Q5)
- new net: R7.2, U2.16 (Q6)
- no-connect marks 65 -> 63
Other:
- moved on the sheet: R1, R2, R3, R4, R5, R6, R7, R8, SW1

Commit message: 251230
Parts:
- C10: renamed from C11; footprint Capacitor_THT:C_Disc_D5.0mm_W2.5mm_P5.00mm -> Capacitor_THT:C_Disc_D5.0mm_W2.5mm_P2.50mm
- C13: renamed from C14; footprint Capacitor_THT:C_Disc_D5.0mm_W2.5mm_P5.00mm -> Capacitor_THT:C_Disc_D5.0mm_W2.5mm_P2.50mm
- J2, J3, J4, J5: footprint TerminalBlock:TerminalBlock_bornier-2_P5.08mm -> TerminalBlock:TerminalBlock_MaiXu_MX126-5.0-02P_1x02_P5.00mm
- renumbered C12 to C11, C13 to C12, C15 to C14, C16 to C15, C17 to C16, C18 to C17, C19 to C18, C20 to C19, C21 to C20, C4 to C3, C5 to C4, C6 to C5, C7 to C6, C8 to C7, C9 to C8, C10 to C9
Other:
- note added: "analog GND"
- note added: "digital GND"
- note removed: "common (a/d) ground"
- moved on the sheet: C1, C10, C11, C12, C13, C14, C15, C16, C17, C18, C19, C2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

Commit message: 260105
Connections:
- net +5VD: now also RN1.1 (common)
- net GNDA: no longer RN1.1 (common)
Changed lines of the file:
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@@
 	(wire
 		(pts
+			(xy 71.12 76.2) (xy 71.12 77.47)
+		)
+		(stroke
+			(width 0)
+			(type default)
+		)
+	)
+	(wire
+		(pts
 			(xy 83.82 85.09) (xy 95.25 85.09)
 		)
@@
 	(wire
 		(pts
+			(xy 71.12 77.47) (xy 73.66 77.47)
+		)
+		(stroke
+			(width 0)
+			(type default)
+		)
+	)
+	(wire
+		(pts
 			(xy 76.2 130.175) (xy 76.2 181.61)
 		)
@@
 	(wire
 		(pts
-			(xy 72.39 77.47) (xy 73.66 77.47)
-		)
-		(stroke
-			(width 0)
-			(type default)
-		)
-	)
-	(wire
-		(pts
 			(xy 248.92 139.7) (xy 251.46 139.7)
 		)
@@
 	)
 	(symbol
-		(lib_id "power:GNDD")
-		(at 72.39 77.47 270)
-		(unit 1)
-		(exclude_from_sim no)
-		(in_bom yes)
-		(on_board yes)
-		(dnp no)
-		(fields_autoplaced yes)
-		(property "Reference" "#PWR07"
-			(at 66.04 77.47 0)
-			(effects
-				(font
-					(size 1.27 1.27)
-				)
-				(hide yes)
-			)
-		)
-		(property "Value" "GNDD"
-			(at 68.58 77.4699 90)
-			(effects
-				(font
-					(size 1.27 1.27)
-				)
-				(justify right)
-				(hide yes)
-			)
-		)
-		(property "Footprint" ""
-			(at 72.39 77.47 0)
-			(effects
-				(font
-					(size 1.27 1.27)
-				)
-				(hide yes)
-			)
-		)
-		(property "Datasheet" ""
-			(at 72.39 77.47 0)
-			(effects
-				(font
-					(size 1.27 1.27)
-				)
-				(hide yes)
-			)
-		)
-		(property "Description" ""
-			(at 72.39 77.47 0)
-			(effects
-				(font
-					(size 1.27 1.27)
-				)
-			)
-		)
-		(pin "1"
-		)
-		(instances
-			(project ""
-				(path "/2b98932b-1694-4573-88df-6f0ce09fa9d6"
-					(reference "#PWR07")
-					(unit 1)
-				)
-			)
-		)
-	)
-	(symbol
 		(lib_id "74xx:74LS32")
 		(at 147.955 64.77 0)
@@
 					(unit 1)
 				)
+			)
+		)
+	)
+	(symbol
+		(lib_id "power:+5VD")
+		(at 71.12 76.2 0)
+		(unit 1)
+		(exclude_from_sim no)
+		(in_bom yes)
+		(on_board yes)
+		(dnp no)
+		(property "Reference" "#PWR07"
+			(at 71.12 80.01 0)
+			(effects
+				(font
+					(size 1.27 1.27)
+				)
+				(hide yes)
+			)
+		)
+		(property "Value" "+5VD"
+			(at 71.12 71.12 0)
+			(effects
+				(font
+					(size 1.27 1.27)
+				)
+			)
+		)
+		(property "Footprint" ""
+			(at 71.12 76.2 0)
+			(effects
+				(font
+					(size 1.27 1.27)
+				)
+				(hide yes)
+			)
+		)
+		(property "Datasheet" ""
+			(at 71.12 76.2 0)
+			(effects
+				(font
+					(size 1.27 1.27)
+				)
+				(hide yes)
+			)
+		)
+		(property "Description" ""
+			(at 71.12 76.2 0)
+			(effects
+				(font
+					(size 1.27 1.27)
+				)
+			)
+		)
+		(pin "1"
+		)
+		(instances
+			(project "pcox"
+				(path "/2b98932b-1694-4573-88df-6f0ce09fa9d6"
+					(reference "#PWR07")
+					(unit 1)
+				)
