File: _planning/pemx/pemx.kicad_sch (KiCad schematic)
At the start: 79 parts, among them J1 Conn_01x03_Male, J2 Conn_01x06, J3 Conn_02x13_Top_Bottom, J4 Screw_Terminal_01x02, J5 Conn_01x03_Male, U1 74LS138, U10 74LS173, U11 74LS173, U12 27512, U13 27512, U14 27512, U15 27512, U16 27512, U17 27512, U18 27512, U19 27512, U2 74LS245, U3 74LS245, U4 DS1833, U5 74LS173, U6 74LS173, U7 74LS173, U8 74LS122, U9 74LS138

Commit message: 260110
Parts:
- J3: footprint Connector_PinHeader_2.54mm:PinHeader_2x13_P2.54mm_Vertical -> pinhead:PinHeader_2x13_P2.54mm_Vertical_Top_Bottom
Connections:
- net BD0: now also J3.10 (Pin_10); no longer J3.13 (Pin_13)
- net BD1: now also J3.23 (Pin_23); no longer J3.26 (Pin_26)
- net BD2: now also J3.11 (Pin_11); no longer J3.12 (Pin_12)
- net BD3: now also J3.24 (Pin_24); no longer J3.25 (Pin_25)
- net BD4: now also J3.12 (Pin_12); no longer J3.11 (Pin_11)
- net BD5: now also J3.25 (Pin_25); no longer J3.24 (Pin_24)
- net BD6: now also J3.13 (Pin_13); no longer J3.10 (Pin_10)
- net BD7: now also J3.26 (Pin_26); no longer J3.23 (Pin_23)
Changed lines of the file:
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@@
     (effects (font (size 1.27 1.27)) (justify right bottom))
   )
-  (label "BD1" (at 33.02 170.815 180)
+  (label "BD7" (at 33.02 170.815 180)
     (effects (font (size 1.27 1.27)) (justify right bottom))
   )
@@
     (effects (font (size 1.27 1.27)) (justify left bottom))
   )
-  (label "BD5" (at 33.02 165.735 180)
+  (label "BD3" (at 33.02 165.735 180)
     (effects (font (size 1.27 1.27)) (justify right bottom))
   )
@@
     (effects (font (size 1.27 1.27)) (justify left bottom))
   )
-  (label "BD0" (at 48.26 170.815 0)
+  (label "BD6" (at 48.26 170.815 0)
     (effects (font (size 1.27 1.27)) (justify left bottom))
   )
@@
     (effects (font (size 1.27 1.27)) (justify left bottom))
   )
-  (label "BD2" (at 48.26 168.275 0)
+  (label "BD4" (at 48.26 168.275 0)
     (effects (font (size 1.27 1.27)) (justify left bottom))
   )
@@
     (effects (font (size 1.27 1.27)) (justify right bottom))
   )
-  (label "BD4" (at 48.26 165.735 0)
+  (label "BD2" (at 48.26 165.735 0)
     (effects (font (size 1.27 1.27)) (justify left bottom))
   )
@@
     (effects (font (size 1.27 1.27)) (justify left bottom))
   )
-  (label "BD6" (at 48.26 163.195 0)
+  (label "BD0" (at 48.26 163.195 0)
     (effects (font (size 1.27 1.27)) (justify left bottom))
   )
@@
     (effects (font (size 1.27 1.27)) (justify right bottom))
   )
-  (label "BD7" (at 33.02 163.195 180)
+  (label "BD1" (at 33.02 163.195 180)
     (effects (font (size 1.27 1.27)) (justify right bottom))
   )
@@
     (effects (font (size 1.27 1.27)) (justify left bottom))
   )
+  (label "{AD[0..7] BD[0..7]}" (at 31.75 183.515 0)
+    (effects (font (size 1.27 1.27)) (justify left bottom))
+  )
   (label "D4" (at 247.65 97.155 0)
     (effects (font (size 1.27 1.27)) (justify left bottom))
@@
     (effects (font (size 1.27 1.27)) (justify right bottom))
   )
-  (label "BD3" (at 33.02 168.275 180)
+  (label "BD5" (at 33.02 168.275 180)
     (effects (font (size 1.27 1.27)) (justify right bottom))
   )
@@
       (effects (font (size 1.27 1.27)) hide)
     )
-    (property "Footprint" "Connector_PinHeader_2.54mm:PinHeader_2x13_P2.54mm_Vertical" (id 2) (at 41.91 155.575 0)
+    (property "Footprint" "pinhead:PinHeader_2x13_P2.54mm_Vertical_Top_Bottom" (id 2) (at 41.91 155.575 0)
       (effects (font (size 1.27 1.27)) hide)
     )
@@
     )
     (path "/36691a9d-d258-49ca-abae-4381b59c8f62"
-      (reference "J3") (unit 1) (value "Conn_02x13_Top_Bottom") (footprint "Connector_PinHeader_2.54mm:PinHeader_2x13_P2.54mm_Vertical")
+      (reference "J3") (unit 1) (value "Conn_02x13_Top_Bottom") (footprint "pinhead:PinHeader_2x13_P2.54mm_Vertical_Top_Bottom")
     )
     (path "/67b7940c-1d09-4328-a5d4-edbbeed320e7"

Commit message: 260110
Parts:
- L1, L2: footprint Inductor_THT:L_Axial_L20.0mm_D8.0mm_P25.40mm_Horizontal -> Inductor_THT:L_Axial_L14.5mm_D5.8mm_P20.32mm_Horizontal_Fastron_HBCC
Changed lines of the file:
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@@
       (effects (font (size 1.27 1.27)) hide)
     )
-    (property "Footprint" "Inductor_THT:L_Axial_L20.0mm_D8.0mm_P25.40mm_Horizontal" (id 2) (at 61.595 245.745 0)
+    (property "Footprint" "Inductor_THT:L_Axial_L14.5mm_D5.8mm_P20.32mm_Horizontal_Fastron_HBCC" (id 2) (at 61.595 245.745 0)
       (effects (font (size 1.27 1.27)) hide)
     )
@@
       (effects (font (size 1.27 1.27)) hide)
     )
-    (property "Footprint" "Inductor_THT:L_Axial_L20.0mm_D8.0mm_P25.40mm_Horizontal" (id 2) (at 61.595 253.365 0)
+    (property "Footprint" "Inductor_THT:L_Axial_L14.5mm_D5.8mm_P20.32mm_Horizontal_Fastron_HBCC" (id 2) (at 61.595 253.365 0)
       (effects (font (size 1.27 1.27)) hide)
     )
@@
     )
     (path "/6227f43c-3af3-4686-a986-632237f8f075"
-      (reference "L1") (unit 1) (value "L_Ferrite") (footprint "Inductor_THT:L_Axial_L20.0mm_D8.0mm_P25.40mm_Horizontal")
+      (reference "L1") (unit 1) (value "L_Ferrite") (footprint "Inductor_THT:L_Axial_L14.5mm_D5.8mm_P20.32mm_Horizontal_Fastron_HBCC")
     )
     (path "/691a884f-f531-48e1-a0a0-c3de6489163c"
-      (reference "L2") (unit 1) (value "L_Ferrite") (footprint "Inductor_THT:L_Axial_L20.0mm_D8.0mm_P25.40mm_Horizontal")
+      (reference "L2") (unit 1) (value "L_Ferrite") (footprint "Inductor_THT:L_Axial_L14.5mm_D5.8mm_P20.32mm_Horizontal_Fastron_HBCC")
     )
     (path "/2a72677a-1508-49cf-8394-19493c267036"
