File: _planning/pemx/pemx.kicad_pcb (KiCad board)
At the start: 2 copper layers, 79 parts, among them J1 Conn_01x03_Male, J2 Conn_01x06, J3 Conn_02x13_Top_Bottom, J4 Screw_Terminal_01x02, J5 Conn_01x03_Male, U1 74LS138, U10 74LS173, U11 74LS173, U12 27512, U13 27512, U14 27512, U15 27512, U16 27512, U17 27512, U18 27512, U19 27512, U2 74LS245, U3 74LS245, U4 DS1833, U5 74LS173, U6 74LS173, U7 74LS173, U8 74LS122, U9 74LS138

Commit message: 260110
Parts:
- J3: footprint Connector_PinHeader_2.54mm:PinHeader_2x13_P2.54mm_Vertical -> pinhead:PinHeader_2x13_P2.54mm_Vertical_Top_Bottom
- moved J4 452.3 mm to (-104.1, 118.7)
- moved C1 266.0 mm to (-98.4, 144.8)
- moved J5 246.9 mm to (108.0, 158.8), turned to 90 degrees
- moved C2 201.5 mm to (-48.8, 149.9)
- moved C4 189.4 mm to (78.7, 147.9), turned to 90 degrees
- moved C5 177.4 mm to (109.2, 147.9), turned to 90 degrees
- moved J2 161.0 mm to (-111.8, 138.6), turned to -90 degrees
- moved C3 156.4 mm to (78.7, 106.0), turned to 90 degrees
- moved C10 153.8 mm to (23.0, 125.4)
- moved C9 153.8 mm to (62.3, 95.1)
- moved R2 153.8 mm to (7.34, 93.8)
- moved R3 153.8 mm to (-4.21, 98.8)
- moved R4 153.8 mm to (6.57, 98.8)
- moved C11 153.8 mm to (50.2, 103.5)
- moved C12 153.8 mm to (42.1, 103.5)
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Connections:
- J3 pad 10: /BD6 -> /BD0
- J3 pad 11: /BD4 -> /BD2
- J3 pad 12: /BD2 -> /BD4
- J3 pad 13: /BD0 -> /BD6
- J3 pad 23: /BD7 -> /BD1
- J3 pad 24: /BD5 -> /BD3
- J3 pad 25: /BD3 -> /BD5
- J3 pad 26: /BD1 -> /BD7
Routing:
- net +5V: track 97.4 -> 267.1 mm
- net /CLK: track 0.00 -> 136.9 mm, vias 0 -> 2
- net /DA0: track 0.00 -> 135.7 mm, vias 0 -> 2
- net /DA1: track 0.00 -> 135.7 mm, vias 0 -> 2
- net /DA2: track 0.00 -> 134.4 mm, vias 0 -> 2
- net /DA3: track 0.00 -> 133.1 mm, vias 0 -> 2
- net /DM2: track 0.00 -> 36.4 mm
- net /DM1: track 0.00 -> 36.4 mm
- net /DM0: track 0.00 -> 36.4 mm
- net /D6: track 283.2 -> 317.9 mm
- net /D7: track 283.2 -> 316.0 mm
- net /A14.2: track 0.00 -> 29.6 mm, vias 0 -> 1
- net /A14.1: track 0.00 -> 28.8 mm, vias 0 -> 1
- net /A14.6: track 0.00 -> 27.1 mm, vias 0 -> 1
- net /A14.5: track 0.00 -> 27.1 mm, vias 0 -> 1
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Other:
- board outline added: 221.6 x 160 mm
- board text added: "JP13"
- board text added: "JP14"

Commit message: 260110
Parts:
- L1, L2: footprint Inductor_THT:L_Axial_L20.0mm_D8.0mm_P25.40mm_Horizontal -> Inductor_THT:L_Axial_L14.5mm_D5.8mm_P20.32mm_Horizontal_Fastron_HBCC
- moved R13 236.8 mm to (172.7, 239.4), turned to 90 degrees
- moved U4 227.4 mm to (169.3, 86.4), turned to 90 degrees
- moved R14 225.3 mm to (101.6, 239.4), turned to 90 degrees
- moved C20 225.0 mm to (168.9, 231.8), turned to -90 degrees
- moved C21 215.3 mm to (97.8, 231.8), turned to -90 degrees
- moved JP14 214.9 mm to (172.7, 222.9), turned to 0 degrees
- moved JP13 213.0 mm to (168.9, 222.9), turned to 0 degrees
- moved L1 203.7 mm to (72.4, 29.8)
- moved JP16 202.8 mm to (97.8, 222.9), turned to 0 degrees
- moved JP15 202.1 mm to (101.6, 222.9), turned to 0 degrees
- moved U18 201.3 mm to (154.9, 218.5), turned to -90 degrees
- moved U19 200.6 mm to (83.8, 218.5), turned to -90 degrees
- moved C2 196.6 mm to (106.0, 28.7), turned to -90 degrees
- moved C1 193.9 mm to (62.2, 36.2), turned to -90 degrees
- moved R11 190.8 mm to (172.7, 204.5), turned to 90 degrees
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Routing:
- net GNDD: track 147.3 -> 578.0 mm, vias 0 -> 1
- net +5V: track 267.1 -> 642.3 mm
- net /A0: track 283.7 -> 420.1 mm, vias 2 -> 3
- net /A1: track 283.7 -> 414.2 mm, vias 2 -> 3
- net /A15: track 0.00 -> 120.0 mm, vias 0 -> 2
- net /A14: track 0.00 -> 113.3 mm
- net /A2: track 283.7 -> 380.7 mm, vias 2 -> 3
- net /DS2: track 0.00 -> 86.5 mm, vias 0 -> 2
- net /DS1: track 0.00 -> 84.7 mm, vias 0 -> 2
- net /DS0: track 0.00 -> 83.6 mm, vias 0 -> 2
- net /DS3: track 0.00 -> 75.6 mm, vias 0 -> 1
- net /A8: track 283.7 -> 349.4 mm, vias 2 -> 3
- net /A9: track 283.7 -> 344.4 mm, vias 2 -> 3
- net /A3: track 283.7 -> 343.0 mm, vias 2 -> 3
- net /A13: track 283.7 -> 336.5 mm, vias 2 -> 3
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Other:
- board size 221.6 x 160 mm -> 150.5 x 219.1 mm

Commit message: 260111
Parts:
- moved R4 30.8 mm to (168.9, 39.4)
- moved U4 25.6 mm to (148.2, 71.8), turned to 180 degrees
- moved R6 23.3 mm to (130.2, 43.8)
- moved D1 19.1 mm to (136.5, 30.6), turned to 0 degrees
- moved R5 18.4 mm to (139.1, 43.8)
- moved R3 17.0 mm to (153.0, 44.5), turned to 180 degrees
- moved D2 16.5 mm to (127.7, 30.6)
- moved U8 15.0 mm to (160.7, 31.8), turned to -90 degrees
- moved C10 10.8 mm to (164.5, 34.3), turned to -90 degrees
- moved C9 10.5 mm to (158.1, 44.5), turned to 0 degrees
- moved C1 8.98 mm to (68.6, 29.9)
- moved C2 6.26 mm to (105.4, 34.9), turned to 90 degrees
- moved U13 0.16 mm to (83.8, 114.8)
Routing:
- net GNDD: track 578.0 -> 1491.9 mm, vias 1 -> 2
- net +5V: track 642.3 -> 1300.1 mm, vias 0 -> 1
- net /-CS7: track 0.00 -> 333.5 mm, vias 0 -> 3
- net /A15: track 120.0 -> 421.3 mm, vias 2 -> 17
- net /-CS6: track 0.00 -> 291.0 mm, vias 0 -> 4
- net /-CS3: track 0.00 -> 277.2 mm, vias 0 -> 1
- net /-CS5: track 0.00 -> 261.8 mm, vias 0 -> 4
- net /-CS2: track 0.00 -> 241.4 mm, vias 0 -> 2
- net /A14: track 113.3 -> 352.9 mm, vias 0 -> 3
- net /-CS4: track 0.00 -> 231.4 mm, vias 0 -> 4
- net /-CS1: track 0.00 -> 207.2 mm, vias 0 -> 2
- net /-OE: track 283.7 -> 487.5 mm, vias 2 -> 3
- net /-CS0: track 0.00 -> 172.9 mm, vias 0 -> 2
- net /-E4: track 0.00 -> 106.6 mm, vias 0 -> 1
- net /RST: track 0.00 -> 93.1 mm
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Other:
- board text removed: "JP13"
- board text removed: "JP14"
