File: hardware/PEMX External memory box/pemx/pemx.kicad_pcb (KiCad board)
At the start: 2 copper layers, 150.5 x 219.1 mm, 79 parts, among them J1 Conn_01x03_Male, J2 Conn_01x06, J3 Conn_02x13_Top_Bottom, J4 Screw_Terminal_01x02, J5 Conn_01x03_Male, U1 74LS138, U10 74LS173, U11 74LS173, U12 27512, U13 27512, U14 27512, U15 27512, U16 27512, U17 27512, U18 27512, U19 27512, U2 74LS245, U3 74LS245, U4 DS1833, U5 74LS173, U6 74LS173, U7 74LS173, U8 74LS122, U9 74LS138

Commit message: 260111
Parts:
- added REF**: MountingHole_3.5mm_Pad, MountingHole:MountingHole_3.5mm_Pad, F.Cu at (117.1, 33.0)
- added REF**: MountingHole_3.5mm_Pad, MountingHole:MountingHole_3.5mm_Pad, F.Cu at (110.5, 237.0)
- added REF**: MountingHole_3.5mm_Pad, MountingHole:MountingHole_3.5mm_Pad, F.Cu at (38.1, 105.7)
- added REF**: MountingHole_3.5mm_Pad, MountingHole:MountingHole_3.5mm_Pad, F.Cu at (111.3, 122.4)
- added REF**: MountingHole_3.5mm_Pad, MountingHole:MountingHole_3.5mm_Pad, F.Cu at (170.7, 144.5)
- added REF**: MountingHole_3.5mm_Pad, MountingHole:MountingHole_3.5mm_Pad, F.Cu at (170.7, 211.8)
- added REF**: MountingHole_3.5mm_Pad, MountingHole:MountingHole_3.5mm_Pad, F.Cu at (38.1, 237.0)
- added REF**: MountingHole_3.5mm_Pad, MountingHole:MountingHole_3.5mm_Pad, F.Cu at (35.6, 43.7)
- added REF**: MountingHole_3.5mm_Pad, MountingHole:MountingHole_3.5mm_Pad, F.Cu at (38.1, 173.7)
- added REF**: MountingHole_3.5mm_Pad, MountingHole:MountingHole_3.5mm_Pad, F.Cu at (174.2, 33.0)
- added REF**: MountingHole_3.5mm_Pad, MountingHole:MountingHole_3.5mm_Pad, F.Cu at (110.5, 190.8)
- moved R1 7.40 mm to (42.9, 40.9), turned to -90 degrees
Routing:
- net +5V: track 1300.1 -> 1289.9 mm
- net Net-(R1-Pad2): track 4.46 -> 9.03 mm
- net /A6: track 339.2 -> 340.7 mm
- net /A15: track 421.3 -> 420.4 mm
Other:
- board text added: "2026 Pozsar Zsolt Zacchaeus Microcomputer"
- board text added: "BANK #0"
- board text added: "BANK #1"
- board text added: "BANK #2"
- board text added: "BANK #3"
- board text added: "BANK #4"
- board text added: "BANK #5"
- board text added: "BANK #6"
- board text added: "BANK #7"
- board text added: "PEMX - External memory box"
- board text added: "PIO/2"
- board text added: "POWER"
- board text added: "POWER LED"
- board text added: "POWER SW"
- board text added: "READ LED"
