File: hardware/PEIX External interface box/ebe-266-1/ebe-266-1/ebe-266-1.kicad_sch (KiCad schematic)
At the start: 32 parts, among them SW1 SW_DIP_x08, U1 74ALS688, U2 74ALS240, U3 74ALS32, U4 74HC259, U5 74HC259

Commit message: 260119
Connections:
- net +5V: no longer C?.2, C?.2, C?.2, C?.2, C?.2, C?.2, C?.2, C?.2, D?.2 (A), R?.1, SW1.1, SW1.2, SW1.3, SW1.4, SW1.5, SW1.6, SW1.7, SW1.8, U1.10 (GND), U1.11 (P4), U1.12 (R4), U1.8 (P3), U1.9 (R3), U2.1 (OEa), U2.10 (GND), U2.19 (OEb), U4.8 (GND), U5.8 (GND)
- new net GNDD: C?.2, C?.2, C?.2, C?.2, C?.2, C?.2, C?.2, C?.2, D?.2 (A), R?.1, SW1.1, SW1.2, SW1.3, SW1.4, SW1.5, SW1.6, SW1.7, SW1.8, U1.10 (GND), U1.11 (P4), U1.12 (R4), U1.8 (P3), U1.9 (R3), U2.1 (OEa), U2.10 (GND), U2.19 (OEb), U4.8 (GND), U5.8 (GND)
Changed lines of the file:
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@@
     (effects (font (size 1.27 1.27) italic) (justify left bottom))
   )
-  (label "GND" (at 68.58 97.79 0)
+  (label "GND" (at 68.58 95.25 0)
     (effects (font (size 1.27 1.27) italic) (justify left bottom))
   )
-  (label "+5V" (at 68.58 95.25 0)
+  (label "+5V" (at 68.58 97.79 0)
     (effects (font (size 1.27 1.27) italic) (justify left bottom))
   )
