File: hardware/PEIX External interface box/ebe_206-1/ebe_206-1/ebe_206-1.kicad_sch (KiCad schematic)
At the start: 26 parts, among them SW1 SW_DIP_x08, U1 74ALS688, U2 74LS244, U3 7400, U4 74ALS251, U5 74ALS251

Commit message: 260124
Connections:
- net D0 is gone; now on net 12a: U2.9 (O0b)
Other:
- title: Integrated circuits important for control -> Control-related circuits
Changed lines of the file:
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@@
   (paper "A4")
   (title_block
-    (title "Integrated circuits important for control")
+    (title "Control-related circuits")
     (date "2026-01-19")
     (rev "1.0")
     (company "Pozsar Zsolt")
-    (comment 1 "EBE-206.1 digital input module")
+    (comment 1 "EBE 206.1 digital input module")
   )
   (junction (at 245.11 101.6) (diameter 0) (color 0 0 0 0)
@@
     (stroke (width 0) (type default) (color 0 0 0 0))
   )
-  (wire (pts (xy 54.61 106.68) (xy 72.39 106.68))
+  (wire (pts (xy 53.34 106.68) (xy 72.39 106.68))
     (stroke (width 0) (type default) (color 0 0 0 0))
   )
@@
   )
   (text "Reconstructed functional schematic (reverse engineered for interoperability)."
-    (at 166.37 43.18 0)
+    (at 196.85 163.83 0)
     (effects (font (size 1.27 1.27) italic) (justify left bottom))
   )
@@
     (effects (font (size 1.27 1.27) italic) (justify left bottom))
   )
-  (label "D0" (at 54.61 106.68 0)
+  (label "DI" (at 54.61 106.68 0)
     (effects (font (size 1.27 1.27) italic) (justify left bottom))
   )
