File: hardware/PEIX External interface box/ebe_266-1/ebe_266-1/ebe_266-1.kicad_sch (KiCad schematic)
At the start: 32 parts, among them SW1 SW_DIP_x08, U1 74ALS688, U2 74ALS240, U3 74ALS32, U4 74HC259, U5 74HC259

Commit message: 260124
Other:
- title: Integrated circuits important for control -> Control-related circuits
Changed lines of the file:
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@@
   (paper "A4")
   (title_block
-    (title "Integrated circuits important for control")
+    (title "Control-related circuits")
     (date "2026-01-18")
     (rev "1.0")
     (company "Pozsar Zsolt")
-    (comment 1 "EBE-266.1 digital output module")
+    (comment 1 "EBE 266.1 digital output module")
   )
   (junction (at 185.42 128.27) (diameter 0) (color 0 0 0 0)
@@
   )
   (text "Reconstructed functional schematic (reverse engineered for interoperability)."
-    (at 144.78 35.56 0)
+    (at 196.85 163.83 0)
     (effects (font (size 1.27 1.27) italic) (justify left bottom))
   )
@@
     (effects (font (size 1.27 1.27) italic) (justify left bottom))
   )
-  (label "D0" (at 68.58 100.33 0)
+  (label "DO" (at 68.58 100.33 0)
     (effects (font (size 1.27 1.27) italic) (justify left bottom))
   )
