File: hardware/PEIX External interface box/ebe_287-1/ebe_287-1/analog.kicad_sch (KiCad schematic)
At the start: 1 part

Commit message: 260125
Changed lines of the file:
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@@
     (effects (font (size 1.27 1.27)) (justify right))
   )
-  (hierarchical_label "(01) UPD" (shape input) (at 76.2 82.55 180)
+  (hierarchical_label "(01) {slash}UPD" (shape input) (at 76.2 82.55 180)
     (effects (font (size 1.27 1.27)) (justify right))
   )
