File: hardware/PEIX External interface box/ebe_287-1/ebe_287-1/ebe_287-1.kicad_sch (KiCad schematic)
At the start: 12 parts, among them U1 74LS245, U10 74LS04, U11 74LS74, U12 74ALS876, U13 74ALS876, U14 74LS139, U2 74LS245, U3 74ALS688, U5 74LS273

Commit message: 260124
Parts:
- gave numbers to parts that had none: 1
Changed lines of the file:
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@@
   (symbol (lib_id "74xx:74LS244") (at 106.045 51.435 0) (unit 1)
     (in_bom yes) (on_board yes)
-    (property "Reference" "U?" (id 0) (at 98.425 34.925 0)
+    (property "Reference" "U9" (id 0) (at 98.425 34.925 0)
       (effects (font (size 1.27 1.27)) (justify left))
     )
@@
       (reference "#PWR?") (unit 1) (value "GNDD") (footprint "")
     )
+    (path "/64b0b3dc-876d-421d-9807-51baf112f6e7/16767644-d139-4c76-8b79-c013d3b78bbf/3ad7327e-d8eb-46ce-ad29-6c826bff655a"
+      (reference "#PWR?") (unit 1) (value "GNDD") (footprint "")
+    )
     (path "/64b0b3dc-876d-421d-9807-51baf112f6e7/d0984119-8bf2-4d32-b301-49786a85755b/3ad7327e-d8eb-46ce-ad29-6c826bff655a"
-      (reference "#PWR?") (unit 1) (value "GNDD") (footprint "")
-    )
-    (path "/64b0b3dc-876d-421d-9807-51baf112f6e7/16767644-d139-4c76-8b79-c013d3b78bbf/3ad7327e-d8eb-46ce-ad29-6c826bff655a"
       (reference "#PWR?") (unit 1) (value "GNDD") (footprint "")
     )
@@
       (reference "Q?") (unit 1) (value "Q_NPN_CBE") (footprint "")
     )
+    (path "/64b0b3dc-876d-421d-9807-51baf112f6e7/16767644-d139-4c76-8b79-c013d3b78bbf/15e8d336-ff33-4878-bb49-1ece76f7f5bb"
+      (reference "R?") (unit 1) (value "R") (footprint "")
+    )
     (path "/64b0b3dc-876d-421d-9807-51baf112f6e7/d0984119-8bf2-4d32-b301-49786a85755b/15e8d336-ff33-4878-bb49-1ece76f7f5bb"
       (reference "R?") (unit 1) (value "R") (footprint "")
     )
-    (path "/64b0b3dc-876d-421d-9807-51baf112f6e7/16767644-d139-4c76-8b79-c013d3b78bbf/15e8d336-ff33-4878-bb49-1ece76f7f5bb"
-      (reference "R?") (unit 1) (value "R") (footprint "")
-    )
     (path "/64b0b3dc-876d-421d-9807-51baf112f6e7/d0984119-8bf2-4d32-b301-49786a85755b/3d77921d-73ff-48d1-bc43-aa2f89794c45"
       (reference "R?") (unit 1) (value "R") (footprint "")
@@
       (reference "U5") (unit 1) (value "74LS273") (footprint "")
     )
+    (path "/97e0f46f-bb8c-4970-b477-38082464e54e"
+      (reference "U9") (unit 1) (value "74LS244") (footprint "")
+    )
     (path "/873a7b2f-a86e-4810-b6f7-f0284644b5f2"
       (reference "U10") (unit 1) (value "74LS04") (footprint "")
@@
       (reference "U14") (unit 2) (value "74LS139") (footprint "")
     )
-    (path "/97e0f46f-bb8c-4970-b477-38082464e54e"
-      (reference "U?") (unit 1) (value "74LS244") (footprint "")
-    )
     (path "/64b0b3dc-876d-421d-9807-51baf112f6e7/d0984119-8bf2-4d32-b301-49786a85755b/da6d998c-22d9-44b8-b9a6-6c04accd3f5f"

Commit message: 260125
Parts:
- removed U10: 74LS04, symbol 74xx:74LS04
- removed U11: 74LS74, symbol 74xx:74LS74
- removed U13: 74ALS876, MODULE, symbol dil:DIL24
- removed U14: 74LS139, symbol 74xx:74LS139
- added R?: R, symbol Device:R
- added U12: 74ALS876, MODULE, symbol dil:DIL24
- renumbered U12 to U11
Connections:
- net +5V: now also R?.1, U12.24
- net GNDD: now also U12.12
- net at U5.1 (~{Mr}): now also U11.1, U11.13, U12.1, U12.13
- net at U2.2 (A0), U5.3 (D0): now also U11.3, U11.7, U12.7
- net at U2.3 (A1), U5.4 (D1): now also U11.4, U11.8, U12.8
- net at U2.4 (A2), U5.7 (D2): now also U11.5, U11.9, U12.9
- net at U2.5 (A3), U5.8 (D3): now also U11.10, U11.6, U12.10
Other:
- sheet Analog board ports: added (01) /UPD; removed (01) UPD
- note added: "1/OC7/4 1/OC6/4"
- note added: "3/OC1/6 2/OC1/7 3/OC2/6 2/OC2/7 3/OC3/6 2/OC3/7 3/OC4/6 2/OC4/7 3/OC5/6 2/OC5/7"
- note added: "optocouplers"
- moved on the sheet: U1, U11, U2, U3, U5, U9
