File: hardware/PFRP Front panel/pfrp/pfrp.kicad_sch (KiCad schematic)
At the start: 74 parts, among them J1 AudioJack2_Ground, J10 Conn_01x01_Female, J11 Conn_01x01_Female, J12 Conn_01x01_Female, J13 Conn_01x01_Female, J14 Conn_01x01_Female, J15 Conn_01x01_Female, J16 Conn_01x01_Female, J17 Conn_01x01_Female, J18 Conn_01x01_Female, J19 Conn_01x01_Female, J2 DIN-5_180degree, J20 Conn_01x01_Female, J21 Conn_01x01_Female, J22 Conn_01x01_Female, J23 Conn_01x01_Female, J24 Conn_01x01_Female, J25 Conn_01x01_Female, J26 Conn_01x01_Female, J27 Conn_01x01_Female, J28 Conn_01x01_Female, J29 Conn_01x01_Female, J3 Conn_01x01_Female, J30 Conn_01x01_Female, J31 Conn_01x01_Female, J32 Conn_01x01_Female, J33 Conn_01x01_Female, J34 Conn_01x01_Female, J35 Conn_01x01_Female, J36 Conn_01x01_Female, J37 Conn_01x01_Female, J38 Conn_01x01_Female, J39 Conn_01x01_Female, J4 Conn_01x01_Female, J40 Conn_01x01_Female, J41 Conn_01x01_Female, J42 Conn_01x01_Female, J5 Conn_01x01_Female, J6 Conn_01x01_Female, J7 Conn_01x01_Female, J8 Conn_01x01_Female, J9 Conn_01x01_Female, P1 470kA, SW1 SW_SPDT, SW10 SW_Push, SW3 SW_Push, SW3 SW_SPDT, SW4 SW_Push, SW4 SW_SPDT, SW5 SW_Push, SW5 SW_SPDT, SW6 SW_Push, SW6 SW_SPDT, SW7 SW_Push, SW7 SW_SPDT, SW8 SW_Push, SW9 SW_Push

Commit message: 251205
Connections:
- net PBP/F1/2 renamed PBKP/F1/2
- net PBP/F2/2 renamed PBKP/F2/2
- net PBP/F3/2 renamed PBKP/F3/2
- net PBP/F4/2 renamed PBKP/F4/2
- net PBP/F5/2 renamed PBKP/F5/2
Changed lines of the file:
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@@
     (stroke (width 0) (type default) (color 0 0 0 0))
   )
-  (wire (pts (xy 218.44 39.37) (xy 226.06 39.37))
+  (wire (pts (xy 218.44 39.37) (xy 224.79 39.37))
     (stroke (width 0) (type default) (color 0 0 0 0))
   )
@@
     (stroke (width 0) (type default) (color 0 0 0 0))
   )
-  (wire (pts (xy 218.44 25.4) (xy 226.06 25.4))
+  (wire (pts (xy 218.44 25.4) (xy 224.79 25.4))
     (stroke (width 0) (type default) (color 0 0 0 0))
   )
@@
     (stroke (width 0) (type default) (color 0 0 0 0))
   )
-  (wire (pts (xy 226.06 81.28) (xy 218.44 81.28))
+  (wire (pts (xy 224.79 81.28) (xy 218.44 81.28))
     (stroke (width 0) (type default) (color 0 0 0 0))
   )
@@
     (stroke (width 0) (type default) (color 0 0 0 0))
   )
-  (wire (pts (xy 218.44 67.31) (xy 226.06 67.31))
+  (wire (pts (xy 218.44 67.31) (xy 224.79 67.31))
     (stroke (width 0) (type default) (color 0 0 0 0))
   )
@@
     (stroke (width 0) (type default) (color 0 0 0 0))
   )
-  (wire (pts (xy 218.44 53.34) (xy 226.06 53.34))
+  (wire (pts (xy 218.44 53.34) (xy 224.79 53.34))
     (stroke (width 0) (type default) (color 0 0 0 0))
   )
@@
     )
   )
-  (global_label "PBP{slash}F5{slash}2" (shape input) (at 226.06 81.28 0) (fields_autoplaced)
+  (global_label "PBKP{slash}F5{slash}2" (shape input) (at 224.79 81.28 0) (fields_autoplaced)
     (effects (font (size 1.27 1.27)) (justify left))
     (property "Intersheet References" "${INTERSHEET_REFS}" (id 0) (at 238.4517 81.2006 0)
@@
     )
   )
-  (global_label "PBP{slash}F4{slash}2" (shape input) (at 226.06 67.31 0) (fields_autoplaced)
+  (global_label "PBKP{slash}F4{slash}2" (shape input) (at 224.79 67.31 0) (fields_autoplaced)
     (effects (font (size 1.27 1.27)) (justify left))
     (property "Intersheet References" "${INTERSHEET_REFS}" (id 0) (at 238.4517 67.2306 0)
@@
     )
   )
-  (global_label "PBP{slash}F3{slash}2" (shape input) (at 226.06 53.34 0) (fields_autoplaced)
+  (global_label "PBKP{slash}F3{slash}2" (shape input) (at 224.79 53.34 0) (fields_autoplaced)
     (effects (font (size 1.27 1.27)) (justify left))
     (property "Intersheet References" "${INTERSHEET_REFS}" (id 0) (at 238.4517 53.2606 0)
@@
     )
   )
-  (global_label "PBP{slash}F2{slash}2" (shape input) (at 226.06 39.37 0) (fields_autoplaced)
+  (global_label "PBKP{slash}F2{slash}2" (shape input) (at 224.79 39.37 0) (fields_autoplaced)
     (effects (font (size 1.27 1.27)) (justify left))
     (property "Intersheet References" "${INTERSHEET_REFS}" (id 0) (at 238.4517 39.2906 0)
@@
     )
   )
-  (global_label "PBP{slash}F1{slash}2" (shape input) (at 226.06 25.4 0) (fields_autoplaced)
+  (global_label "PBKP{slash}F1{slash}2" (shape input) (at 224.79 25.4 0) (fields_autoplaced)
     (effects (font (size 1.27 1.27)) (justify left))
     (property "Intersheet References" "${INTERSHEET_REFS}" (id 0) (at 238.4517 25.3206 0)

Commit message: 260115
Connections:
- net MM8D/J10/1 renamed PIOI/J10/1
- net MM8D/J10/2 renamed PIOI/J10/2
- net MM8D/J10/3 renamed PIOI/J10/3
- net MM8D/J10/4 renamed PIOI/J10/4
- net MM8D/J10/5 renamed PIOI/J10/5
- net MM8D/J1/1 renamed PIOI/J1/1
- net MM8D/J1/2 renamed PIOI/J1/2
- net MM8D/J1/3 renamed PIOI/J1/3
- net MM8D/J1/4 renamed PIOI/J1/4
- net MM8D/J1/5 renamed PIOI/J1/5
- net MM8D/J6/1 renamed PIOI/J6/1
- net MM8D/J6/2 renamed PIOI/J6/2
- net MM8D/J6/3 renamed PIOI/J6/3
- net MM8D/J7/1 renamed PIOI/J7/1
- net MM8D/J7/2 renamed PIOI/J7/2
- net MM8D/J7/3 renamed PIOI/J7/3
- net MM8D/J8/1 renamed PIOI/J8/1
- net MM8D/J8/2 renamed PIOI/J8/2
- net MM8D/J8/3 renamed PIOI/J8/3
- net MM8D/J9/1 renamed PIOI/J9/1
- net MM8D/J9/2 renamed PIOI/J9/2
- net MM8D/J9/3 renamed PIOI/J9/3
- net PCOX/Jx/1 renamed PCOX/J5/1
- net PCOX/Jx/2 renamed PCOX/J5/2
- net PCOX/Jy/1 renamed PCOX/J3/1
- net PCOX/Jy/2 renamed PCOX/J3/2

Commit message: 260128
Connections:
- net PCAS/Jx/1 renamed PTAP/J2/1
- net PCAS/Jx/2 renamed PTAP/J2/2
- net PCAS/Jx/3 renamed PTAP/J2/3
- net PCAS/Jx/4 renamed PTAP/J2/4
- net PCAS/Jx/5 renamed PTAP/J2/5
- net PCAS/Jy/1 renamed PTAP/J3/1
- net PCAS/Jy/2 renamed PTAP/J3/2
- net PCAS/Jy/3 renamed PTAP/J4/1
- net PCAS/Jy/4 renamed PTAP/J4/2
- net PCAS/Jy/5 renamed PTAP/J5/1
- net PCAS/Jy/6 renamed PTAP/J5/2
Other:
- note added: "DIN"
- note added: "DOUT"
- note added: "MLED"
- note added: "REL"
- note added: "RLED"
- note added: "WLED"
- note removed: "data in"
- note removed: "data out"
- note removed: "motor on"
- note removed: "motor relay"
- note removed: "read"
- note removed: "write"
Changed lines of the file:
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@@
     (effects (font (size 1.27 1.27)) (justify left bottom))
   )
-  (text "read" (at 78.74 120.015 180)
-    (effects (font (size 1.27 1.27) italic) (justify right bottom))
-  )
-  (text "motor on" (at 78.74 132.715 180)
+  (text "RLED" (at 78.74 120.015 180)
+    (effects (font (size 1.27 1.27) italic) (justify right bottom))
+  )
+  (text "MLED" (at 78.74 132.715 180)
     (effects (font (size 1.27 1.27) italic) (justify right bottom))
   )
@@
     (effects (font (size 1.27 1.27) italic) (justify right bottom))
   )
-  (text "motor relay" (at 78.74 88.265 180)
+  (text "REL" (at 78.74 88.265 180)
     (effects (font (size 1.27 1.27) italic) (justify right bottom))
   )
@@
     (effects (font (size 1.27 1.27) italic) (justify left bottom))
   )
-  (text "write" (at 78.74 126.365 180)
+  (text "WLED" (at 78.74 126.365 180)
     (effects (font (size 1.27 1.27) italic) (justify right bottom))
   )
@@
     (effects (font (size 1.27 1.27)) (justify left bottom))
   )
-  (text "data out" (at 78.74 107.315 180)
+  (text "DOUT" (at 78.74 107.315 180)
     (effects (font (size 1.27 1.27) italic) (justify right bottom))
   )
@@
     (effects (font (size 1.27 1.27)) (justify left bottom))
   )
-  (text "data in" (at 78.74 94.615 180)
+  (text "DIN" (at 78.74 94.615 180)
     (effects (font (size 1.27 1.27) italic) (justify right bottom))
   )
@@
     (effects (font (size 1.27 1.27)) (justify left bottom))
   )
-  (text "motor relay" (at 78.74 113.665 180)
+  (text "REL" (at 78.74 113.665 180)
     (effects (font (size 1.27 1.27) italic) (justify right bottom))
   )
@@
     (effects (font (size 1.27 1.27)) (justify left bottom))
   )
-  (global_label "PCAS{slash}Jx{slash}2" (shape input) (at 66.04 90.805 0) (fields_autoplaced)
-    (effects (font (size 1.27 1.27)) (justify left))
-    (property "Intersheet References" "${INTERSHEET_REFS}" (id 0) (at 79.1574 90.7256 0)
+  (global_label "PTAP{slash}J2{slash}2" (shape input) (at 66.04 90.805 0) (fields_autoplaced)
+    (effects (font (size 1.27 1.27)) (justify left))
+    (property "Intersheet References" "${INTERSHEET_REFS}" (id 0) (at 79.0969 90.7256 0)
       (effects (font (size 1.27 1.27)) (justify left) hide)
     )
@@
     )
   )
-  (global_label "PCAS{slash}Jx{slash}3" (shape input) (at 66.04 97.155 0) (fields_autoplaced)
-    (effects (font (size 1.27 1.27)) (justify left))
-    (property "Intersheet References" "${INTERSHEET_REFS}" (id 0) (at 79.1574 97.0756 0)
+  (global_label "PTAP{slash}J2{slash}3" (shape input) (at 66.04 97.155 0) (fields_autoplaced)
+    (effects (font (size 1.27 1.27)) (justify left))
+    (property "Intersheet References" "${INTERSHEET_REFS}" (id 0) (at 79.0969 97.0756 0)
       (effects (font (size 1.27 1.27)) (justify left) hide)
     )
@@
     )
   )
-  (global_label "PCAS{slash}Jx{slash}4" (shape input) (at 66.04 103.505 0) (fields_autoplaced)
-    (effects (font (size 1.27 1.27)) (justify left))
-    (property "Intersheet References" "${INTERSHEET_REFS}" (id 0) (at 79.1574 103.4256 0)
+  (global_label "PTAP{slash}J2{slash}4" (shape input) (at 66.04 103.505 0) (fields_autoplaced)
+    (effects (font (size 1.27 1.27)) (justify left))
+    (property "Intersheet References" "${INTERSHEET_REFS}" (id 0) (at 79.0969 103.4256 0)
       (effects (font (size 1.27 1.27)) (justify left) hide)
     )
@@
     )
   )
-  (global_label "PCAS{slash}Jy{slash}4" (shape input) (at 66.04 122.555 0) (fields_autoplaced)
+  (global_label "PTAP{slash}J4{slash}2" (shape input) (at 66.04 122.555 0) (fields_autoplaced)
     (effects (font (size 1.27 1.27)) (justify left))
     (property "Intersheet References" "${INTERSHEET_REFS}" (id 0) (at 79.0969 122.4756 0)
@@
     )
   )
-  (global_label "PCAS{slash}Jy{slash}3" (shape input) (at 35.56 122.555 180) (fields_autoplaced)
+  (global_label "PTAP{slash}J4{slash}1" (shape input) (at 35.56 122.555 180) (fields_autoplaced)
     (effects (font (size 1.27 1.27)) (justify right))
     (property "Intersheet References" "${INTERSHEET_REFS}" (id 0) (at 22.5031 122.4756 0)
@@
     )
   )
-  (global_label "PCAS{slash}Jy{slash}5" (shape input) (at 35.56 128.905 180) (fields_autoplaced)
+  (global_label "PTAP{slash}J5{slash}1" (shape input) (at 35.56 128.905 180) (fields_autoplaced)
     (effects (font (size 1.27 1.27)) (justify right))
     (property "Intersheet References" "${INTERSHEET_REFS}" (id 0) (at 22.5031 128.8256 0)
@@
     )
   )
-  (global_label "PCAS{slash}Jx{slash}5" (shape input) (at 66.04 109.855 0) (fields_autoplaced)
-    (effects (font (size 1.27 1.27)) (justify left))
-    (property "Intersheet References" "${INTERSHEET_REFS}" (id 0) (at 79.1574 109.7756 0)
+  (global_label "PTAP{slash}J2{slash}5" (shape input) (at 66.04 109.855 0) (fields_autoplaced)
+    (effects (font (size 1.27 1.27)) (justify left))
+    (property "Intersheet References" "${INTERSHEET_REFS}" (id 0) (at 79.0969 109.7756 0)
       (effects (font (size 1.27 1.27)) (justify left) hide)
     )
@@
     )
   )
-  (global_label "PCAS{slash}Jy{slash}2" (shape input) (at 66.04 116.205 0) (fields_autoplaced)
+  (global_label "PTAP{slash}J3{slash}2" (shape input) (at 66.04 116.205 0) (fields_autoplaced)
     (effects (font (size 1.27 1.27)) (justify left))
     (property "Intersheet References" "${INTERSHEET_REFS}" (id 0) (at 79.0969 116.1256 0)
@@
     )
   )
-  (global_label "PCAS{slash}Jx{slash}1" (shape input) (at 66.04 84.455 0) (fields_autoplaced)
-    (effects (font (size 1.27 1.27)) (justify left))
-    (property "Intersheet References" "${INTERSHEET_REFS}" (id 0) (at 79.1574 84.3756 0)
+  (global_label "PTAP{slash}J2{slash}1" (shape input) (at 66.04 84.455 0) (fields_autoplaced)
+    (effects (font (size 1.27 1.27)) (justify left))
+    (property "Intersheet References" "${INTERSHEET_REFS}" (id 0) (at 79.0969 84.3756 0)
       (effects (font (size 1.27 1.27)) (justify left) hide)
     )
@@
     )
   )
-  (global_label "PCAS{slash}Jy{slash}6" (shape input) (at 66.04 128.905 0) (fields_autoplaced)
+  (global_label "PTAP{slash}J5{slash}2" (shape input) (at 66.04 128.905 0) (fields_autoplaced)
     (effects (font (size 1.27 1.27)) (justify left))
     (property "Intersheet References" "${INTERSHEET_REFS}" (id 0) (at 79.0969 128.8256 0)
@@
     )
   )
-  (global_label "PCAS{slash}Jy{slash}1" (shape input) (at 35.56 116.205 180) (fields_autoplaced)
+  (global_label "PTAP{slash}J3{slash}1" (shape input) (at 35.56 116.205 180) (fields_autoplaced)
     (effects (font (size 1.27 1.27)) (justify right))
     (property "Intersheet References" "${INTERSHEET_REFS}" (id 0) (at 22.5031 116.1256 0)
