File: PEIX External interface box/hardware/peix/peix.kicad_pcb (KiCad board)
At the start: 2 copper layers, 160 x 100.3 mm, 885 parts, among them J1 Conn_01x08_Male, J2 Conn_01x03_Male, J3 Conn_01x04_Male, J4 Conn_01x08_Male, J5 Conn_01x08_Male, J6 Conn_01x08_Male, J7 DB9_Female_MountingHoles, J8 DIN41612_02x16_AC_EvenPins, U1 87C51, U2 27C64, U3 74LS573, U4 74LS08, U5 MAX232, U6 74LS245, U7 74LS245, U8 74LS245, Y1 11.0592 MHz

Commit message: 260215
Parts:
- removed ? (x839): , 
- J4, J5: value Conn_01x08_Male -> locked
- J8: value DIN41612_02x16_AC_EvenPins -> locked
- R1, R2, R3, R4, R5, R6, R7, R8: footprint Resistor_THT:R_Axial_DIN0207_L6.3mm_D2.5mm_P5.08mm_Vertical -> Resistor_THT:R_Axial_DIN0207_L6.3mm_D2.5mm_P2.54mm_Vertical
- moved JP1 175.3 mm to (176.3, 135.1), turned to 180 degrees
- moved C12 152.0 mm to (216.2, 51.5), turned to 90 degrees
- moved J2 142.5 mm to (158.8, 125.7), turned to 90 degrees
- moved R1 116.6 mm to (126.7, 128.5)
- moved C6 113.9 mm to (126.7, 136.1)
- moved C11 105.1 mm to (165.4, 93.4), turned to 90 degrees
- moved C5 94.4 mm to (96.3, 129.8), turned to -90 degrees
- moved C3 94.1 mm to (184.4, 135.3), turned to 90 degrees
- moved C4 92.3 mm to (180.6, 135.3), turned to 90 degrees
- moved J1 82.1 mm to (137.2, 125.7), turned to 90 degrees
- moved Y1 80.9 mm to (180.6, 126.7), turned to 0 degrees
- moved J3 77.8 mm to (167.6, 125.7), turned to 90 degrees
- moved U1 75.2 mm to (138.7, 120.7), turned to 90 degrees
- moved R8 70.6 mm to (195.6, 92.0), turned to 90 degrees
- moved C9 66.8 mm to (134.6, 88.7), turned to -90 degrees
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Connections:
- D1 pad 2: Net-(D1-Pad2) -> +5V
- D2 pad 2: Net-(D2-Pad2) -> +5V
- D3 pad 2: Net-(D3-Pad2) -> +5V
- J7 pad 0: GNDD -> Earth
- J8 pad c2: unconnected-(J8-Padc2) -> GNDD
- J8 pad c4: unconnected-(J8-Padc4) -> +5V
- JP2 pad 1: Net-(J2-Pad3) -> Net-(J2-Pad1)
- R4 pad 1: Net-(D1-Pad2) -> Net-(U4-Pad3)
- R4 pad 2: +5V -> Net-(D1-Pad1)
- R5 pad 1: +5V -> Net-(D2-Pad1)
- R5 pad 2: Net-(D2-Pad2) -> Net-(U4-Pad6)
- R6 pad 1: Net-(D3-Pad2) -> Net-(U4-Pad8)
- R6 pad 2: +5V -> Net-(D3-Pad1)
- U1 pad 26: Net-(J2-Pad1) -> Net-(J2-Pad3)
- U1 pad 28: Net-(J2-Pad3) -> Net-(J2-Pad1)
- U4 pad 1: /-RD -> Net-(JP2-Pad2)
- U4 pad 10: Net-(U1-Pad10) -> Net-(U1-Pad11)
- U4 pad 11: Net-(D3-Pad1) -> Net-(U4-Pad11)
- U4 pad 12: Net-(U1-Pad11) -> /-RD
- U4 pad 13: Net-(U1-Pad11) -> /-WR
- U4 pad 2: /-WR -> Net-(JP2-Pad2)
- U4 pad 4: Net-(JP2-Pad2) -> Net-(U1-Pad10)
- U4 pad 5: Net-(JP2-Pad2) -> Net-(U1-Pad10)
- U4 pad 6: Net-(D1-Pad1) -> Net-(U4-Pad6)
- U4 pad 8: Net-(D2-Pad1) -> Net-(U4-Pad8)
- U4 pad 9: Net-(U1-Pad10) -> Net-(U1-Pad11)
- U6 pad 19: Net-(U4-Pad3) -> Net-(U4-Pad11)
- U8 pad 11: /-RD -> /-WR
- U8 pad 12: /-WR -> /-RD
Routing:
- net /A12: track 7.61 -> 110.5 mm, vias 0 -> 2
- net /-PSEN: track 0.00 -> 100.1 mm, vias 0 -> 2
- net /D7: track 7.58 -> 102.5 mm, vias 0 -> 3
- net /D6: track 7.58 -> 98.3 mm, vias 0 -> 3
- net /A8: track 7.61 -> 97.2 mm, vias 0 -> 2
- net Earth: track 0.00 -> 88.9 mm
- net /D5: track 7.58 -> 95.5 mm, vias 0 -> 3
- net /A9: track 7.61 -> 92.3 mm, vias 0 -> 2
- net /D4: track 7.58 -> 90.4 mm, vias 0 -> 3
- net /D3: track 7.58 -> 85.8 mm, vias 0 -> 3
- net /A11: track 7.61 -> 83.4 mm, vias 0 -> 2
- net /A10: track 7.61 -> 78.3 mm, vias 0 -> 2
- net /D2: track 7.58 -> 70.8 mm, vias 0 -> 2
- net /D1: track 7.58 -> 65.7 mm, vias 0 -> 2
- net /EA: track 0.00 -> 54.7 mm, vias 0 -> 2
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
Commit message: 260215
Parts:
- added REF**: MountingHole_2.2mm_M2_DIN965_Pad, MountingHole:MountingHole_2.2mm_M2_DIN965_Pad, F.Cu at (162.6, 137.2)
- added REF**: MountingHole_2.2mm_M2_DIN965_Pad, MountingHole:MountingHole_2.2mm_M2_DIN965_Pad, F.Cu at (167.6, 134.6)
- added REF**: MountingHole_2.2mm_M2_DIN965_Pad, MountingHole:MountingHole_2.2mm_M2_DIN965_Pad, F.Cu at (142.2, 134.6)
- added REF**: MountingHole_2.2mm_M2_DIN965_Pad, MountingHole:MountingHole_2.2mm_M2_DIN965_Pad, F.Cu at (139.7, 134.6)
- added REF**: MountingHole_2.2mm_M2_DIN965_Pad, MountingHole:MountingHole_2.2mm_M2_DIN965_Pad, F.Cu at (154.9, 129.5)
- added REF**: MountingHole_2.2mm_M2_DIN965_Pad, MountingHole:MountingHole_2.2mm_M2_DIN965_Pad, F.Cu at (157.5, 129.5)
- added REF**: MountingHole_2.2mm_M2_DIN965_Pad, MountingHole:MountingHole_2.2mm_M2_DIN965_Pad, F.Cu at (147.3, 134.6)
- added REF**: MountingHole_2.2mm_M2_DIN965_Pad, MountingHole:MountingHole_2.2mm_M2_DIN965_Pad, F.Cu at (165.1, 129.5)
- added REF**: MountingHole_2.2mm_M2_DIN965_Pad, MountingHole:MountingHole_2.2mm_M2_DIN965_Pad, F.Cu at (137.2, 134.6)
- added REF**: MountingHole_2.2mm_M2_DIN965_Pad, MountingHole:MountingHole_2.2mm_M2_DIN965_Pad, F.Cu at (162.6, 129.5)
- added REF**: MountingHole_2.2mm_M2_DIN965_Pad, MountingHole:MountingHole_2.2mm_M2_DIN965_Pad, F.Cu at (134.6, 134.6)
- added REF**: MountingHole_2.2mm_M2_DIN965_Pad, MountingHole:MountingHole_2.2mm_M2_DIN965_Pad, F.Cu at (160.0, 134.6)
- added REF**: MountingHole_2.2mm_M2_DIN965_Pad, MountingHole:MountingHole_2.2mm_M2_DIN965_Pad, F.Cu at (154.9, 134.6)
- added REF**: MountingHole_2.2mm_M2_DIN965_Pad, MountingHole:MountingHole_2.2mm_M2_DIN965_Pad, F.Cu at (167.6, 137.2)
- added REF**: MountingHole_2.2mm_M2_DIN965_Pad, MountingHole:MountingHole_2.2mm_M2_DIN965_Pad, F.Cu at (137.2, 137.2)
- added REF**: MountingHole_2.2mm_M2_DIN965_Pad, MountingHole:MountingHole_2.2mm_M2_DIN965_Pad, F.Cu at (162.6, 134.6)
- added REF**: MountingHole_2.2mm_M2_DIN965_Pad, MountingHole:MountingHole_2.2mm_M2_DIN965_Pad, F.Cu at (139.7, 132.1)
- added REF**: MountingHole_2.2mm_M2_DIN965_Pad, MountingHole:MountingHole_2.2mm_M2_DIN965_Pad, F.Cu at (157.5, 132.1)
- added REF**: MountingHole_2.2mm_M2_DIN965_Pad, MountingHole:MountingHole_2.2mm_M2_DIN965_Pad, F.Cu at (160.0, 129.5)
- added REF**: MountingHole_2.2mm_M2_DIN965_Pad, MountingHole:MountingHole_2.2mm_M2_DIN965_Pad, F.Cu at (134.6, 132.1)
- added REF**: MountingHole_2.2mm_M2_DIN965_Pad, MountingHole:MountingHole_2.2mm_M2_DIN965_Pad, F.Cu at (152.4, 134.6)
- added REF**: MountingHole_2.2mm_M2_DIN965_Pad, MountingHole:MountingHole_2.2mm_M2_DIN965_Pad, F.Cu at (152.4, 132.1)
- added REF**: MountingHole_2.2mm_M2_DIN965_Pad, MountingHole:MountingHole_2.2mm_M2_DIN965_Pad, F.Cu at (165.1, 134.6)
- added REF**: MountingHole_2.2mm_M2_DIN965_Pad, MountingHole:MountingHole_2.2mm_M2_DIN965_Pad, F.Cu at (142.2, 137.2)
- added REF**: MountingHole_2.2mm_M2_DIN965_Pad, MountingHole:MountingHole_2.2mm_M2_DIN965_Pad, F.Cu at (149.9, 137.2)
- added REF**: MountingHole_2.2mm_M2_DIN965_Pad, MountingHole:MountingHole_2.2mm_M2_DIN965_Pad, F.Cu at (137.2, 132.1)
- added REF**: MountingHole_2.2mm_M2_DIN965_Pad, MountingHole:MountingHole_2.2mm_M2_DIN965_Pad, F.Cu at (162.6, 132.1)
- added REF**: MountingHole_2.2mm_M2_DIN965_Pad, MountingHole:MountingHole_2.2mm_M2_DIN965_Pad, F.Cu at (144.8, 137.2)
- added REF**: MountingHole_2.2mm_M2_DIN965_Pad, MountingHole:MountingHole_2.2mm_M2_DIN965_Pad, F.Cu at (157.5, 137.2)
- added REF**: MountingHole_2.2mm_M2_DIN965_Pad, MountingHole:MountingHole_2.2mm_M2_DIN965_Pad, F.Cu at (152.4, 137.2)
- added REF**: MountingHole_2.2mm_M2_DIN965_Pad, MountingHole:MountingHole_2.2mm_M2_DIN965_Pad, F.Cu at (154.9, 137.2)
- added REF**: MountingHole_2.2mm_M2_DIN965_Pad, MountingHole:MountingHole_2.2mm_M2_DIN965_Pad, F.Cu at (170.2, 129.5)
- added REF**: MountingHole_2.2mm_M2_DIN965_Pad, MountingHole:MountingHole_2.2mm_M2_DIN965_Pad, F.Cu at (170.2, 137.2)
- added REF**: MountingHole_2.2mm_M2_DIN965_Pad, MountingHole:MountingHole_2.2mm_M2_DIN965_Pad, F.Cu at (137.2, 129.5)
- added REF**: MountingHole_2.2mm_M2_DIN965_Pad, MountingHole:MountingHole_2.2mm_M2_DIN965_Pad, F.Cu at (170.2, 134.6)
- added REF**: MountingHole_2.2mm_M2_DIN965_Pad, MountingHole:MountingHole_2.2mm_M2_DIN965_Pad, F.Cu at (152.4, 129.5)
- added REF**: MountingHole_2.2mm_M2_DIN965_Pad, MountingHole:MountingHole_2.2mm_M2_DIN965_Pad, F.Cu at (134.6, 137.2)
- added REF**: MountingHole_2.2mm_M2_DIN965_Pad, MountingHole:MountingHole_2.2mm_M2_DIN965_Pad, F.Cu at (142.2, 132.1)
- added REF**: MountingHole_2.2mm_M2_DIN965_Pad, MountingHole:MountingHole_2.2mm_M2_DIN965_Pad, F.Cu at (144.8, 129.5)
- added REF**: MountingHole_2.2mm_M2_DIN965_Pad, MountingHole:MountingHole_2.2mm_M2_DIN965_Pad, F.Cu at (165.1, 137.2)
- added REF**: MountingHole_2.2mm_M2_DIN965_Pad, MountingHole:MountingHole_2.2mm_M2_DIN965_Pad, F.Cu at (165.1, 132.1)
- added REF**: MountingHole_2.2mm_M2_DIN965_Pad, MountingHole:MountingHole_2.2mm_M2_DIN965_Pad, F.Cu at (149.9, 134.6)
- added REF**: MountingHole_2.2mm_M2_DIN965_Pad, MountingHole:MountingHole_2.2mm_M2_DIN965_Pad, F.Cu at (157.5, 134.6)
- added REF**: MountingHole_2.2mm_M2_DIN965_Pad, MountingHole:MountingHole_2.2mm_M2_DIN965_Pad, F.Cu at (149.9, 129.5)
- added REF**: MountingHole_2.2mm_M2_DIN965_Pad, MountingHole:MountingHole_2.2mm_M2_DIN965_Pad, F.Cu at (134.6, 129.5)
- added REF**: MountingHole_2.2mm_M2_DIN965_Pad, MountingHole:MountingHole_2.2mm_M2_DIN965_Pad, F.Cu at (139.7, 137.2)
- added REF**: MountingHole_2.2mm_M2_DIN965_Pad, MountingHole:MountingHole_2.2mm_M2_DIN965_Pad, F.Cu at (167.6, 129.5)
- added REF**: MountingHole_2.2mm_M2_DIN965_Pad, MountingHole:MountingHole_2.2mm_M2_DIN965_Pad, F.Cu at (144.8, 134.6)
- added REF**: MountingHole_2.2mm_M2_DIN965_Pad, MountingHole:MountingHole_2.2mm_M2_DIN965_Pad, F.Cu at (139.7, 129.5)
- added REF**: MountingHole_2.2mm_M2_DIN965_Pad, MountingHole:MountingHole_2.2mm_M2_DIN965_Pad, F.Cu at (147.3, 129.5)
- added REF**: MountingHole_2.2mm_M2_DIN965_Pad, MountingHole:MountingHole_2.2mm_M2_DIN965_Pad, F.Cu at (142.2, 129.5)
- added REF**: MountingHole_2.2mm_M2_DIN965_Pad, MountingHole:MountingHole_2.2mm_M2_DIN965_Pad, F.Cu at (170.2, 132.1)
- added REF**: MountingHole_2.2mm_M2_DIN965_Pad, MountingHole:MountingHole_2.2mm_M2_DIN965_Pad, F.Cu at (160.0, 132.1)
- added REF**: MountingHole_2.2mm_M2_DIN965_Pad, MountingHole:MountingHole_2.2mm_M2_DIN965_Pad, F.Cu at (147.3, 132.1)
- added REF**: MountingHole_2.2mm_M2_DIN965_Pad, MountingHole:MountingHole_2.2mm_M2_DIN965_Pad, F.Cu at (144.8, 132.1)
- added REF**: MountingHole_2.2mm_M2_DIN965_Pad, MountingHole:MountingHole_2.2mm_M2_DIN965_Pad, F.Cu at (149.9, 132.1)
- added REF**: MountingHole_2.2mm_M2_DIN965_Pad, MountingHole:MountingHole_2.2mm_M2_DIN965_Pad, F.Cu at (147.3, 137.2)
- added REF**: MountingHole_2.2mm_M2_DIN965_Pad, MountingHole:MountingHole_2.2mm_M2_DIN965_Pad, F.Cu at (167.6, 132.1)
- added REF**: MountingHole_2.2mm_M2_DIN965_Pad, MountingHole:MountingHole_2.2mm_M2_DIN965_Pad, F.Cu at (154.9, 132.1)
- added REF**: MountingHole_2.2mm_M2_DIN965_Pad, MountingHole:MountingHole_2.2mm_M2_DIN965_Pad, F.Cu at (160.0, 137.2)
- moved C1 10.9 mm to (97.7, 84.1), turned to -90 degrees
- moved R8 6.81 mm to (192.0, 97.8), turned to -90 degrees
- moved JP1 0.13 mm to (176.3, 135.3)
Routing:
- net GNDD: track 49.0 -> 396.1 mm, vias 0 -> 3
- net +5V: track 29.5 -> 283.1 mm, vias 0 -> 2
- net Net-(U1-Pad11): track 2.54 -> 61.1 mm, vias 0 -> 2
- net Net-(U1-Pad10): track 2.54 -> 61.1 mm, vias 0 -> 2
- net Net-(J2-Pad1): track 29.8 -> 78.7 mm
- net Net-(J7-Pad2): track 26.7 -> 63.8 mm, vias 0 -> 2
- net Net-(J7-Pad3): track 23.0 -> 55.9 mm, vias 0 -> 2
- net /-RD: track 29.0 -> 51.1 mm
- net /-WR: track 29.0 -> 39.7 mm
- net Net-(R8-Pad2): track 5.28 -> 15.6 mm
- net Net-(R3-Pad2): track 0.00 -> 3.57 mm
- net Net-(C6-Pad2): track 44.2 -> 43.1 mm

Commit message: 260216
Parts:
- removed REF** (x60): MountingHole_2.2mm_M2_DIN965_Pad, MountingHole:MountingHole_2.2mm_M2_DIN965_Pad
- moved U4 32.9 mm to (72.6, 78.0), turned to 90 degrees
- moved C7 25.3 mm to (69.1, 71.6), turned to -90 degrees
- moved JP2 14.4 mm to (69.1, 65.0), turned to 180 degrees
- moved J5 5.08 mm to (122.9, 77.7)
- moved J4 1.65 mm to (143.8, 80.9)
- moved J6 1.65 mm to (189.5, 80.9)
- moved C13 0.11 mm to (76.4, 96.5)
Connections:
- R4 pad 1: Net-(U4-Pad3) -> Net-(R4-Pad1)
- R5 pad 2: Net-(U4-Pad6) -> Net-(R5-Pad2)
- R6 pad 1: Net-(U4-Pad8) -> Net-(R6-Pad1)
- U4 pad 1: Net-(JP2-Pad2) -> Net-(U1-Pad10)
- U4 pad 10: Net-(U1-Pad11) -> /-WR
- U4 pad 11: Net-(U4-Pad11) -> Net-(R4-Pad1)
- U4 pad 12: /-RD -> Net-(JP2-Pad2)
- U4 pad 13: /-WR -> Net-(JP2-Pad2)
- U4 pad 2: Net-(JP2-Pad2) -> Net-(U1-Pad10)
- U4 pad 3: Net-(U4-Pad3) -> Net-(R5-Pad2)
- U4 pad 4: Net-(U1-Pad10) -> Net-(U1-Pad11)
- U4 pad 5: Net-(U1-Pad10) -> Net-(U1-Pad11)
- U4 pad 6: Net-(U4-Pad6) -> Net-(R6-Pad1)
- U4 pad 9: Net-(U1-Pad11) -> /-RD
- U6 pad 19: Net-(U4-Pad11) -> Net-(U4-Pad8)
Routing:
- net /-RD: track 51.1 -> 152.4 mm, vias 0 -> 3
- net /-WR: track 39.7 -> 135.4 mm, vias 0 -> 1
- net Net-(J2-Pad1): track 78.7 -> 167.7 mm, vias 2 -> 4
- net Net-(U1-Pad11): track 61.1 -> 132.4 mm, vias 2 -> 5
- net Net-(U1-Pad10): track 61.1 -> 131.1 mm, vias 2 -> 3
- net Net-(U4-Pad8): track 16.0 -> 65.6 mm, vias 0 -> 2
- net Net-(R5-Pad2): track 0.00 -> 24.8 mm
- net Net-(R4-Pad1): track 0.00 -> 18.7 mm
- net Net-(R6-Pad1): track 0.00 -> 15.1 mm
- net Net-(JP2-Pad2): track 2.54 -> 15.6 mm
- net +5V: track 283.1 -> 295.9 mm
- net GNDD: track 396.1 -> 408.0 mm
- net Net-(U4-Pad3): track 8.18 -> 0.00 mm
- net Net-(U4-Pad6): track 6.60 -> 0.00 mm
- net Net-(J5-Pad7): track 4.33 -> 9.41 mm
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
Commit message: 260216
Parts:
- added ?: , , F.Cu at (204.5, 83.2)
- added ?: , , F.Cu at (113.0, 62.9)
- added ?: , , F.Cu at (168.9, 47.6)
- added ?: , , F.Cu at (209.6, 134.0)
- added ?: , , F.Cu at (209.6, 85.7)
- added ?: , , F.Cu at (204.5, 118.7)
- added ?: , , F.Cu at (199.4, 55.2)
- added ?: , , F.Cu at (125.7, 50.2)
- added ?: , , F.Cu at (95.2, 47.6)
- added ?: , , F.Cu at (92.7, 65.4)
- added ?: , , F.Cu at (148.6, 139.1)
- added ?: , , F.Cu at (148.6, 131.4)
- added ?: , , F.Cu at (128.3, 47.6)
- added ?: , , F.Cu at (148.6, 47.6)
- added ?: , , F.Cu at (179.1, 75.6)
- added ?: , , F.Cu at (95.2, 65.4)
- added ?: , , F.Cu at (204.5, 128.9)
- added ?: , , F.Cu at (135.9, 47.6)
- added ?: , , F.Cu at (146.1, 136.5)
- added ?: , , F.Cu at (90.2, 47.6)
- added ?: , , F.Cu at (186.7, 70.5)
- added ?: , , F.Cu at (199.4, 83.2)
- added ?: , , F.Cu at (102.9, 57.8)
- added ?: , , F.Cu at (90.2, 57.8)
- added ?: , , F.Cu at (148.6, 136.5)
- added ?: , , F.Cu at (201.9, 57.8)
- added ?: , , F.Cu at (151.1, 57.8)
- added ?: , , F.Cu at (87.6, 52.7)
- added ?: , , F.Cu at (201.9, 67.9)
- added ?: , , F.Cu at (92.7, 55.2)
- added ?: , , F.Cu at (181.6, 47.6)
- added ?: , , F.Cu at (186.7, 52.7)
- added ?: , , F.Cu at (125.7, 57.8)
- added ?: , , F.Cu at (186.7, 55.2)
- added ?: , , F.Cu at (209.6, 55.2)
- added ?: , , F.Cu at (153.7, 75.6)
- added ?: , , F.Cu at (138.4, 65.4)
- added ?: , , F.Cu at (184.2, 52.7)
- added ?: , , F.Cu at (133.3, 52.7)
- added ?: , , F.Cu at (148.6, 50.2)
- added ?: , , F.Cu at (95.2, 52.7)
- added ?: , , F.Cu at (196.8, 131.4)
- added ?: , , F.Cu at (105.4, 65.4)
- added ?: , , F.Cu at (141.0, 134.0)
- added ?: , , F.Cu at (156.2, 70.5)
- added ?: , , F.Cu at (201.9, 123.8)
- added ?: , , F.Cu at (161.3, 136.5)
- added ?: , , F.Cu at (194.3, 113.7)
- added ?: , , F.Cu at (95.2, 70.5)
- added ?: , , F.Cu at (176.5, 67.9)
- added ?: , , F.Cu at (204.5, 60.3)
- added ?: , , F.Cu at (207.0, 73.0)
- added ?: , , F.Cu at (171.4, 136.5)
- added ?: , , F.Cu at (204.5, 106.0)
- added ?: , , F.Cu at (168.9, 55.2)
- added ?: , , F.Cu at (209.6, 62.9)
- added ?: , , F.Cu at (207.0, 50.2)
- added ?: , , F.Cu at (207.0, 85.7)
- added ?: , , F.Cu at (138.4, 55.2)
- added ?: , , F.Cu at (87.6, 55.2)
- added ?: , , F.Cu at (163.8, 67.9)
- added ?: , , F.Cu at (209.6, 126.4)
- added ?: , , F.Cu at (69.8, 52.7)
- added ?: , , F.Cu at (158.8, 136.5)
- added ?: , , F.Cu at (108.0, 65.4)
- added ?: , , F.Cu at (153.7, 136.5)
- added ?: , , F.Cu at (156.2, 67.9)
- added ?: , , F.Cu at (125.7, 47.6)
- added ?: , , F.Cu at (102.9, 60.3)
- added ?: , , F.Cu at (148.6, 60.3)
- added ?: , , F.Cu at (143.5, 62.9)
- added ?: , , F.Cu at (181.6, 70.5)
- added ?: , , F.Cu at (201.9, 108.6)
- added ?: , , F.Cu at (199.4, 134.0)
- added ?: , , F.Cu at (95.2, 60.3)
- added ?: , , F.Cu at (209.6, 75.6)
- added ?: , , F.Cu at (97.8, 60.3)
- added ?: , , F.Cu at (90.2, 60.3)
- added ?: , , F.Cu at (135.9, 131.4)
- added ?: , , F.Cu at (196.8, 116.2)
- added ?: , , F.Cu at (196.8, 126.4)
- added ?: , , F.Cu at (209.6, 111.1)
- added ?: , , F.Cu at (143.5, 65.4)
- added ?: , , F.Cu at (105.4, 52.7)
- added ?: , , F.Cu at (194.3, 52.7)
- added ?: , , F.Cu at (204.5, 85.7)
- added ?: , , F.Cu at (138.4, 60.3)
- added ?: , , F.Cu at (204.5, 134.0)
- added ?: , , F.Cu at (199.4, 80.6)
- added ?: , , F.Cu at (102.9, 67.9)
- added ?: , , F.Cu at (201.9, 128.9)
- added ?: , , F.Cu at (204.5, 95.9)
- added ?: , , F.Cu at (194.3, 134.0)
- added ?: , , F.Cu at (151.1, 55.2)
- added ?: , , F.Cu at (196.8, 136.5)
- added ?: , , F.Cu at (201.9, 65.4)
- added ?: , , F.Cu at (135.9, 70.5)
- added ?: , , F.Cu at (130.8, 50.2)
- added ?: , , F.Cu at (194.3, 139.1)
- added ?: , , F.Cu at (133.3, 75.6)
- added ?: , , F.Cu at (163.8, 134.0)
- added ?: , , F.Cu at (125.7, 60.3)
- added ?: , , F.Cu at (199.4, 123.8)
- added ?: , , F.Cu at (128.3, 67.9)
- added ?: , , F.Cu at (209.6, 98.4)
- added ?: , , F.Cu at (204.5, 136.5)
- added ?: , , F.Cu at (199.4, 73.0)
- added ?: , , F.Cu at (156.2, 75.6)
- added ?: , , F.Cu at (156.2, 65.4)
- added ?: , , F.Cu at (184.2, 70.5)
- added ?: , , F.Cu at (199.4, 47.6)
- added ?: , , F.Cu at (138.4, 52.7)
- added ?: , , F.Cu at (199.4, 95.9)
- added ?: , , F.Cu at (153.7, 73.0)
- added ?: , , F.Cu at (199.4, 116.2)
- added ?: , , F.Cu at (176.5, 50.2)
- added ?: , , F.Cu at (207.0, 126.4)
- added ?: , , F.Cu at (196.8, 85.7)
- added ?: , , F.Cu at (158.8, 57.8)
- added ?: , , F.Cu at (158.8, 73.0)
- added ?: , , F.Cu at (138.4, 128.9)
- added ?: , , F.Cu at (194.3, 57.8)
- added ?: , , F.Cu at (204.5, 57.8)
- added ?: , , F.Cu at (176.5, 65.4)
- added ?: , , F.Cu at (110.5, 65.4)
- added ?: , , F.Cu at (72.4, 47.6)
- added ?: , , F.Cu at (207.0, 134.0)
- added ?: , , F.Cu at (199.4, 65.4)
- added ?: , , F.Cu at (90.2, 52.7)
- added ?: , , F.Cu at (143.5, 67.9)
- added ?: , , F.Cu at (179.1, 50.2)
- added ?: , , F.Cu at (201.9, 103.5)
- added ?: , , F.Cu at (207.0, 65.4)
- added ?: , , F.Cu at (153.7, 52.7)
- added ?: , , F.Cu at (110.5, 52.7)
- added ?: , , F.Cu at (209.6, 116.2)
- added ?: , , F.Cu at (118.1, 60.3)
- added ?: , , F.Cu at (128.3, 62.9)
- added ?: , , F.Cu at (108.0, 73.0)
- added ?: , , F.Cu at (179.1, 47.6)
- added ?: , , F.Cu at (207.0, 123.8)
- added ?: , , F.Cu at (184.2, 65.4)
- added ?: , , F.Cu at (194.3, 67.9)
- added ?: , , F.Cu at (151.1, 70.5)
- added ?: , , F.Cu at (151.1, 62.9)
- added ?: , , F.Cu at (85.1, 47.6)
- added ?: , , F.Cu at (153.7, 128.9)
- added ?: , , F.Cu at (87.6, 57.8)
- added ?: , , F.Cu at (156.2, 57.8)
- added ?: , , F.Cu at (97.8, 70.5)
- added ?: , , F.Cu at (207.0, 52.7)
- added ?: , , F.Cu at (184.2, 57.8)
- added ?: , , F.Cu at (168.9, 73.0)
- added ?: , , F.Cu at (179.1, 65.4)
- added ?: , , F.Cu at (201.9, 139.1)
- added ?: , , F.Cu at (90.2, 55.2)
- added ?: , , F.Cu at (209.6, 60.3)
- added ?: , , F.Cu at (209.6, 123.8)
- added ?: , , F.Cu at (181.6, 50.2)
- added ?: , , F.Cu at (151.1, 139.1)
- added ?: , , F.Cu at (168.9, 60.3)
- added ?: , , F.Cu at (118.1, 70.5)
- added ?: , , F.Cu at (207.0, 101.0)
- added ?: , , F.Cu at (199.4, 101.0)
- added ?: , , F.Cu at (166.4, 128.9)
- added ?: , , F.Cu at (204.5, 88.3)
- added ?: , , F.Cu at (143.5, 70.5)
- added ?: , , F.Cu at (207.0, 113.7)
- added ?: , , F.Cu at (141.0, 128.9)
- added ?: , , F.Cu at (199.4, 103.5)
- added ?: , , F.Cu at (80.0, 52.7)
- added ?: , , F.Cu at (186.7, 62.9)
- added ?: , , F.Cu at (189.2, 52.7)
- added ?: , , F.Cu at (102.9, 47.6)
- added ?: , , F.Cu at (207.0, 67.9)
- added ?: , , F.Cu at (97.8, 65.4)
- added ?: , , F.Cu at (194.3, 65.4)
- added ?: , , F.Cu at (174.0, 60.3)
- added ?: , , F.Cu at (161.3, 47.6)
- added ?: , , F.Cu at (204.5, 113.7)
- added ?: , , F.Cu at (97.8, 57.8)
- added ?: , , F.Cu at (163.8, 73.0)
- added ?: , , F.Cu at (168.9, 70.5)
- added ?: , , F.Cu at (174.0, 73.0)
- added ?: , , F.Cu at (85.1, 52.7)
- added ?: , , F.Cu at (201.9, 116.2)
- added ?: , , F.Cu at (161.3, 55.2)
- added ?: , , F.Cu at (209.6, 118.7)
- added ?: , , F.Cu at (186.7, 73.0)
- added ?: , , F.Cu at (118.1, 57.8)
- added ?: , , F.Cu at (123.2, 55.2)
- added ?: , , F.Cu at (97.8, 50.2)
- added ?: , , F.Cu at (176.5, 47.6)
- added ?: , , F.Cu at (130.8, 65.4)
- added ?: , , F.Cu at (97.8, 67.9)
- added ?: , , F.Cu at (181.6, 57.8)
- added ?: , , F.Cu at (153.7, 55.2)
- added ?: , , F.Cu at (156.2, 134.0)
- added ?: , , F.Cu at (209.6, 57.8)
- added ?: , , F.Cu at (135.9, 62.9)
- added ?: , , F.Cu at (179.1, 52.7)
- added ?: , , F.Cu at (209.6, 78.1)
- added ?: , , F.Cu at (100.3, 70.5)
- added ?: , , F.Cu at (181.6, 62.9)
- added ?: , , F.Cu at (100.3, 62.9)
- added ?: , , F.Cu at (179.1, 70.5)
- added ?: , , F.Cu at (102.9, 55.2)
- added ?: , , F.Cu at (196.8, 78.1)
- added ?: , , F.Cu at (105.4, 67.9)
- added ?: , , F.Cu at (194.3, 111.1)
- added ?: , , F.Cu at (201.9, 73.0)
- added ?: , , F.Cu at (199.4, 93.3)
- added ?: , , F.Cu at (158.8, 62.9)
- added ?: , , F.Cu at (196.8, 83.2)
- added ?: , , F.Cu at (161.3, 70.5)
- added ?: , , F.Cu at (174.0, 70.5)
- added ?: , , F.Cu at (174.0, 50.2)
- added ?: , , F.Cu at (151.1, 128.9)
- added ?: , , F.Cu at (123.2, 65.4)
- added ?: , , F.Cu at (196.8, 103.5)
- added ?: , , F.Cu at (161.3, 62.9)
- added ?: , , F.Cu at (130.8, 62.9)
- added ?: , , F.Cu at (74.9, 47.6)
- added ?: , , F.Cu at (77.5, 47.6)
- added ?: , , F.Cu at (100.3, 47.6)
- added ?: , , F.Cu at (135.9, 75.6)
- added ?: , , F.Cu at (105.4, 60.3)
- added ?: , , F.Cu at (128.3, 73.0)
- added ?: , , F.Cu at (168.9, 50.2)
- added ?: , , F.Cu at (82.5, 50.2)
- added ?: , , F.Cu at (209.6, 121.3)
- added ?: , , F.Cu at (133.3, 57.8)
- added ?: , , F.Cu at (153.7, 70.5)
- added ?: , , F.Cu at (199.4, 128.9)
- added ?: , , F.Cu at (207.0, 118.7)
- added ?: , , F.Cu at (196.8, 121.3)
- added ?: , , F.Cu at (194.3, 50.2)
- added ?: , , F.Cu at (163.8, 139.1)
- added ?: , , F.Cu at (176.5, 139.1)
- added ?: , , F.Cu at (189.2, 73.0)
- added ?: , , F.Cu at (123.2, 67.9)
- added ?: , , F.Cu at (181.6, 55.2)
- added ?: , , F.Cu at (92.7, 47.6)
- added ?: , , F.Cu at (151.1, 134.0)
- added ?: , , F.Cu at (209.6, 52.7)
- added ?: , , F.Cu at (87.6, 50.2)
- added ?: , , F.Cu at (194.3, 136.5)
- added ?: , , F.Cu at (148.6, 134.0)
- added ?: , , F.Cu at (87.6, 62.9)
- added ?: , , F.Cu at (153.7, 57.8)
- added ?: , , F.Cu at (207.0, 98.4)
- added ?: , , F.Cu at (201.9, 52.7)
- added ?: , , F.Cu at (204.5, 62.9)
- added ?: , , F.Cu at (163.8, 65.4)
- added ?: , , F.Cu at (158.8, 134.0)
- added ?: , , F.Cu at (148.6, 52.7)
- added ?: , , F.Cu at (161.3, 67.9)
- added ?: , , F.Cu at (179.1, 60.3)
- added ?: , , F.Cu at (133.3, 128.9)
- added ?: , , F.Cu at (209.6, 95.9)
- added ?: , , F.Cu at (196.8, 98.4)
- added ?: , , F.Cu at (148.6, 128.9)
- added ?: , , F.Cu at (194.3, 103.5)
- added ?: , , F.Cu at (189.2, 65.4)
- added ?: , , F.Cu at (148.6, 55.2)
- added ?: , , F.Cu at (130.8, 60.3)
- added ?: , , F.Cu at (174.0, 52.7)
- added ?: , , F.Cu at (174.0, 55.2)
- added ?: , , F.Cu at (151.1, 60.3)
- added ?: , , F.Cu at (201.9, 50.2)
- added ?: , , F.Cu at (143.5, 128.9)
- added ?: , , F.Cu at (125.7, 52.7)
- added ?: , , F.Cu at (105.4, 47.6)
- added ?: , , F.Cu at (128.3, 52.7)
- added ?: , , F.Cu at (189.2, 57.8)
- added ?: , , F.Cu at (174.0, 75.6)
- added ?: , , F.Cu at (163.8, 47.6)
- added ?: , , F.Cu at (186.7, 60.3)
- added ?: , , F.Cu at (204.5, 98.4)
- added ?: , , F.Cu at (151.1, 50.2)
- added ?: , , F.Cu at (138.4, 47.6)
- added ?: , , F.Cu at (209.6, 88.3)
- added ?: , , F.Cu at (102.9, 50.2)
- added ?: , , F.Cu at (207.0, 70.5)
- added ?: , , F.Cu at (199.4, 67.9)
- added ?: , , F.Cu at (209.6, 136.5)
- added ?: , , F.Cu at (196.8, 108.6)
- added ?: , , F.Cu at (189.2, 67.9)
- added ?: , , F.Cu at (130.8, 67.9)
- added ?: , , F.Cu at (199.4, 85.7)
- added ?: , , F.Cu at (209.6, 67.9)
- added ?: , , F.Cu at (72.4, 52.7)
- added ?: , , F.Cu at (143.5, 73.0)
- added ?: , , F.Cu at (108.0, 67.9)
- added ?: , , F.Cu at (118.1, 55.2)
- added ?: , , F.Cu at (207.0, 121.3)
- added ?: , , F.Cu at (130.8, 73.0)
- added ?: , , F.Cu at (181.6, 60.3)
- added ?: , , F.Cu at (201.9, 136.5)
- added ?: , , F.Cu at (194.3, 118.7)
- added ?: , , F.Cu at (135.9, 128.9)
- added ?: , , F.Cu at (161.3, 65.4)
- added ?: , , F.Cu at (156.2, 62.9)
- added ?: , , F.Cu at (77.5, 50.2)
- added ?: , , F.Cu at (123.2, 60.3)
- added ?: , , F.Cu at (181.6, 75.6)
- added ?: , , F.Cu at (153.7, 139.1)
- added ?: , , F.Cu at (108.0, 70.5)
- added ?: , , F.Cu at (146.1, 128.9)
- added ?: , , F.Cu at (201.9, 55.2)
- added ?: , , F.Cu at (161.3, 128.9)
- added ?: , , F.Cu at (69.8, 50.2)
- added ?: , , F.Cu at (138.4, 131.4)
- added ?: , , F.Cu at (110.5, 47.6)
- added ?: , , F.Cu at (201.9, 101.0)
- added ?: , , F.Cu at (207.0, 57.8)
- added ?: , , F.Cu at (133.3, 70.5)
- added ?: , , F.Cu at (148.6, 65.4)
- added ?: , , F.Cu at (143.5, 47.6)
- added ?: , , F.Cu at (204.5, 90.8)
- added ?: , , F.Cu at (204.5, 80.6)
- added ?: , , F.Cu at (186.7, 50.2)
- added ?: , , F.Cu at (163.8, 75.6)
- added ?: , , F.Cu at (77.5, 52.7)
- added ?: , , F.Cu at (204.5, 101.0)
- added ?: , , F.Cu at (130.8, 55.2)
- added ?: , , F.Cu at (113.0, 52.7)
- added ?: , , F.Cu at (108.0, 60.3)
- added ?: , , F.Cu at (204.5, 70.5)
- added ?: , , F.Cu at (161.3, 139.1)
- added ?: , , F.Cu at (204.5, 75.6)
- added ?: , , F.Cu at (168.9, 62.9)
- added ?: , , F.Cu at (143.5, 52.7)
- added ?: , , F.Cu at (204.5, 126.4)
- added ?: , , F.Cu at (194.3, 47.6)
- added ?: , , F.Cu at (158.8, 60.3)
- added ?: , , F.Cu at (156.2, 60.3)
- added ?: , , F.Cu at (128.3, 70.5)
- added ?: , , F.Cu at (97.8, 47.6)
- added ?: , , F.Cu at (196.8, 106.0)
- added ?: , , F.Cu at (204.5, 93.3)
- added ?: , , F.Cu at (199.4, 52.7)
- added ?: , , F.Cu at (146.1, 134.0)
- added ?: , , F.Cu at (156.2, 128.9)
- added ?: , , F.Cu at (199.4, 75.6)
- added ?: , , F.Cu at (201.9, 75.6)
- added ?: , , F.Cu at (161.3, 134.0)
- added ?: , , F.Cu at (110.5, 67.9)
- added ?: , , F.Cu at (174.0, 47.6)
- added ?: , , F.Cu at (156.2, 55.2)
- added ?: , , F.Cu at (194.3, 73.0)
- added ?: , , F.Cu at (207.0, 60.3)
- added ?: , , F.Cu at (201.9, 85.7)
- added ?: , , F.Cu at (204.5, 121.3)
- added ?: , , F.Cu at (108.0, 50.2)
- added ?: , , F.Cu at (100.3, 60.3)
- added ?: , , F.Cu at (196.8, 88.3)
- added ?: , , F.Cu at (204.5, 139.1)
- added ?: , , F.Cu at (143.5, 55.2)
- added ?: , , F.Cu at (100.3, 55.2)
- added ?: , , F.Cu at (87.6, 65.4)
- added ?: , , F.Cu at (153.7, 47.6)
- added ?: , , F.Cu at (108.0, 47.6)
- added ?: , , F.Cu at (148.6, 75.6)
- added ?: , , F.Cu at (156.2, 52.7)
- added ?: , , F.Cu at (194.3, 70.5)
- added ?: , , F.Cu at (135.9, 67.9)
- added ?: , , F.Cu at (186.7, 57.8)
- added ?: , , F.Cu at (128.3, 55.2)
- added ?: , , F.Cu at (148.6, 67.9)
- added ?: , , F.Cu at (135.9, 134.0)
- added ?: , , F.Cu at (184.2, 62.9)
- added ?: , , F.Cu at (97.8, 62.9)
- added ?: , , F.Cu at (110.5, 60.3)
- added ?: , , F.Cu at (69.8, 47.6)
- added ?: , , F.Cu at (209.6, 128.9)
- added ?: , , F.Cu at (201.9, 62.9)
- added ?: , , F.Cu at (201.9, 121.3)
- added ?: , , F.Cu at (156.2, 131.4)
- added ?: , , F.Cu at (191.8, 139.1)
- added ?: , , F.Cu at (143.5, 50.2)
- added ?: , , F.Cu at (199.4, 50.2)
- added ?: , , F.Cu at (133.3, 131.4)
- added ?: , , F.Cu at (209.6, 80.6)
- added ?: , , F.Cu at (143.5, 139.1)
- added ?: , , F.Cu at (168.9, 139.1)
- added ?: , , F.Cu at (186.7, 47.6)
- added ?: , , F.Cu at (158.8, 67.9)
- added ?: , , F.Cu at (199.4, 62.9)
- added ?: , , F.Cu at (100.3, 50.2)
- added ?: , , F.Cu at (92.7, 67.9)
- added ?: , , F.Cu at (156.2, 73.0)
- added ?: , , F.Cu at (133.3, 62.9)
- added ?: , , F.Cu at (194.3, 106.0)
- added ?: , , F.Cu at (90.2, 50.2)
- added ?: , , F.Cu at (194.3, 60.3)
- added ?: , , F.Cu at (90.2, 65.4)
- added ?: , , F.Cu at (171.4, 131.4)
- added ?: , , F.Cu at (209.6, 101.0)
- added ?: , , F.Cu at (204.5, 73.0)
- added ?: , , F.Cu at (153.7, 134.0)
- added ?: , , F.Cu at (194.3, 62.9)
- added ?: , , F.Cu at (199.4, 121.3)
- added ?: , , F.Cu at (151.1, 131.4)
- added ?: , , F.Cu at (194.3, 55.2)
- added ?: , , F.Cu at (85.1, 55.2)
- added ?: , , F.Cu at (176.5, 57.8)
- added ?: , , F.Cu at (158.8, 55.2)
- added ?: , , F.Cu at (179.1, 67.9)
- added ?: , , F.Cu at (123.2, 52.7)
- added ?: , , F.Cu at (207.0, 75.6)
- added ?: , , F.Cu at (196.8, 101.0)
- added ?: , , F.Cu at (181.6, 52.7)
- added ?: , , F.Cu at (113.0, 50.2)
- added ?: , , F.Cu at (181.6, 65.4)
- added ?: , , F.Cu at (201.9, 83.2)
- added ?: , , F.Cu at (130.8, 70.5)
- added ?: , , F.Cu at (133.3, 47.6)
- added ?: , , F.Cu at (196.8, 123.8)
- added ?: , , F.Cu at (194.3, 123.8)
- added ?: , , F.Cu at (125.7, 62.9)
- added ?: , , F.Cu at (92.7, 57.8)
- added ?: , , F.Cu at (204.5, 52.7)
- added ?: , , F.Cu at (151.1, 47.6)
- added ?: , , F.Cu at (201.9, 113.7)
- added ?: , , F.Cu at (153.7, 50.2)
- added ?: , , F.Cu at (207.0, 139.1)
- added ?: , , F.Cu at (204.5, 116.2)
- added ?: , , F.Cu at (207.0, 95.9)
- added ?: , , F.Cu at (85.1, 50.2)
- added ?: , , F.Cu at (135.9, 65.4)
- added ?: , , F.Cu at (207.0, 55.2)
- added ?: , , F.Cu at (199.4, 118.7)
- added ?: , , F.Cu at (199.4, 136.5)
- added ?: , , F.Cu at (113.0, 60.3)
- added ?: , , F.Cu at (163.8, 57.8)
- added ?: , , F.Cu at (207.0, 88.3)
- added ?: , , F.Cu at (158.8, 70.5)
- added ?: , , F.Cu at (207.0, 108.6)
- added ?: , , F.Cu at (179.1, 62.9)
- added ?: , , F.Cu at (204.5, 103.5)
- added ?: , , F.Cu at (153.7, 60.3)
- added ?: , , F.Cu at (184.2, 47.6)
- added ?: , , F.Cu at (133.3, 134.0)
- added ?: , , F.Cu at (141.0, 136.5)
- added ?: , , F.Cu at (92.7, 50.2)
- added ?: , , F.Cu at (133.3, 50.2)
- added ?: , , F.Cu at (174.0, 57.8)
- added ?: , , F.Cu at (110.5, 62.9)
- added ?: , , F.Cu at (163.8, 136.5)
- added ?: , , F.Cu at (138.4, 57.8)
- added ?: , , F.Cu at (201.9, 90.8)
- added ?: , , F.Cu at (194.3, 121.3)
- added ?: , , F.Cu at (123.2, 73.0)
- added ?: , , F.Cu at (199.4, 57.8)
- added ?: , , F.Cu at (176.5, 60.3)
- added ?: , , F.Cu at (176.5, 70.5)
- added ?: , , F.Cu at (201.9, 95.9)
- added ?: , , F.Cu at (102.9, 73.0)
- added ?: , , F.Cu at (110.5, 73.0)
- added ?: , , F.Cu at (199.4, 131.4)
- added ?: , , F.Cu at (207.0, 131.4)
- added ?: , , F.Cu at (105.4, 73.0)
- added ?: , , F.Cu at (141.0, 139.1)
- added ?: , , F.Cu at (163.8, 55.2)
- added ?: , , F.Cu at (199.4, 78.1)
- added ?: , , F.Cu at (184.2, 67.9)
- added ?: , , F.Cu at (199.4, 111.1)
- added ?: , , F.Cu at (207.0, 106.0)
- added ?: , , F.Cu at (209.6, 65.4)
- added ?: , , F.Cu at (181.6, 139.1)
- added ?: , , F.Cu at (176.5, 52.7)
- added ?: , , F.Cu at (143.5, 60.3)
- added ?: , , F.Cu at (108.0, 57.8)
- added ?: , , F.Cu at (82.5, 47.6)
- added ?: , , F.Cu at (138.4, 75.6)
- added ?: , , F.Cu at (174.0, 65.4)
- added ?: , , F.Cu at (133.3, 139.1)
- added ?: , , F.Cu at (80.0, 50.2)
- added ?: , , F.Cu at (207.0, 83.2)
- added ?: , , F.Cu at (209.6, 83.2)
- added ?: , , F.Cu at (158.8, 50.2)
- added ?: , , F.Cu at (113.0, 55.2)
- added ?: , , F.Cu at (128.3, 50.2)
- added ?: , , F.Cu at (168.9, 67.9)
- added ?: , , F.Cu at (168.9, 57.8)
- added ?: , , F.Cu at (138.4, 62.9)
- added ?: , , F.Cu at (179.1, 57.8)
- added ?: , , F.Cu at (146.1, 139.1)
- added ?: , , F.Cu at (171.4, 134.0)
- added ?: , , F.Cu at (201.9, 70.5)
- added ?: , , F.Cu at (135.9, 50.2)
- added ?: , , F.Cu at (207.0, 80.6)
- added ?: , , F.Cu at (123.2, 70.5)
- added ?: , , F.Cu at (196.8, 113.7)
- added ?: , , F.Cu at (168.9, 131.4)
- added ?: , , F.Cu at (82.5, 52.7)
- added ?: , , F.Cu at (158.8, 128.9)
- added ?: , , F.Cu at (100.3, 52.7)
- added ?: , , F.Cu at (100.3, 73.0)
- added ?: , , F.Cu at (194.3, 108.6)
- added ?: , , F.Cu at (92.7, 52.7)
- added ?: , , F.Cu at (87.6, 60.3)
- added ?: , , F.Cu at (207.0, 93.3)
- added ?: , , F.Cu at (201.9, 78.1)
- added ?: , , F.Cu at (179.1, 73.0)
- added ?: , , F.Cu at (209.6, 93.3)
- added ?: , , F.Cu at (158.8, 139.1)
- added ?: , , F.Cu at (184.2, 50.2)
- added ?: , , F.Cu at (199.4, 60.3)
- added ?: , , F.Cu at (80.0, 47.6)
- added ?: , , F.Cu at (168.9, 75.6)
- added ?: , , F.Cu at (201.9, 47.6)
- added ?: , , F.Cu at (189.2, 60.3)
- added ?: , , F.Cu at (189.2, 47.6)
- added ?: , , F.Cu at (151.1, 136.5)
- added ?: , , F.Cu at (125.7, 67.9)
- added ?: , , F.Cu at (108.0, 55.2)
- added ?: , , F.Cu at (176.5, 55.2)
- added ?: , , F.Cu at (125.7, 73.0)
- added ?: , , F.Cu at (196.8, 80.6)
- added ?: , , F.Cu at (189.2, 55.2)
- added ?: , , F.Cu at (171.4, 128.9)
- added ?: , , F.Cu at (186.7, 65.4)
- added ?: , , F.Cu at (204.5, 65.4)
- added ?: , , F.Cu at (189.2, 50.2)
- added ?: , , F.Cu at (209.6, 90.8)
- added ?: , , F.Cu at (110.5, 50.2)
- added ?: , , F.Cu at (161.3, 52.7)
- added ?: , , F.Cu at (201.9, 106.0)
- added ?: , , F.Cu at (153.7, 131.4)
- added ?: , , F.Cu at (199.4, 108.6)
- added ?: , , F.Cu at (207.0, 116.2)
- added ?: , , F.Cu at (97.8, 52.7)
- added ?: , , F.Cu at (176.5, 73.0)
- added ?: , , F.Cu at (163.8, 131.4)
- added ?: , , F.Cu at (199.4, 88.3)
- added ?: , , F.Cu at (176.5, 62.9)
- added ?: , , F.Cu at (135.9, 136.5)
- added ?: , , F.Cu at (135.9, 55.2)
- added ?: , , F.Cu at (105.4, 55.2)
- added ?: , , F.Cu at (92.7, 70.5)
- added ?: , , F.Cu at (143.5, 57.8)
- added ?: , , F.Cu at (161.3, 131.4)
- added ?: , , F.Cu at (102.9, 70.5)
- added ?: , , F.Cu at (138.4, 134.0)
- added ?: , , F.Cu at (95.2, 57.8)
- added ?: , , F.Cu at (133.3, 65.4)
- added ?: , , F.Cu at (118.1, 67.9)
- added ?: , , F.Cu at (209.6, 73.0)
- added ?: , , F.Cu at (110.5, 55.2)
- added ?: , , F.Cu at (151.1, 65.4)
- added ?: , , F.Cu at (184.2, 60.3)
- added ?: , , F.Cu at (196.8, 139.1)
- added ?: , , F.Cu at (163.8, 60.3)
- added ?: , , F.Cu at (158.8, 65.4)
- added ?: , , F.Cu at (105.4, 70.5)
- added ?: , , F.Cu at (138.4, 73.0)
- added ?: , , F.Cu at (199.4, 126.4)
- added ?: , , F.Cu at (189.2, 75.6)
- added ?: , , F.Cu at (184.2, 139.1)
- added ?: , , F.Cu at (128.3, 57.8)
- added ?: , , F.Cu at (92.7, 60.3)
- added ?: , , F.Cu at (204.5, 131.4)
- added ?: , , F.Cu at (207.0, 136.5)
- added ?: , , F.Cu at (204.5, 67.9)
- added ?: , , F.Cu at (181.6, 67.9)
- added ?: , , F.Cu at (118.1, 73.0)
- added ?: , , F.Cu at (163.8, 70.5)
- added ?: , , F.Cu at (135.9, 139.1)
- added ?: , , F.Cu at (148.6, 57.8)
- added ?: , , F.Cu at (209.6, 50.2)
- added ?: , , F.Cu at (113.0, 73.0)
- added ?: , , F.Cu at (130.8, 52.7)
- added ?: , , F.Cu at (168.9, 128.9)
- added ?: , , F.Cu at (184.2, 55.2)
- added ?: , , F.Cu at (168.9, 134.0)
- added ?: , , F.Cu at (156.2, 136.5)
- added ?: , , F.Cu at (102.9, 52.7)
- added ?: , , F.Cu at (90.2, 62.9)
- added ?: , , F.Cu at (128.3, 60.3)
- added ?: , , F.Cu at (204.5, 111.1)
- added ?: , , F.Cu at (113.0, 65.4)
- added ?: , , F.Cu at (97.8, 55.2)
- added ?: , , F.Cu at (148.6, 73.0)
- added ?: , , F.Cu at (204.5, 47.6)
- added ?: , , F.Cu at (161.3, 50.2)
- added ?: , , F.Cu at (100.3, 57.8)
- added ?: , , F.Cu at (196.8, 93.3)
- added ?: , , F.Cu at (201.9, 111.1)
- added ?: , , F.Cu at (174.0, 67.9)
- added ?: , , F.Cu at (148.6, 70.5)
- added ?: , , F.Cu at (201.9, 131.4)
- added ?: , , F.Cu at (189.2, 139.1)
- added ?: , , F.Cu at (118.1, 65.4)
- added ?: , , F.Cu at (105.4, 50.2)
- added ?: , , F.Cu at (209.6, 47.6)
- added ?: , , F.Cu at (199.4, 139.1)
- added ?: , , F.Cu at (158.8, 52.7)
- added ?: , , F.Cu at (196.8, 134.0)
- added ?: , , F.Cu at (186.7, 75.6)
- added ?: , , F.Cu at (151.1, 75.6)
- added ?: , , F.Cu at (113.0, 70.5)
- added ?: , , F.Cu at (123.2, 57.8)
- added ?: , , F.Cu at (166.4, 134.0)
- added ?: , , F.Cu at (204.5, 50.2)
- added ?: , , F.Cu at (161.3, 60.3)
- added ?: , , F.Cu at (153.7, 65.4)
- added ?: , , F.Cu at (168.9, 65.4)
- added ?: , , F.Cu at (163.8, 50.2)
- added ?: , , F.Cu at (135.9, 60.3)
- added ?: , , F.Cu at (143.5, 131.4)
- added ?: , , F.Cu at (181.6, 73.0)
- added ?: , , F.Cu at (158.8, 75.6)
- added ?: , , F.Cu at (128.3, 75.6)
- added ?: , , F.Cu at (130.8, 75.6)
- added ?: , , F.Cu at (133.3, 60.3)
- added ?: , , F.Cu at (118.1, 62.9)
- added ?: , , F.Cu at (156.2, 47.6)
- added ?: , , F.Cu at (158.8, 47.6)
- added ?: , , F.Cu at (179.1, 139.1)
- added ?: , , F.Cu at (118.1, 52.7)
- added ?: , , F.Cu at (110.5, 70.5)
- added ?: , , F.Cu at (125.7, 65.4)
- added ?: , , F.Cu at (209.6, 103.5)
- added ?: , , F.Cu at (189.2, 70.5)
- added ?: , , F.Cu at (108.0, 62.9)
- added ?: , , F.Cu at (72.4, 50.2)
- added ?: , , F.Cu at (146.1, 131.4)
- added ?: , , F.Cu at (92.7, 62.9)
- added ?: , , F.Cu at (105.4, 57.8)
- added ?: , , F.Cu at (201.9, 93.3)
- added ?: , , F.Cu at (156.2, 50.2)
- added ?: , , F.Cu at (110.5, 57.8)
- added ?: , , F.Cu at (135.9, 52.7)
- added ?: , , F.Cu at (133.3, 73.0)
- added ?: , , F.Cu at (204.5, 108.6)
- added ?: , , F.Cu at (95.2, 55.2)
- added ?: , , F.Cu at (133.3, 136.5)
- added ?: , , F.Cu at (163.8, 52.7)
- added ?: , , F.Cu at (158.8, 131.4)
- added ?: , , F.Cu at (209.6, 139.1)
- added ?: , , F.Cu at (207.0, 103.5)
- added ?: , , F.Cu at (201.9, 98.4)
- added ?: , , F.Cu at (196.8, 90.8)
- added ?: , , F.Cu at (194.3, 116.2)
- added ?: , , F.Cu at (100.3, 65.4)
- added ?: , , F.Cu at (151.1, 73.0)
- added ?: , , F.Cu at (135.9, 73.0)
- added ?: , , F.Cu at (161.3, 75.6)
- added ?: , , F.Cu at (171.4, 139.1)
- added ?: , , F.Cu at (138.4, 50.2)
- added ?: , , F.Cu at (204.5, 55.2)
- added ?: , , F.Cu at (95.2, 67.9)
- added ?: , , F.Cu at (135.9, 57.8)
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Connections:
- J8 pad a10: unconnected-(J8-Pada10) -> (no net)
- J8 pad a12: unconnected-(J8-Pada12) -> (no net)
- J8 pad a14: unconnected-(J8-Pada14) -> (no net)
- J8 pad a16: unconnected-(J8-Pada16) -> (no net)
- J8 pad a18: unconnected-(J8-Pada18) -> (no net)
- J8 pad a2: unconnected-(J8-Pada2) -> GNDD
- J8 pad a20: unconnected-(J8-Pada20) -> (no net)
- J8 pad a22: unconnected-(J8-Pada22) -> (no net)
- J8 pad a24: unconnected-(J8-Pada24) -> (no net)
- J8 pad a26: unconnected-(J8-Pada26) -> (no net)
- J8 pad a28: unconnected-(J8-Pada28) -> (no net)
- J8 pad a30: unconnected-(J8-Pada30) -> (no net)
- J8 pad a32: unconnected-(J8-Pada32) -> (no net)
- J8 pad a4: unconnected-(J8-Pada4) -> +5V
- J8 pad a6: unconnected-(J8-Pada6) -> (no net)
- J8 pad a8: unconnected-(J8-Pada8) -> (no net)
Routing:
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
Commit message: 260216
Routing:
- net Earth: track 88.9 -> 142.6 mm
Other:
- board text added: "2026"
- board text added: "JP1: EXT ROM JP2: ACT LED"
- board text added: "PEIX External interface box"
- board text added: "Pozsar Zsolt"
Changed lines of the file:
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@@
     (pad_to_mask_clearance 0)
     (pcbplotparams
-      (layerselection 0x0000020_ffffffff)
+      (layerselection 0x00010e0_ffffffff)
       (disableapertmacros false)
       (usegerberextensions false)
@@
       (sketchpadsonfab false)
       (subtractmaskfromsilk false)
-      (outputformat 4)
+      (outputformat 1)
       (mirror false)
-      (drillshape 2)
+      (drillshape 0)
       (scaleselection 1)
       (outputdirectory "")
@@
     (pad "" thru_hole roundrect (at 0 0) (size 1.8 1.8) (drill 0.8) (layers F&B.Cu *.Mask) (roundrect_rratio 0.25))
   )
+  (gr_rect (start 81.28 139.7) (end 125.095 143.51) (layer "B.Mask") (width 0.15) (fill solid))
+  (gr_rect (start 81.28 139.7) (end 125.095 143.51) (layer "F.Mask") (width 0.15) (fill solid))
   (gr_line locked (start 226.06 143.51) (end 66.04 143.51) (layer "Edge.Cuts") (width 0.1))
   (gr_line (start 81.28 135.89) (end 81.28 102.87) (layer "Edge.Cuts") (width 0.1))
@@
   (gr_line (start 226.06 140.462) (end 66.04 140.462) (layer "User.6") (width 0.15))
   (gr_line locked (start 226.06 46.228) (end 66.04 46.228) (layer "User.6") (width 0.15))
+  (gr_text "2026" (at 182.245 113.03) (layer "B.Cu")
+    (effects (font (size 1.5 1.5) (thickness 0.3)) (justify mirror))
+  )
+  (gr_text "JP1: EXT ROM\nJP2: ACT LED" (at 189.865 135.255 90) (layer "F.SilkS")
+    (effects (font (size 1 1) (thickness 0.15)) (justify left))
+  )
+  (gr_text "Pozsar Zsolt" (at 114.3 82.55) (layer "F.SilkS")
+    (effects (font (size 1.5 1.5) (thickness 0.3)))
+  )
+  (gr_text "PEIX External interface box" (at 138.43 100.33) (layer "F.SilkS")
+    (effects (font (size 1.5 1.5) (thickness 0.3)))
+  )
   (segment (start 142.494 83.566) (end 141.732 82.804) (width 0.25) (layer "F.Cu") (net 1))
   (segment (start 140.97 78.74) (end 126.238 78.74) (width 0.25) (layer "F.Cu") (net 1))
@@
   (segment (start 84.074 67.564) (end 82.55 66.04) (width 0.25) (layer "B.Cu") (net 101))
   (segment (start 84.074 76.728) (end 84.074 67.564) (width 0.25) (layer "B.Cu") (net 101))
+  (segment (start 89.281 141.605) (end 125.349 141.605) (width 3.5) (layer "F.Cu") (net 102))
+  (segment (start 81.026 141.605) (end 89.154 141.605) (width 3.5) (layer "F.Cu") (net 102))
+  (segment (start 89.535 141.277) (end 89.535 131.773) (width 3.5) (layer "F.Cu") (net 102))
   (segment (start 89.408 141.732) (end 89.235 141.559) (width 3.5) (layer "B.Cu") (net 102))
   (segment (start 89.235 141.559) (end 89.235 132.055) (width 3.5) (layer "B.Cu") (net 102))
