File: PEIX External interface box/hardware/peix/peix.kicad_sch (KiCad schematic)
At the start: 45 parts, among them J1 Conn_01x08_Male, J2 Conn_01x03_Male, J3 Conn_01x04_Male, J4 Conn_01x08_Male, J5 Conn_01x08_Male, J6 Conn_01x08_Male, J7 DB9_Female_MountingHoles, U1 87C51, U2 27C64, U3 74LS573, U4 74LS08, U5 MAX232, U6 74LS245, U7 74LS245, U8 74LS245, Y1 11.0592 MHz

Commit message: 260215
Parts:
- R1, R2, R3, R4, R5, R6, R7, R8: footprint Resistor_THT:R_Axial_DIN0207_L6.3mm_D2.5mm_P5.08mm_Vertical -> Resistor_THT:R_Axial_DIN0207_L6.3mm_D2.5mm_P2.54mm_Vertical
Connections:
- net +5V: now also D1.2 (A), D2.2 (A), D3.2 (A); no longer R4.2, R5.1, R6.2
- net -RD: now also U4.12, U8.12 (B6); no longer U4.1, U8.11 (B7)
- net -WR: now also U4.13, U8.11 (B7); no longer U4.2, U8.12 (B6)
- net GNDD: no longer J7.0 (PAD)
- net at D2.1 (K): now also R5.1; no longer U4.8
- net at R5.2: now also U4.6; no longer D2.2 (A)
- net at JP2.1 (A), U1.28 (PC7): now also J2.1 (Pin_1); no longer J2.3 (Pin_3)
- net at D3.1 (K): now also R6.2; no longer U4.11
- net at U1.11 (PD1), U5.11 (T1IN): now also U4.10, U4.9; no longer U4.12, U4.13
- net at U1.10 (PD0), U5.12 (R1OUT): now also U4.4, U4.5; no longer U4.10, U4.9
- net at U1.26 (PC5): now also J2.3 (Pin_3); no longer J2.1 (Pin_1)
- net at U6.19 (CE): now also U4.11; no longer U4.3
- net at D1.1 (K): now also R4.2; no longer U4.6
- net at R4.1: now also U4.3; no longer D1.2 (A)
- net at R6.1: now also U4.8; no longer D3.2 (A)
- new net: JP2.2 (C), U4.1, U4.2
- new net Earth: J7.0 (PAD)
Other:
- note added: "A8 A9 A10 A11 A12 ALE -RD -WR"
- note added: "PC7 PC6 PC5"
- note removed: "A8 A9 A10 A11 A12 ALE -WR -RD"
- note removed: "PC5 PC6 PC7"
- moved on the sheet: D1, D2, D3, J2, R4, R5, R6

Commit message: 260216
Connections:
- net -RD: now also U4.9; no longer U4.12
- net -WR: now also U4.10; no longer U4.13
- net at R5.2: now also U4.3; no longer U4.6
- net at U1.11 (PD1), U5.11 (T1IN): now also U4.4, U4.5; no longer U4.10, U4.9
- net at R6.1: now also U4.6; no longer U4.8
- net at U1.10 (PD0), U5.12 (R1OUT): now also U4.1, U4.2; no longer U4.4, U4.5
- net at U6.19 (CE): now also U4.8; no longer U4.11
- net at R4.1: now also U4.11; no longer U4.3
- new net: JP2.2 (C), U4.12, U4.13
Changed lines of the file:
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@@
   (symbol (lib_id "power:GNDD") (at 173.355 182.245 0) (unit 1)
     (in_bom yes) (on_board yes) (fields_autoplaced)
-    (property "Reference" "#PWR023" (id 0) (at 173.355 188.595 0)
+    (property "Reference" "#PWR024" (id 0) (at 173.355 188.595 0)
       (effects (font (size 1.27 1.27)) hide)
     )
@@
     (pin "2")
   )
-  (symbol (lib_id "74xx:74LS08") (at 120.015 175.895 0) (unit 3)
+  (symbol (lib_id "74xx:74LS08") (at 120.015 175.895 0) (unit 2)
     (in_bom yes) (on_board yes)
     (property "Reference" "U4" (id 0) (at 113.665 175.895 0))
@@
   (symbol (lib_id "power:+5V") (at 173.355 154.94 0) (mirror y) (unit 1)
     (in_bom yes) (on_board yes)
-    (property "Reference" "#PWR022" (id 0) (at 173.355 158.75 0)
+    (property "Reference" "#PWR023" (id 0) (at 173.355 158.75 0)
       (effects (font (size 1.27 1.27)) hide)
     )
@@
     (pin "2")
   )
-  (symbol (lib_id "74xx:74LS08") (at 137.16 66.04 0) (unit 4)
+  (symbol (lib_id "74xx:74LS08") (at 137.16 66.04 0) (unit 3)
     (in_bom yes) (on_board yes)
     (property "Reference" "U4" (id 0) (at 133.35 60.325 0))
@@
     (pin "1")
   )
-  (symbol (lib_id "74xx:74LS08") (at 120.015 158.115 0) (unit 1)
+  (symbol (lib_id "74xx:74LS08") (at 120.015 158.115 0) (unit 4)
     (in_bom yes) (on_board yes)
     (property "Reference" "U4" (id 0) (at 113.665 158.115 0))
@@
   (symbol (lib_id "power:Earth") (at 172.72 233.68 0) (unit 1)
     (in_bom yes) (on_board yes) (fields_autoplaced)
-    (property "Reference" "#PWR0101" (id 0) (at 172.72 240.03 0)
+    (property "Reference" "#PWR022" (id 0) (at 172.72 240.03 0)
       (effects (font (size 1.27 1.27)) hide)
     )
@@
     (pin "2")
   )
-  (symbol (lib_id "74xx:74LS08") (at 120.015 167.005 0) (unit 2)
+  (symbol (lib_id "74xx:74LS08") (at 120.015 167.005 0) (unit 1)
     (in_bom yes) (on_board yes)
     (property "Reference" "U4" (id 0) (at 113.665 167.005 0))
@@
       (reference "#PWR021") (unit 1) (value "GNDD") (footprint "")
     )
+    (path "/dedf885d-1cd1-49a8-b7ec-ff2b60facf97"
+      (reference "#PWR022") (unit 1) (value "Earth") (footprint "")
+    )
     (path "/7b414570-ce45-41cb-a313-ffbd1c4da6dd"
-      (reference "#PWR022") (unit 1) (value "+5V") (footprint "")
+      (reference "#PWR023") (unit 1) (value "+5V") (footprint "")
     )
     (path "/1b8242f1-89e0-432c-9ee0-1fe9efa49474"
-      (reference "#PWR023") (unit 1) (value "GNDD") (footprint "")
-    )
-    (path "/dedf885d-1cd1-49a8-b7ec-ff2b60facf97"
-      (reference "#PWR0101") (unit 1) (value "Earth") (footprint "")
+      (reference "#PWR024") (unit 1) (value "GNDD") (footprint "")
     )
     (path "/fc8001d8-72e6-41ee-b3bf-0966ff2f4855"
@@
       (reference "U3") (unit 1) (value "74LS573") (footprint "Package_DIP:DIP-20_W7.62mm_LongPads")
     )
+    (path "/f33ff044-8785-49e0-ac11-52da7985dccf"
+      (reference "U4") (unit 1) (value "74LS08") (footprint "Package_DIP:DIP-14_W7.62mm_LongPads")
+    )
+    (path "/607c2fb4-1042-41a8-9550-a30d4985cad6"
+      (reference "U4") (unit 2) (value "74LS08") (footprint "Package_DIP:DIP-14_W7.62mm_LongPads")
+    )
+    (path "/96a9c403-6146-4a86-9af0-b33783808bec"
+      (reference "U4") (unit 3) (value "74LS08") (footprint "Package_DIP:DIP-14_W7.62mm_LongPads")
+    )
     (path "/da6e6ede-e5f4-41e8-9589-91eff309c139"
-      (reference "U4") (unit 1) (value "74LS08") (footprint "Package_DIP:DIP-14_W7.62mm_LongPads")
-    )
-    (path "/f33ff044-8785-49e0-ac11-52da7985dccf"
-      (reference "U4") (unit 2) (value "74LS08") (footprint "Package_DIP:DIP-14_W7.62mm_LongPads")
-    )
-    (path "/607c2fb4-1042-41a8-9550-a30d4985cad6"
-      (reference "U4") (unit 3) (value "74LS08") (footprint "Package_DIP:DIP-14_W7.62mm_LongPads")
-    )
-    (path "/96a9c403-6146-4a86-9af0-b33783808bec"
       (reference "U4") (unit 4) (value "74LS08") (footprint "Package_DIP:DIP-14_W7.62mm_LongPads")
     )

Commit message: 260216
Other:
- moved on the sheet: U4E
Changed lines of the file:
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@@
   (title_block
     (title "Control and communication card")
-    (date "2026-02-13")
+    (date "2026-02-16")
     (rev "1.0")
     (company "Pozsar Zsolt")
@@
   (junction (at 83.82 264.795) (diameter 0) (color 0 0 0 0)
   )
+  (junction (at 168.91 189.23) (diameter 0) (color 0 0 0 0)
+  )
   (junction (at 152.4 111.125) (diameter 0) (color 0 0 0 0)
   )
@@
   )
   (junction (at 60.96 133.35) (diameter 0) (color 0 0 0 0)
+  )
+  (junction (at 168.91 163.195) (diameter 0) (color 0 0 0 0)
   )
   (junction (at 152.4 67.945) (diameter 0) (color 0 0 0 0)
@@
     (stroke (width 0) (type default) (color 0 0 0 0))
   )
+  (wire (pts (xy 168.91 163.195) (xy 175.26 163.195))
+    (stroke (width 0) (type default) (color 0 0 0 0))
+  )
   (wire (pts (xy 152.4 153.67) (xy 150.495 153.67))
     (stroke (width 0) (type default) (color 0 0 0 0))
@@
     (stroke (width 0) (type default) (color 0 0 0 0))
   )
+  (wire (pts (xy 168.91 189.23) (xy 175.26 189.23))
+    (stroke (width 0) (type default) (color 0 0 0 0))
+  )
   (wire (pts (xy 76.2 80.645) (xy 88.9 80.645))
     (stroke (width 0) (type default) (color 0 0 0 0))
@@
     (stroke (width 0) (type default) (color 0 0 0 0))
   )
+  (wire (pts (xy 168.91 163.195) (xy 168.91 163.83))
+    (stroke (width 0) (type default) (color 0 0 0 0))
+  )
   (wire (pts (xy 60.96 238.125) (xy 60.96 238.76))
     (stroke (width 0) (type default) (color 0 0 0 0))
@@
     (stroke (width 0) (type default) (color 0 0 0 0))
   )
-  (wire (pts (xy 173.355 154.94) (xy 173.355 156.21))
+  (wire (pts (xy 168.91 162.56) (xy 168.91 163.195))
     (stroke (width 0) (type default) (color 0 0 0 0))
   )
@@
     (stroke (width 0) (type default) (color 0 0 0 0))
   )
-  (wire (pts (xy 173.355 181.61) (xy 173.355 182.245))
+  (wire (pts (xy 168.91 189.23) (xy 168.91 189.865))
     (stroke (width 0) (type default) (color 0 0 0 0))
   )
@@
   (label "A9" (at 128.27 121.285 0)
     (effects (font (size 1.27 1.27)) (justify left bottom))
+  )
+  (global_label "J8{slash}a2" (shape input) (at 175.26 189.23 0) (fields_autoplaced)
+    (effects (font (size 1.27 1.27)) (justify left))
+    (property "Intersheet References" "${INTERSHEET_REFS}" (id 0) (at 183.5393 189.1506 0)
+      (effects (font (size 1.27 1.27)) (justify left) hide)
+    )
+  )
+  (global_label "J8{slash}a4" (shape input) (at 175.26 163.195 0) (fields_autoplaced)
+    (effects (font (size 1.27 1.27)) (justify left))
+    (property "Intersheet References" "${INTERSHEET_REFS}" (id 0) (at 183.5393 163.1156 0)
+      (effects (font (size 1.27 1.27)) (justify left) hide)
+    )
   )
   (symbol (lib_id "power:GNDD") (at 21.59 22.225 270) (unit 1)
@@
     (pin "2")
   )
-  (symbol (lib_id "power:GNDD") (at 173.355 182.245 0) (unit 1)
+  (symbol (lib_id "power:GNDD") (at 168.91 189.865 0) (unit 1)
     (in_bom yes) (on_board yes) (fields_autoplaced)
-    (property "Reference" "#PWR024" (id 0) (at 173.355 188.595 0)
-      (effects (font (size 1.27 1.27)) hide)
-    )
-    (property "Value" "GNDD" (id 1) (at 173.355 187.325 0)
-      (effects (font (size 1.27 1.27)) hide)
-    )
-    (property "Footprint" "" (id 2) (at 173.355 182.245 0)
-      (effects (font (size 1.27 1.27)) hide)
-    )
-    (property "Datasheet" "" (id 3) (at 173.355 182.245 0)
+    (property "Reference" "#PWR024" (id 0) (at 168.91 196.215 0)
+      (effects (font (size 1.27 1.27)) hide)
+    )
+    (property "Value" "GNDD" (id 1) (at 168.91 194.945 0)
+      (effects (font (size 1.27 1.27)) hide)
+    )
+    (property "Footprint" "" (id 2) (at 168.91 189.865 0)
+      (effects (font (size 1.27 1.27)) hide)
+    )
+    (property "Datasheet" "" (id 3) (at 168.91 189.865 0)
       (effects (font (size 1.27 1.27)) hide)
     )
@@
     (pin "4")
   )
-  (symbol (lib_id "74xx:74LS08") (at 173.355 168.91 0) (unit 5)
-    (in_bom yes) (on_board yes)
-    (property "Reference" "U4" (id 0) (at 169.545 163.195 0))
-    (property "Value" "74LS08" (id 1) (at 173.355 175.26 0)
-      (effects (font (size 1.6 1.6) bold) hide)
-    )
-    (property "Footprint" "Package_DIP:DIP-14_W7.62mm_LongPads" (id 2) (at 173.355 168.91 0)
-      (effects (font (size 1.27 1.27)) hide)
-    )
-    (property "Datasheet" "http://www.ti.com/lit/gpn/sn74LS08" (id 3) (at 173.355 168.91 0)
+  (symbol (lib_id "74xx:74LS08") (at 168.91 176.53 0) (unit 5)
+    (in_bom yes) (on_board yes)
+    (property "Reference" "U4" (id 0) (at 172.72 167.005 0))
+    (property "Value" "74LS08" (id 1) (at 158.115 176.53 0)
+      (effects (font (size 1.6 1.6) bold))
+    )
+    (property "Footprint" "Package_DIP:DIP-14_W7.62mm_LongPads" (id 2) (at 168.91 176.53 0)
+      (effects (font (size 1.27 1.27)) hide)
+    )
+    (property "Datasheet" "http://www.ti.com/lit/gpn/sn74LS08" (id 3) (at 168.91 176.53 0)
       (effects (font (size 1.27 1.27)) hide)
     )
@@
     (in_bom yes) (on_board yes)
     (property "Reference" "U4" (id 0) (at 113.665 175.895 0))
-    (property "Value" "74LS08" (id 1) (at 120.015 182.245 0)
-      (effects (font (size 1.6 1.6) bold) hide)
+    (property "Value" "74LS08" (id 1) (at 120.015 182.88 0)
+      (effects (font (size 1.6 1.6) bold))
     )
     (property "Footprint" "Package_DIP:DIP-14_W7.62mm_LongPads" (id 2) (at 120.015 175.895 0)
@@
     (pin "1")
   )
-  (symbol (lib_id "power:+5V") (at 173.355 154.94 0) (mirror y) (unit 1)
-    (in_bom yes) (on_board yes)
-    (property "Reference" "#PWR023" (id 0) (at 173.355 158.75 0)
-      (effects (font (size 1.27 1.27)) hide)
-    )
-    (property "Value" "+5V" (id 1) (at 172.72 150.495 0))
-    (property "Footprint" "" (id 2) (at 173.355 154.94 0)
-      (effects (font (size 1.27 1.27)) hide)
-    )
-    (property "Datasheet" "" (id 3) (at 173.355 154.94 0)
-      (effects (font (size 1.27 1.27)) hide)
-    )
+  (symbol (lib_id "power:+5V") (at 168.91 162.56 0) (mirror y) (unit 1)
+    (in_bom yes) (on_board yes)
+    (property "Reference" "#PWR023" (id 0) (at 168.91 166.37 0)
+      (effects (font (size 1.27 1.27)) hide)
+    )
+    (property "Value" "+5V" (id 1) (at 168.275 158.115 0))
+    (property "Footprint" "" (id 2) (at 168.91 162.56 0)
+      (effects (font (size 1.27 1.27)) hide)
+    )
+    (property "Datasheet" "" (id 3) (at 168.91 162.56 0)
+      (effects (font (size 1.27 1.27)) hide)
+    )
