File: Zacchaeus computer/hardware/PMAN-IF Interface module/pman-if/pman-if-3.kicad_sch (KiCad schematic)
At the start: 35 parts, among them J5 Conn_01x04_Pin, J6 Conn_01x08_Pin, J7 Conn_01x05_Pin, U10 74LS273, U11 74LS273, U6 74HCT4066, U7 74HCT4066, U8 74LS14, U9 74LS245

Commit message: 260329
Parts:
- removed R10, R11, R12, R13, R14, R15, R16, R17: 1M, Resistor_THT:R_Axial_DIN0207_L6.3mm_D2.5mm_P5.08mm_Vertical, symbol Device:R
- removed R2, R3, R4, R5, R6, R7, R8, R9: R, Resistor_THT:R_Axial_DIN0207_L6.3mm_D2.5mm_P5.08mm_Vertical, symbol Device:R
- added RN2: 4x1k, Resistor_THT:R_Array_SIP5, symbol Device:R_Network04
- J5: footprint Connector_PinHeader_2.54mm:PinHeader_1x04_P2.54mm_Horizontal -> Connector_PinHeader_2.54mm:PinHeader_1x04_P2.54mm_Vertical
- J6: footprint Connector_PinHeader_2.54mm:PinHeader_1x08_P2.54mm_Horizontal -> Connector_PinHeader_2.54mm:PinHeader_1x08_P2.54mm_Vertical
- J7: footprint Connector_PinHeader_2.54mm:PinHeader_1x05_P2.54mm_Horizontal -> Connector_PinHeader_2.54mm:PinHeader_1x05_P2.54mm_Vertical
- U6, U7, U8: footprint Package_DIP:DIP-14_W7.62mm -> Package_DIP:DIP-14_W7.62mm_Socket_LongPads
Connections:
- net +5VD: now also RN2.1 (common)
- net at J5.3 (Pin_3): now also C7.2, U8.5, RN2.4 (R3)
- net at J6.8 (Pin_8): now also U6.9; no longer U6.10
- net at U6.1, U6.4: now also U6.11, U6.8; no longer U6.11, U6.8
- net at U10.12 (Q4): now also U6.6; no longer U6.12
- net at J6.3 (Pin_3): now also U7.2; no longer U7.3
- net at J6.4 (Pin_4): now also U7.3; no longer U7.2
- net at J6.7 (Pin_7): now also U6.10; no longer U6.9
- net at C8.2, U8.9: now also J5.4 (Pin_4), RN2.5 (R4)
- net at U10.15 (Q5): now also U6.12; no longer U6.6
- net at J5.1 (Pin_1): now also C10.1, U8.1, RN2.2 (R1)
- net at J5.2 (Pin_2): now also C9.1, U8.3, RN2.3 (R2)
- net at U7.11, U7.8: now also U7.1, U7.4; no longer U7.1, U7.4
- net at U10.2 (Q0): now also U7.5; no longer U7.13
- net at U10.5 (Q1): now also U7.13; no longer U7.5
