File: Zacchaeus computer/hardware/PMAN-IF Interface module/pman-if/pman-if.kicad_sch (KiCad schematic)
At the start: 10 parts, among them J1 Conn_02x40_Top_Bottom, SW2 SW_DIP_x08, U1 74LS08, U2 74LS138, U3 74HCT688, U4 74LS245, U6 74LS32

Commit message: 260329
Parts:
- removed C2: 47u, Capacitor_THT:CP_Radial_D8.0mm_P3.80mm, symbol Device:C_Polarized
- removed J1: Conn_02x40_Top_Bottom, pinhead:PinHeader_2x40_P2.54mm_Vertical_Top_Bottom, symbol Connector_Generic:Conn_02x40_Top_Bottom
- removed R1: R, symbol Device:R
- removed RN1: 8x1k, Resistor_THT:R_Array_SIP9, symbol Device:R_Network08
- removed SW2: SW_DIP_x08, Package_DIP:DIP-16_W7.62mm_LongPads, symbol Switch:SW_DIP_x08
- removed U1: 74LS08, symbol 74xx:74LS08
- removed U2: 74LS138, symbol 74xx:74LS138
- removed U3: 74HCT688, Package_DIP:DIP-20_W7.62mm_Socket_LongPads, symbol 74xx:74HCT688
- removed U4: 74LS245, symbol 74xx:74LS245
- removed U6: 74LS32, Package_DIP:DIP-14_W7.62mm_Socket_LongPads, symbol 74xx:74LS32
Connections:
- no-connect marks 58 -> 9
Other:
- added sheet Address decoder (pman-if-1.kicad_sch)
- added sheet PMAN-DP interface (pman-if-2.kicad_sch)
- added sheet PMAN-SW interface (pman-if-3.kicad_sch)
- note removed: "I/O address"
- title: PMAN-IF - Manual control panel interface modue -> PMAN-IF - Manual control panel interface module

Commit message: 260330
Other:
- sheet Address decoder renamed address decoder
- sheet PMAN-DP interface renamed display interface
- sheet PMAN-SW interface renamed switch interface
Changed lines of the file:
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@@
 	(wire
 		(pts
-			(xy 138.43 134.62) (xy 143.51 134.62)
+			(xy 138.43 130.81) (xy 143.51 130.81)
 		)
 		(stroke
@@
 	(sheet
 		(at 98.425 116.84)
-		(size 40.005 31.115)
+		(size 40.005 17.145)
 		(exclude_from_sim no)
 		(in_bom yes)
@@
 			(color 0 0 0 0.0000)
 		)
-		(property "Sheetname" "PMAN-SW interface"
-			(at 98.044 150.876 0)
+		(property "Sheetname" "switch interface"
+			(at 98.298 136.144 0)
 			(effects
 				(font
@@
 		)
 		(pin "BLANK" output
-			(at 138.43 134.62 0)
+			(at 138.43 130.81 0)
 			(effects
 				(font
@@
 	)
 	(sheet
-		(at 111.125 44.45)
-		(size 76.835 31.75)
+		(at 111.125 57.15)
+		(size 76.835 19.05)
 		(exclude_from_sim no)
 		(in_bom yes)
 		(on_board yes)
 		(dnp no)
-		(fields_autoplaced yes)
 		(stroke
 			(width 0.1524)
@@
 			(color 0 0 0 0.0000)
 		)
-		(property "Sheetname" "Address decoder"
-			(at 110.4134 76.2 90)
-			(show_name yes)
+		(property "Sheetname" "address decoder"
+			(at 110.998 56.642 0)
 			(effects
 				(font
@@
 		)
 		(property "Sheetfile" "pman-if-1.kicad_sch"
-			(at 188.5446 76.2 90)
+			(at 188.5446 88.9 90)
 			(effects
 				(font
@@
 	(sheet
 		(at 143.51 116.84)
-		(size 37.465 30.48)
+		(size 37.465 17.145)
 		(exclude_from_sim no)
 		(in_bom yes)
@@
 			(color 0 0 0 0.0000)
 		)
-		(property "Sheetname" "PMAN-DP interface"
-			(at 143.51 149.479 0)
+		(property "Sheetname" "display interface"
+			(at 143.256 136.398 0)
 			(effects
 				(font
@@
 		)
 		(pin "BLANK" input
-			(at 143.51 134.62 180)
-			(effects
-				(font
+			(at 143.51 130.81 180)
+			(effects
+				(font
