File: Zacchaeus computer/hardware/PMAN-IF Interface module/pman-if/pman-if.kicad_pcb (KiCad board)
At the start: 2 copper layers, 102.6 x 72.4 mm, 56 parts, among them J1 Conn_02x40_Top_Bottom, J2 Screw_Terminal_01x02, J3 Screw_Terminal_01x02, J4 Screw_Terminal_01x02, J5 Screw_Terminal_01x02, SW1 SW_DIP_x08, U1 74LS32, U2 74LS273, U3 74HCT688, U4 MC3340P, U5 7809, U6 LM386

Commit message: 260329
Parts:
- removed C17: 100u, Capacitor_THT:CP_Radial_D8.0mm_P3.80mm
- removed C18: **, Capacitor_THT:C_Disc_D5.0mm_W2.5mm_P5.00mm
- removed C19: 50n, Capacitor_THT:C_Disc_D5.0mm_W2.5mm_P5.00mm
- removed C20: 220u, Capacitor_THT:CP_Radial_D8.0mm_P3.80mm
- removed D1: 1N5395, Diode_THT:D_DO-15_P5.08mm_Vertical_KathodeUp
- removed D2: LED, LED_THT:LED_Rectangular_W5.0mm_H2.0mm_Horizontal_O1.27mm_Z1.0mm
- removed R18: 47k-100k, Resistor_THT:R_Axial_DIN0207_L6.3mm_D2.5mm_P2.54mm_Vertical
- removed R19: 470, Resistor_THT:R_Axial_DIN0207_L6.3mm_D2.5mm_P2.54mm_Vertical
- removed R20: *, Resistor_THT:R_Axial_DIN0207_L6.3mm_D2.5mm_P2.54mm_Vertical
- removed R21: 10, Resistor_THT:R_Axial_DIN0207_L6.3mm_D2.5mm_P2.54mm_Vertical
- added J6: Conn_01x08_Pin, Connector_PinHeader_2.54mm:PinHeader_1x08_P2.54mm_Horizontal, F.Cu at (100.3, 160.0)
- added J7: Conn_01x05_Pin, Connector_PinHeader_2.54mm:PinHeader_1x05_P2.54mm_Horizontal, F.Cu at (103.5, 174.6)
- added U10: 74LS273, Package_DIP:DIP-20_W7.62mm_Socket_LongPads, F.Cu at (263.4, 53.5)
- added U11: 74LS273, Package_DIP:DIP-20_W7.62mm_Socket_LongPads, F.Cu at (275.1, 53.5)
- added U7: 74HCT4066, Package_DIP:DIP-14_W7.62mm, F.Cu at (262.0, 80.5)
- added U8: 74LS14, Package_DIP:DIP-14_W7.62mm, F.Cu at (272.8, 80.5)
- added U9: 74LS245, Package_DIP:DIP-20_W7.62mm_Socket_LongPads, F.Cu at (251.7, 53.5)
- C1: value 100n -> 47u; footprint Capacitor_THT:C_Disc_D5.0mm_W2.5mm_P5.00mm -> Capacitor_THT:CP_Radial_D8.0mm_P3.80mm
- C10: value 1n -> 100; footprint Capacitor_THT:C_Disc_D5.0mm_W2.5mm_P2.50mm -> Capacitor_THT:C_Disc_D5.0mm_W2.5mm_P5.00mm
- C12: value 50n -> 100n
- C13: value 1n -> 100n; footprint Capacitor_THT:C_Disc_D5.0mm_W2.5mm_P2.50mm -> Capacitor_THT:C_Disc_D5.0mm_W2.5mm_P5.00mm
- C14: value 220u -> 100n; footprint Capacitor_THT:CP_Radial_D8.0mm_P3.80mm -> Capacitor_THT:C_Disc_D5.0mm_W2.5mm_P5.00mm
- C15, C6: value 1u Ta -> 100n; footprint Capacitor_THT:CP_Radial_Tantal_D5.0mm_P2.50mm -> Capacitor_THT:C_Disc_D5.0mm_W2.5mm_P5.00mm
- C2: value 47u -> 100n; footprint Capacitor_THT:CP_Radial_D8.0mm_P3.80mm -> Capacitor_THT:C_Disc_D5.0mm_W2.5mm_P5.00mm
- C5: value 10n -> 100n
- C7: value 100n -> 100
- C8: value 10u -> 100; footprint Capacitor_THT:CP_Radial_D5.0mm_P2.50mm -> Capacitor_THT:C_Disc_D5.0mm_W2.5mm_P5.00mm
- C9: value 220u -> 100; footprint Capacitor_THT:CP_Radial_D8.0mm_P3.80mm -> Capacitor_THT:C_Disc_D5.0mm_W2.5mm_P5.00mm
- J2: value Screw_Terminal_01x02 -> Conn_01x08_Pin; footprint TerminalBlock:TerminalBlock_MaiXu_MX126-5.0-02P_1x02_P5.00mm -> Connector_PinHeader_2.54mm:PinHeader_1x08_P2.54mm_Horizontal
- J3: value Screw_Terminal_01x02 -> Conn_01x05_Pin; footprint TerminalBlock:TerminalBlock_MaiXu_MX126-5.0-02P_1x02_P5.00mm -> Connector_PinHeader_2.54mm:PinHeader_1x05_P2.54mm_Horizontal
- J4: value Screw_Terminal_01x02 -> Conn_01x02_Pin; footprint TerminalBlock:TerminalBlock_MaiXu_MX126-5.0-02P_1x02_P5.00mm -> Connector_PinHeader_2.54mm:PinHeader_1x02_P2.54mm_Horizontal
- J5: value Screw_Terminal_01x02 -> Conn_01x04_Pin; footprint TerminalBlock:TerminalBlock_MaiXu_MX126-5.0-02P_1x02_P5.00mm -> Connector_PinHeader_2.54mm:PinHeader_1x04_P2.54mm_Horizontal
- R1: value 20k -> 1k; footprint Resistor_THT:R_Axial_DIN0207_L6.3mm_D2.5mm_P2.54mm_Vertical -> Resistor_THT:R_Axial_DIN0207_L6.3mm_D2.5mm_P5.08mm_Vertical
- R10, R11, R12, R13, R14, R15, R16, R17: value 10k -> 1M; footprint Resistor_THT:R_Axial_DIN0207_L6.3mm_D2.5mm_P2.54mm_Vertical -> Resistor_THT:R_Axial_DIN0207_L6.3mm_D2.5mm_P5.08mm_Vertical
- R2, R3, R4, R5, R6, R7, R8: value 20k -> R; footprint Resistor_THT:R_Axial_DIN0207_L6.3mm_D2.5mm_P2.54mm_Vertical -> Resistor_THT:R_Axial_DIN0207_L6.3mm_D2.5mm_P5.08mm_Vertical
- R9: value 10k -> R; footprint Resistor_THT:R_Axial_DIN0207_L6.3mm_D2.5mm_P2.54mm_Vertical -> Resistor_THT:R_Axial_DIN0207_L6.3mm_D2.5mm_P5.08mm_Vertical
- U1: value 74LS32 -> 74LS138; footprint Package_DIP:DIP-14_W7.62mm_Socket_LongPads -> Package_DIP:DIP-16_W7.62mm_LongPads
- U2: value 74LS273 -> 74LS138; footprint Package_DIP:DIP-20_W7.62mm_Socket_LongPads -> Package_DIP:DIP-16_W7.62mm_LongPads
- U4: value MC3340P -> 74LS20; footprint Package_DIP:DIP-8_W7.62mm_Socket_LongPads -> Package_DIP:DIP-14_W7.62mm
- U5: value 7809 -> 74LS245; footprint Package_TO_SOT_THT:TO-220-3_Horizontal_TabDown -> Package_DIP:DIP-20_W7.62mm_Socket_LongPads
- U6: value LM386 -> 74HCT4066; footprint Package_DIP:DIP-8_W7.62mm_Socket_LongPads -> Package_DIP:DIP-14_W7.62mm
- moved C9 142.7 mm to (243.1, 61.5)
- moved U5 132.1 mm to (138.4, 208.9), turned to 90 degrees
- moved C10 132.0 mm to (243.1, 65.5), turned to 0 degrees
- moved R9 131.5 mm to (292.7, 84.5), turned to 0 degrees
- moved R1 128.7 mm to (288.3, 114.9), turned to 0 degrees
- moved R10 127.6 mm to (292.7, 88.5), turned to 0 degrees
- moved J4 124.5 mm to (150.5, 174.6), turned to 90 degrees
- moved R11 123.8 mm to (292.7, 92.6), turned to 0 degrees
- moved U4 122.2 mm to (143.5, 190.5), turned to 90 degrees
- moved R14 121.4 mm to (301.4, 80.4), turned to 0 degrees
- moved R12 120.2 mm to (292.7, 96.6), turned to 0 degrees
- moved R2 119.7 mm to (284.0, 80.4), turned to 0 degrees
- moved R15 117.4 mm to (301.4, 84.5), turned to 0 degrees
- moved C13 117.3 mm to (243.1, 77.7)
- moved R13 116.7 mm to (292.7, 100.7), turned to 0 degrees
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Connections:
- net /-IORQ renamed /Address decoder/-IORQ
- net /A3 renamed /Address decoder/A3
- net /A4 renamed /Address decoder/A4
- net /A5 renamed /Address decoder/A5
- net /A6 renamed /Address decoder/A6
- net /A7 renamed /Address decoder/A7
- C1 pad 2: GNDA -> GNDD
- C10 pad 1: /+12VA -> Net-(C10-Pad1)
- C10 pad 2: GNDA -> GNDD
- C11 pad 1: +9VA -> +5VD
- C11 pad 2: GNDA -> GNDD
- C12 pad 1: Net-(U4-Roll-off) -> +5VD
- C12 pad 2: GNDA -> GNDD
- C13 pad 1: +9VA -> +5VD
- C13 pad 2: GNDA -> GNDD
- C14 pad 1: Net-(U4-Output) -> +5VD
- C14 pad 2: Net-(U6-+) -> GNDD
- C15 pad 1: +9VA -> +5VD
- C15 pad 2: GNDA -> GNDD
- C16 pad 1: GNDA -> +5VD
- C16 pad 2: +9VA -> GNDD
- C2 pad 2: GNDA -> GNDD
- C3 pad 1: GNDA -> +5VD
- C3 pad 2: +5VD -> GNDD
- C4 pad 2: GNDA -> GNDD
- C5 pad 1: GNDA -> +5VD
- C5 pad 2: Net-(C5-Pad2) -> GNDD
- C6 pad 1: Net-(C5-Pad2) -> +5VD
- C6 pad 2: Net-(J2-Pin_1) -> GNDD
- C7 pad 1: GNDA -> GNDD
- C7 pad 2: Net-(J3-Pin_1) -> Net-(C7-Pad2)
- C8 pad 1: Net-(J3-Pin_1) -> GNDD
- C8 pad 2: GNDA -> Net-(C8-Pad2)
- C9 pad 1: /+12VA -> Net-(C9-Pad1)
- C9 pad 2: GNDA -> GNDD
- J1 pad 14: /A2 -> /Address decoder/A2
- J1 pad 15: /A1 -> /Address decoder/A1
- J1 pad 16: /A0 -> /Address decoder/A0
- J1 pad 17: GNDA -> GNDD
- J1 pad 20: /RESET -> /Address decoder/-RESET
- J1 pad 24: /-WR -> /Address decoder/-WR
- J1 pad 25: unconnected-(J1-Pin_25-Pad25) -> /Address decoder/-RD
- J1 pad 27: /D0 -> /Address decoder/D0
- J1 pad 28: /D1 -> /Address decoder/D1
- J1 pad 29: /D2 -> /Address decoder/D2
- J1 pad 30: /D3 -> /Address decoder/D3
- J1 pad 31: /D4 -> /Address decoder/D4
- J1 pad 32: /D5 -> /Address decoder/D5
- J1 pad 33: /D6 -> /Address decoder/D6
- J1 pad 34: /D7 -> /Address decoder/D7
- J1 pad 57: GNDA -> GNDD
- J2 pad 2: GNDA -> Net-(J2-Pin_2)
- J3 pad 1: Net-(J3-Pin_1) -> /Address decoder/-WRSEL0
- J3 pad 2: GNDA -> /Address decoder/-WRSEL1
- J4 pad 1: /+12VA -> +5VD
- J4 pad 2: GNDA -> GNDD
- J5 pad 2: GNDA -> Net-(J5-Pin_2)
- R1 pad 1: Net-(R1-Pad1) -> Net-(U5-A->B)
- R1 pad 2: Net-(U2-Q0) -> +5VD
- R10 pad 1: Net-(R10-Pad1) -> GNDD
- R10 pad 2: Net-(R1-Pad1) -> Net-(J6-Pin_5)
- R11 pad 1: Net-(R11-Pad1) -> GNDD
- R11 pad 2: Net-(R10-Pad1) -> Net-(J6-Pin_6)
- R12 pad 1: Net-(R12-Pad1) -> GNDD
- R12 pad 2: Net-(R11-Pad1) -> Net-(J6-Pin_7)
- R13 pad 1: Net-(R13-Pad1) -> GNDD
- R13 pad 2: Net-(R12-Pad1) -> Net-(J6-Pin_8)
- R14 pad 1: Net-(R14-Pad1) -> Net-(J6-Pin_4)
- R14 pad 2: Net-(R13-Pad1) -> GNDD
- R15 pad 1: Net-(R15-Pad1) -> Net-(J6-Pin_3)
- R15 pad 2: Net-(R14-Pad1) -> GNDD
- R16 pad 1: Net-(R16-Pad1) -> Net-(J6-Pin_2)
- R16 pad 2: Net-(R15-Pad1) -> GNDD
- R17 pad 1: Net-(R16-Pad1) -> Net-(J6-Pin_1)
- R17 pad 2: Net-(C5-Pad2) -> GNDD
- R2 pad 1: Net-(R10-Pad1) -> +5VD
- R2 pad 2: Net-(U2-Q1) -> Net-(J5-Pin_3)
- R3 pad 1: Net-(R11-Pad1) -> +5VD
- R3 pad 2: Net-(U2-Q2) -> Net-(J5-Pin_4)
- R4 pad 1: Net-(R12-Pad1) -> Net-(J5-Pin_4)
- R4 pad 2: Net-(U2-Q3) -> Net-(C8-Pad2)
- R5 pad 1: Net-(R13-Pad1) -> Net-(J5-Pin_3)
- R5 pad 2: Net-(U2-Q4) -> Net-(C7-Pad2)
- R6 pad 1: Net-(R14-Pad1) -> Net-(J5-Pin_2)
- R6 pad 2: Net-(U2-Q5) -> Net-(C9-Pad1)
- R7 pad 1: Net-(R15-Pad1) -> Net-(J5-Pin_1)
- R7 pad 2: Net-(U2-Q6) -> Net-(C10-Pad1)
- R8 pad 1: Net-(R16-Pad1) -> Net-(J5-Pin_2)
- R8 pad 2: Net-(U2-Q7) -> +5VD
- R9 pad 1: Net-(R1-Pad1) -> Net-(J5-Pin_1)
- R9 pad 2: GNDA -> +5VD
- SW1 pad 1: GNDA -> GNDD
- SW1 pad 2: GNDA -> GNDD
- SW1 pad 3: GNDA -> GNDD
- SW1 pad 4: GNDA -> GNDD
- SW1 pad 5: GNDA -> GNDD
- SW1 pad 6: GNDA -> GNDD
- SW1 pad 7: GNDA -> GNDD
- SW1 pad 8: GNDA -> GNDD
- U1 pad 1: /-WR -> /Address decoder/A0
- U1 pad 10: GNDA -> /Address decoder/-WRSEL5
- U1 pad 11: unconnected-(U1-Pad11) -> /Address decoder/-WRSEL4
- U1 pad 12: GNDA -> /Address decoder/-WRSEL3
- U1 pad 13: GNDA -> /Address decoder/-WRSEL2
- U1 pad 14: +5VD -> /Address decoder/-WRSEL1
- U1 pad 2: Net-(U3-P=R) -> /Address decoder/A1
- U1 pad 3: Net-(U2-Cp) -> /Address decoder/A2
- U1 pad 4: GNDA -> Net-(U1-E1)
- U1 pad 5: GNDA -> /Address decoder/-WR
- U1 pad 6: unconnected-(U1-Pad6) -> Net-(RN1-R8)
- U1 pad 7: GNDA -> /Address decoder/-WRSEL7
- U1 pad 8: unconnected-(U1-Pad8) -> GNDD
- U1 pad 9: GNDA -> /Address decoder/-WRSEL6
- U2 pad 1: /RESET -> /Address decoder/A0
- U2 pad 10: GNDA -> /Address decoder/-RDSEL5
- U2 pad 11: Net-(U2-Cp) -> /Address decoder/-RDSEL4
- U2 pad 12: Net-(U2-Q4) -> /Address decoder/-RDSEL3
- U2 pad 13: /D4 -> /Address decoder/-RDSEL2
- U2 pad 14: /D5 -> /Address decoder/-RDSEL1
- U2 pad 15: Net-(U2-Q5) -> /Address decoder/-RDSEL0
- U2 pad 16: Net-(U2-Q6) -> +5VD
- U2 pad 2: Net-(U2-Q0) -> /Address decoder/A1
- U2 pad 3: /D0 -> /Address decoder/A2
- U2 pad 4: /D1 -> Net-(U1-E1)
- U2 pad 5: Net-(U2-Q1) -> /Address decoder/-RD
- U2 pad 6: Net-(U2-Q2) -> Net-(RN1-R8)
- U2 pad 7: /D2 -> /Address decoder/-RDSEL7
- U2 pad 8: /D3 -> GNDD
- U2 pad 9: Net-(U2-Q3) -> /Address decoder/-RDSEL6
- U3 pad 10: GNDA -> GNDD
- U3 pad 19: Net-(U3-P=R) -> Net-(U1-E1)
- U3 pad 2: Net-(RN1-R8) -> GNDD
- U3 pad 3: /A0 -> GNDD
- U3 pad 4: Net-(RN1-R7) -> GNDD
- U3 pad 5: /A1 -> GNDD
- U3 pad 6: Net-(RN1-R6) -> GNDD
- U3 pad 7: /A2 -> GNDD
- U4 pad 1: Net-(J2-Pin_1) -> /Address decoder/-WRSEL0
- U4 pad 2: Net-(J3-Pin_1) -> /Address decoder/-WRSEL1
- U4 pad 3: GNDA -> (no net)
- U4 pad 4: unconnected-(U4-N.C.-Pad4) -> /Address decoder/-WRSEL2
- U4 pad 5: unconnected-(U4-N.C.-Pad5) -> /Address decoder/-WRSEL3
- U4 pad 6: Net-(U4-Roll-off) -> Net-(U4-Pad10)
- U4 pad 7: Net-(U4-Output) -> GNDD
- U4 pad 8: +9VA -> Net-(U5-CE)
- U5 pad 1: /+12VA -> Net-(U5-A->B)
- U5 pad 2: GNDA -> /Address decoder/D0
- U5 pad 3: +9VA -> /Address decoder/D1
- U6 pad 1: Net-(R20-Pad2) -> Net-(U6-Pad1)
- U6 pad 2: GNDA -> Net-(J6-Pin_5)
- U6 pad 3: Net-(U6-+) -> Net-(J6-Pin_6)
- U6 pad 4: GNDA -> Net-(U6-Pad1)
- U6 pad 6: +9VA -> Net-(U10-Q5)
- U6 pad 7: unconnected-(U6-BYPASS-Pad7) -> GNDD
- U6 pad 8: Net-(C18-Pad2) -> Net-(U6-Pad1)
Routing:
- net GNDA: track 595.5 -> 0.00 mm
- net GNDD: track 0.00 -> 276.1 mm, vias 0 -> 1
- net +9VA: track 123.5 -> 0.00 mm
- net +5VD: track 112.3 -> 8.96 mm
- net Net-(RN1-R8): track 49.8 -> 0.00 mm
- net /+12VA: track 44.7 -> 0.00 mm
- net Net-(U2-Cp): track 44.5 -> 0.00 mm, vias 2 -> 0
- net Net-(RN1-R7): track 42.1 -> 0.00 mm
- net /A0: track 38.9 -> 0.00 mm
- net Net-(U2-Q7): track 37.3 -> 0.00 mm, vias 2 -> 0
- net /-WR: track 36.5 -> 0.00 mm
- net Net-(RN1-R6): track 35.6 -> 0.00 mm
- net /D7: track 35.0 -> 0.00 mm, vias 2 -> 0
- net /A1: track 32.4 -> 0.00 mm
- net /Address decoder/-IORQ: track 69.3 -> 37.2 mm, vias 1 -> 0
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Other:
- board text removed: "PCOX"
- board text removed: "Pozsár Zsolt 2025"
- board text removed: "analog GND"
- board text removed: "digital GND"

Commit message: 260329
Parts:
- removed R10, R11, R12, R13, R14, R15, R16, R17: 1M, Resistor_THT:R_Axial_DIN0207_L6.3mm_D2.5mm_P5.08mm_Vertical
- removed R2, R3, R4, R5, R6, R7, R8, R9: R, Resistor_THT:R_Axial_DIN0207_L6.3mm_D2.5mm_P5.08mm_Vertical
- added RN2: 4x1k, Resistor_THT:R_Array_SIP5, F.Cu at (190.0, 90.2)
- J2: footprint Connector_PinHeader_2.54mm:PinHeader_1x08_P2.54mm_Horizontal -> Connector_PinHeader_2.54mm:PinHeader_1x07_P2.54mm_Vertical
- J3, J7: footprint Connector_PinHeader_2.54mm:PinHeader_1x05_P2.54mm_Horizontal -> Connector_PinHeader_2.54mm:PinHeader_1x05_P2.54mm_Vertical
- J4: footprint Connector_PinHeader_2.54mm:PinHeader_1x02_P2.54mm_Horizontal -> Connector_PinHeader_2.54mm:PinHeader_1x02_P2.54mm_Vertical
- J5: footprint Connector_PinHeader_2.54mm:PinHeader_1x04_P2.54mm_Horizontal -> Connector_PinHeader_2.54mm:PinHeader_1x04_P2.54mm_Vertical
- J6: footprint Connector_PinHeader_2.54mm:PinHeader_1x08_P2.54mm_Horizontal -> Connector_PinHeader_2.54mm:PinHeader_1x08_P2.54mm_Vertical
- SW1, U1, U2: footprint Package_DIP:DIP-16_W7.62mm_LongPads -> Package_DIP:DIP-16_W7.62mm_Socket_LongPads
- U4, U6, U7, U8: footprint Package_DIP:DIP-14_W7.62mm -> Package_DIP:DIP-14_W7.62mm_Socket_LongPads
- moved R1 156.1 mm to (132.7, 127.6), turned to 90 degrees
- moved U11 139.9 mm to (136.7, 73.7), turned to 90 degrees
- moved U10 131.8 mm to (136.7, 89.5), turned to 90 degrees
- moved U9 128.7 mm to (136.7, 111.1), turned to 90 degrees
- moved J7 120.5 mm to (141.7, 60.3)
- moved J6 120.3 mm to (167.8, 60.3)
- moved C6 113.7 mm to (129.5, 120.7), turned to -90 degrees
- moved C14 112.6 mm to (132.8, 104.8), turned to -90 degrees
- moved U8 106.8 mm to (170.3, 110.5), turned to 90 degrees
- moved J3 104.5 mm to (110.6, 60.3)
- moved J5 103.5 mm to (194.4, 92.7), turned to 0 degrees
- moved J4 100.3 mm to (194.4, 84.5), turned to 0 degrees
- moved C16 99.6 mm to (132.8, 67.3), turned to -90 degrees
- moved C15 96.4 mm to (132.8, 83.2), turned to -90 degrees
- moved U7 92.0 mm to (170.3, 73.7), turned to 90 degrees
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Connections:
- C10 pad 1: Net-(C10-Pad1) -> Net-(J5-Pin_1)
- C7 pad 2: Net-(C7-Pad2) -> Net-(J5-Pin_3)
- C8 pad 2: Net-(C8-Pad2) -> Net-(J5-Pin_4)
- C9 pad 1: Net-(C9-Pad1) -> Net-(J5-Pin_2)
- U6 pad 10: Net-(J6-Pin_8) -> Net-(J6-Pin_7)
- U6 pad 12: Net-(U10-Q4) -> Net-(U10-Q5)
- U6 pad 6: Net-(U10-Q5) -> Net-(U10-Q4)
- U6 pad 9: Net-(J6-Pin_7) -> Net-(J6-Pin_8)
- U7 pad 13: Net-(U10-Q0) -> Net-(U10-Q1)
- U7 pad 2: Net-(J6-Pin_4) -> Net-(J6-Pin_3)
- U7 pad 3: Net-(J6-Pin_3) -> Net-(J6-Pin_4)
- U7 pad 5: Net-(U10-Q1) -> Net-(U10-Q0)
- U8 pad 1: Net-(C10-Pad1) -> Net-(J5-Pin_1)
- U8 pad 3: Net-(C9-Pad1) -> Net-(J5-Pin_2)
- U8 pad 5: Net-(C7-Pad2) -> Net-(J5-Pin_3)
- U8 pad 9: Net-(C8-Pad2) -> Net-(J5-Pin_4)
Routing:
- net +5VD: track 8.96 -> 532.1 mm, vias 0 -> 5
- net GNDD: track 276.1 -> 634.7 mm, vias 1 -> 4
- net /Address decoder/D4: track 0.00 -> 68.9 mm, vias 0 -> 2
- net /Address decoder/D5: track 0.00 -> 63.8 mm
- net /Address decoder/D2: track 0.00 -> 62.4 mm, vias 0 -> 2
- net /Address decoder/D3: track 0.00 -> 62.3 mm, vias 0 -> 2
- net /Address decoder/D1: track 0.00 -> 56.6 mm
- net /Address decoder/D0: track 0.00 -> 56.3 mm
- net /Address decoder/A7: track 41.6 -> 0.00 mm
- net Net-(J5-Pin_1): track 0.00 -> 38.2 mm
- net /Address decoder/-IORQ: track 37.2 -> 0.00 mm
- net /Address decoder/A6: track 35.7 -> 0.00 mm
- net /Address decoder/D7: track 0.00 -> 33.6 mm
- net /Address decoder/D6: track 0.00 -> 33.6 mm
- net Net-(J5-Pin_2): track 0.00 -> 31.8 mm
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Other:
- board size 102.6 x 72.4 mm -> 102.6 x 85.1 mm

Commit message: 260329
Parts:
- moved J2 53.0 mm to (141.6, 115.6), turned to 90 degrees
Routing:
- net /Address decoder/D7: track 33.6 -> 115.1 mm, vias 0 -> 2
- net /Address decoder/-RESET: track 0.00 -> 75.6 mm, vias 0 -> 2
- net /Address decoder/D6: track 33.6 -> 107.2 mm, vias 0 -> 2
- net /Address decoder/-IORQ: track 0.00 -> 69.2 mm, vias 0 -> 1
- net +5VD: track 532.1 -> 596.7 mm, vias 5 -> 1
- net GNDD: track 634.7 -> 696.0 mm, vias 4 -> 2
- net /Address decoder/-WRSEL5: track 0.00 -> 58.4 mm, vias 0 -> 1
- net Net-(U10-Q6): track 0.00 -> 52.0 mm, vias 0 -> 1
- net /Address decoder/-WRSEL4: track 0.00 -> 44.3 mm, vias 0 -> 1
- net Net-(U1-E1): track 16.8 -> 59.9 mm, vias 0 -> 1
- net /PMAN-DP interface/BLANK: track 0.00 -> 41.4 mm, vias 0 -> 1
- net Net-(U10-Q4): track 0.00 -> 41.0 mm, vias 0 -> 1
- net /Address decoder/D3: track 62.3 -> 99.2 mm
- net /Address decoder/D4: track 68.9 -> 103.4 mm
- net /Address decoder/D5: track 63.8 -> 97.8 mm
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Other:
- board size 102.6 x 85.1 mm -> 106.3 x 85.1 mm

Commit message: 260329
Routing:
- net /Address decoder/-WRSEL2: track 5.72 -> 126.2 mm, vias 0 -> 1
- net /Address decoder/-WRSEL3: track 5.72 -> 124.9 mm, vias 0 -> 6
- net /Address decoder/-WRSEL1: track 5.72 -> 123.1 mm, vias 0 -> 2
- net /Address decoder/-WRSEL0: track 5.72 -> 121.6 mm, vias 0 -> 2
- net /Address decoder/-WR: track 0.00 -> 93.3 mm, vias 0 -> 3
- net /Address decoder/-RD: track 0.00 -> 79.5 mm, vias 0 -> 1
- net /Address decoder/A0: track 17.0 -> 88.2 mm, vias 0 -> 1
- net /Address decoder/A1: track 16.9 -> 84.6 mm, vias 0 -> 1
- net Net-(U10-Q1): track 0.00 -> 62.2 mm, vias 0 -> 1
- net Net-(U10-Q0): track 0.00 -> 61.5 mm, vias 0 -> 1
- net /Address decoder/A2: track 16.8 -> 73.2 mm
- net Net-(U10-Q2): track 0.00 -> 51.1 mm, vias 0 -> 1
- net Net-(U5-CE): track 0.00 -> 50.7 mm
- net Net-(U9-B2): track 0.00 -> 47.8 mm, vias 0 -> 1
- net Net-(U9-B1): track 0.00 -> 47.3 mm, vias 0 -> 1
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
Commit message: 260330
Routing:
- net /Address decoder/-WRSEL2: track 126.2 -> 131.4 mm
- net Net-(U10-Q1): track 62.2 -> 57.5 mm
- net Net-(U5-CE): track 50.7 -> 53.6 mm
- net Net-(RN1-R8): track 35.1 -> 32.9 mm
- net Net-(U10-Q7): track 45.1 -> 47.2 mm
- net Net-(U9-B1): track 47.3 -> 48.5 mm
- net Net-(U10-Q5): track 30.8 -> 31.8 mm
- net Net-(U10-Q0): track 61.5 -> 62.5 mm
- net Net-(J6-Pin_2): track 16.9 -> 17.7 mm
- net /Address decoder/-WRSEL3: track 124.9 -> 124.1 mm
- net /Address decoder/A1: track 84.6 -> 83.9 mm
- net /Address decoder/A2: track 73.2 -> 72.5 mm
Other:
- board text added: "2026 https://www.pozsarzs.hu"
- board text added: "PMAN-IF"

Commit message: 260330
Parts:
- added J8: Conn_01x02_Pin, Connector_PinHeader_2.54mm:PinHeader_1x02_P2.54mm_Vertical, F.Cu at (194.4, 127.0)
Connections:
- net /Address decoder/-IORQ renamed /address decoder/-IORQ
- net /Address decoder/-RD renamed /address decoder/-RD
- net /Address decoder/-RDSEL0 renamed /address decoder/-RDSEL0
- net /Address decoder/-RDSEL1 renamed /address decoder/-RDSEL1
- net /Address decoder/-RDSEL2 renamed /address decoder/-RDSEL2
- net /Address decoder/-RDSEL3 renamed /address decoder/-RDSEL3
- net /Address decoder/-RDSEL4 renamed /address decoder/-RDSEL4
- net /Address decoder/-RDSEL5 renamed /address decoder/-RDSEL5
- net /Address decoder/-RDSEL6 renamed /address decoder/-RDSEL6
- net /Address decoder/-RDSEL7 renamed /address decoder/-RDSEL7
- net /Address decoder/-RESET renamed /address decoder/-RESET
- net /Address decoder/-WR renamed /address decoder/-WR
- net /Address decoder/-WRSEL0 renamed /address decoder/-WRSEL0
- net /Address decoder/-WRSEL1 renamed /address decoder/-WRSEL1
- net /Address decoder/-WRSEL2 renamed /address decoder/-WRSEL2
- net /Address decoder/-WRSEL3 renamed /address decoder/-WRSEL3
- net /Address decoder/-WRSEL4 renamed /address decoder/-WRSEL4
- net /Address decoder/-WRSEL5 renamed /address decoder/-WRSEL5
- net /Address decoder/-WRSEL6 renamed /address decoder/-WRSEL6
- net /Address decoder/-WRSEL7 renamed /address decoder/-WRSEL7
- net /Address decoder/A0 renamed /address decoder/A0
- net /Address decoder/A1 renamed /address decoder/A1
- net /Address decoder/A2 renamed /address decoder/A2
- net /Address decoder/A3 renamed /address decoder/A3
- net /Address decoder/A4 renamed /address decoder/A4
- net /Address decoder/A5 renamed /address decoder/A5
- net /Address decoder/A6 renamed /address decoder/A6
- net /Address decoder/A7 renamed /address decoder/A7
- net /Address decoder/D0 renamed /address decoder/D0
- net /Address decoder/D1 renamed /address decoder/D1
- net /Address decoder/D2 renamed /address decoder/D2
- net /Address decoder/D3 renamed /address decoder/D3
- net /Address decoder/D4 renamed /address decoder/D4
- net /Address decoder/D5 renamed /address decoder/D5
- net /Address decoder/D6 renamed /address decoder/D6
- net /Address decoder/D7 renamed /address decoder/D7
- net /PMAN-DP interface/BLANK renamed /display interface/BLANK
- J1 pad 66: unconnected-(J1-Pin_66-Pad66) -> Net-(J1-Pin_66)
Routing:
- net Net-(J1-Pin_66): track 0.00 -> 38.1 mm, vias 0 -> 2
- net GNDD: track 697.8 -> 703.4 mm
- net +5VD: track 599.6 -> 595.2 mm
