File: Zacchaeus computer/hardware/PTAP Tape interface module/ptap/ptap-3.kicad_sch (KiCad schematic)
At the start: 29 parts, among them J7 Screw_Terminal_01x03, J8 Screw_Terminal_01x05, P1 1.5k, U7 TL071, U8 TL071

Commit message: 260405
Parts:
- added D1, D2: 1N4001, symbol Device:D
- added D3, D4: LED, symbol Device:LED
- added R14, R15: 2.2k, symbol Device:R
- renumbered R16 to R12, R17 to R13, R18 to R16, R19 to R17, R20 to R18, R21 to R19, R22 to R20, R23 to R21, R24 to R22, R25 to R23, R26 to R24, U7 to U8, U8 to U9
Connections:
- net +12VA: now also D1.1 (K), D3.2 (A)
- net -12VA: now also D2.2 (A), D4.1 (K)
- net GNDA: now also R14.2, R15.2
- new net: D3.1 (K), R14.1
- new net: D4.2 (A), R15.1
- new net: D1.2 (A), D2.1 (K)
Other:
- note added: "output level (mic-line)"
- moved on the sheet: C16, C17, C18, C19, C20, C21, J7
