File: Zacchaeus computer/hardware/PTAP Tape interface module/ptap/ptap.kicad_sch (KiCad schematic)
At the start: 9 parts

Commit message: 260404
Parts:
- removed C? (x2): C, symbol Device:C
- removed R?: R, symbol Device:R
- removed U?: DS87C520, MODULE, symbol DS87C520:DS87C520
- removed U?: 74LS373, symbol 74xx:74LS373
- removed U? (x2): 74LS139, symbol 74xx:74LS139
- removed U?: 74LS245, symbol 74xx:74LS245
- removed Y?: Crystal, symbol Device:Crystal
Connections:
- no-connect marks 16 -> 2
Other:
- added sheet address decoder (ptap-1.kicad_sch)
- added sheet analog circuits (ptap-3.kicad_sch)
- added sheet controller circuit (ptap-2.kicad_sch)
- company: (none) -> Pozsar Zsolt
- title: (none) -> PTAP - Tape and speaker interface

Commit message: 260405
Other:
- sheet address decoder ports: added RESET; removed ~{RESET}
- sheet controller circuit ports: added RESET; removed ~{RESET}
